Commit message: Hands orientation fixed, forearm upgraded

File: mechanical/master_assembly.xacro (robot description, xacro)
@@ -2,4 +2,8 @@
 <robot name="RevEx_Full_Assembly" xmlns:xacro="http://wiki.ros.org/xacro">
   <xacro:property name="mesh_dir" value="C:/Projects/RevExBot/RevEx_Phase1_Hardware/mechanical/meshes" />
+  <xacro:property name="leg_scale" value="1.5" />
+  <xacro:property name="leg_inertia_scale" value="${leg_scale * leg_scale}" />
+  <xacro:property name="effort_scale" value="${leg_scale}" />
+  <xacro:property name="pelvis_raise" value="0.24515" />
   <material name="Grey"><color rgba="0.6 0.6 0.6 1.0" /></material>
   <material name="DarkGrey"><color rgba="0.22 0.22 0.22 1.0" /></material>
@@ -9,7 +13,6 @@
     <parent link="base_link" />
     <child link="pelvis_link" />
-    <origin xyz="0 0 0" rpy="0 0 0" />
-  </joint>
-  <!-- ========== PELVIS ========== -->
+    <origin xyz="0 0 ${pelvis_raise}" rpy="0 0 0" />
+  </joint>
   <link name="pelvis_link">
     <inertial>
@@ -29,6 +32,4 @@
     </collision>
   </link>
-  <!-- ========== LEFT LEG (full inertials, collisions) ========== -->
-  <!-- left_hip_pitch_link -->
   <link name="left_hip_pitch_link">
     <inertial>
@@ -48,8 +49,7 @@
     <parent link="pelvis_link" /><child link="left_hip_pitch_link" />
     <axis xyz="0 1 0" />
-    <limit lower="-2.094" upper="1.047" effort="120" velocity="8" />
+    <limit lower="-2.094" upper="1.047" effort="${120 * effort_scale}" velocity="8" />
     <dynamics damping="0.095625" friction="0" />
   </joint>
-  <!-- left_hip_roll_link -->
   <link name="left_hip_roll_link">
     <inertial>
@@ -65,19 +65,18 @@
     <parent link="left_hip_pitch_link" /><child link="left_hip_roll_link" />
     <axis xyz="1 0 0" />
-    <limit lower="-0.698" upper="0.698" effort="100" velocity="8" />
+    <limit lower="-0.698" upper="0.698" effort="${100 * effort_scale}" velocity="8" />
     <dynamics damping="0.11" friction="0" />
   </joint>
-  <!-- left_hip_yaw_link -->
   <link name="left_hip_yaw_link">
     <inertial>
-      <origin xyz="0.00107948196019631 0.00102490074879569 -0.120338859084698" rpy="0 0 0" />
-      <mass value="1.86657016436158" />
-      <inertia ixx="0.00341632805787578" ixy="1.12872344062739E-05" ixz="2.89779048114687E-05"
-               iyy="0.00356015908770306" iyz="-0.000119761895425219" izz="0.00137524372110325" />
-    </inertial>
-    <visual><geometry><mesh filename="${mesh_dir}/LEFT_HIP_YAW.STL" /></geometry><material name="Grey" /></visual>
+      <origin xyz="0.00107948196019631 0.00102490074879569 ${-0.120338859084698 * leg_scale}" rpy="0 0 0" />
+      <mass value="${1.86657016436158 * leg_scale}" />
+      <inertia ixx="${0.00341632805787578 * leg_inertia_scale}" ixy="1.12872344062739E-05" ixz="2.89779048114687E-05"
+               iyy="${0.00356015908770306 * leg_inertia_scale}" iyz="-0.000119761895425219" izz="${0.00137524372110325 * leg_scale}" />
+    </inertial>
+    <visual><geometry><mesh filename="${mesh_dir}/LEFT_HIP_YAW.STL" scale="1 1 ${leg_scale}"/></geometry><material name="Grey" /></visual>
     <collision name="left_hip_yaw_collision">
-      <origin xyz="0 0 -0.085" rpy="0 0 0" />
-      <geometry><cylinder radius="0.04" length="0.07" /></geometry>
+      <origin xyz="0 0 ${-0.085 * leg_scale}" rpy="0 0 0" />
+      <geometry><cylinder radius="0.04" length="${0.07 * leg_scale}" /></geometry>
     </collision>
   </link>
@@ -86,29 +85,27 @@
     <parent link="left_hip_roll_link" /><child link="left_hip_yaw_link" />
     <axis xyz="0 0 -1" />
-    <limit lower="-0.698" upper="0.698" effort="80" velocity="8" />
+    <limit lower="-0.698" upper="0.698" effort="${80 * effort_scale}" velocity="8" />
     <dynamics damping="0.038" friction="0" />
   </joint>
-  <!-- left_knee_link -->
   <link name="left_knee_link">
     <inertial>
-      <origin xyz="-0.000500664455004187 0.000509289489479564 -0.11269288769412" rpy="0 0 0" />
-      <mass value="2.39114151033076" />
-      <inertia ixx="0.00962172060189828" ixy="9.87646392241852E-06" ixz="-0.000645140055016828"
-               iyy="0.00975314356560942" iyz="-7.94058135611557E-06" izz="0.00233095236940007" />
-    </inertial>
-    <visual><geometry><mesh filename="${mesh_dir}/LEFT_KNEE.STL" /></geometry><material name="Grey" /></visual>
+      <origin xyz="-0.000500664455004187 0.000509289489479564 ${-0.11269288769412 * leg_scale}" rpy="0 0 0" />
+      <mass value="${2.39114151033076 * leg_scale}" />
+      <inertia ixx="${0.00962172060189828 * leg_inertia_scale}" ixy="9.87646392241852E-06" ixz="-0.000645140055016828"
+               iyy="${0.00975314356560942 * leg_inertia_scale}" iyz="-7.94058135611557E-06" izz="${0.00233095236940007 * leg_scale}" />
+    </inertial>
+    <visual><geometry><mesh filename="${mesh_dir}/LEFT_KNEE.STL" scale="1 1 ${leg_scale}"/></geometry><material name="Grey" /></visual>
     <collision name="left_knee_collision">
-      <origin xyz="0 0 -0.13" rpy="0 0 0" />
-      <geometry><cylinder radius="0.04" length="0.18" /></geometry>
+      <origin xyz="0 0 ${-0.13 * leg_scale}" rpy="0 0 0" />
+      <geometry><cylinder radius="0.04" length="${0.18 * leg_scale}" /></geometry>
     </collision>
   </link>
   <joint name="left_knee_joint" type="revolute">
-    <origin xyz="0 0 -0.195639999999998" rpy="0 0 0" />
+    <origin xyz="0 0 ${-0.195639999999998 * leg_scale}" rpy="0 0 0" />
     <parent link="left_hip_yaw_link" /><child link="left_knee_link" />
     <axis xyz="0 1 0" />
-    <limit lower="0" upper="1.5" effort="150" velocity="8" />
+    <limit lower="0" upper="1.5" effort="${150 * effort_scale}" velocity="8" />
     <dynamics damping="0.0339552" friction="0" />
   </joint>
-  <!-- left_ankle_pitch_link -->
   <link name="left_ankle_pitch_link">
     <inertial>
@@ -121,11 +118,10 @@
   </link>
   <joint name="left_ankle_pitch_joint" type="revolute">
-    <origin xyz="0 0 -0.294662336087024" rpy="0 0 0" />
+    <origin xyz="0 0 ${-0.294662336087024 * leg_scale}" rpy="0 0 0" />
     <parent link="left_knee_link" /><child link="left_ankle_pitch_link" />
     <axis xyz="0 1 0" />
-    <limit lower="-0.35" upper="0.35" effort="80" velocity="8" />
+    <limit lower="-0.35" upper="0.35" effort="${80 * effort_scale}" velocity="8" />
     <dynamics damping="0.0565056" friction="0" />
   </joint>
-  <!-- left_ankle_roll_link -->
   <link name="left_ankle_roll_link">
     <inertial>
@@ -141,8 +137,7 @@
     <parent link="left_ankle_pitch_link" /><child link="left_ankle_roll_link" />
     <axis xyz="-1 0 0" />
-    <limit lower="-0.1" upper="0.1" effort="50" velocity="8" />
+    <limit lower="-0.1" upper="0.1" effort="${50 * effort_scale}" velocity="8" />
     <dynamics damping="0.0565056" friction="0" />
   </joint>
-  <!-- left_toe_link -->
   <link name="left_toe_link">
     <inertial>
@@ -161,9 +156,7 @@
     <parent link="left_ankle_roll_link" /><child link="left_toe_link" />
     <axis xyz="0.010532 0.99994 0" />
-    <limit lower="-1.047" upper="0.349" effort="30" velocity="8" />
+    <limit lower="-1.047" upper="0.349" effort="${30 * effort_scale}" velocity="8" />
     <dynamics damping="0.001" friction="0.02" />
   </joint>
-  <!-- ========== RIGHT LEG (mirrored) ========== -->
-  <!-- right_hip_pitch_link -->
   <link name="right_hip_pitch_link">
     <inertial>
@@ -183,8 +176,7 @@
     <parent link="pelvis_link" /><child link="right_hip_pitch_link" />
     <axis xyz="0 -1 0" />
-    <limit lower="-1.047" upper="2.094" effort="120" velocity="8" />
+    <limit lower="-1.047" upper="2.094" effort="${120 * effort_scale}" velocity="8" />
     <dynamics damping="0.095625" friction="0" />
   </joint>
-  <!-- right_hip_roll_link -->
   <link name="right_hip_roll_link">
     <inertial>
@@ -200,19 +192,18 @@
     <parent link="right_hip_pitch_link" /><child link="right_hip_roll_link" />
     <axis xyz="1 0 0" />
-    <limit lower="-0.698" upper="0.698" effort="100" velocity="8" />
+    <limit lower="-0.698" upper="0.698" effort="${100 * effort_scale}" velocity="8" />
     <dynamics damping="0.11" friction="0" />
   </joint>
-  <!-- right_hip_yaw_link -->
   <link name="right_hip_yaw_link">
     <inertial>
-      <origin xyz="0.0010759524804974 -0.00102176499629938 -0.120345116027848" rpy="0 0 0" />
-      <mass value="1.86647220449567" />
-      <inertia ixx="0.00341588734528233" ixy="-1.17597783272228E-05" ixz="2.91733595327906E-05"
-               iyy="0.00355990015451682" iyz="0.00011971567133214" izz="0.00137525272174267" />
-    </inertial>
-    <visual><geometry><mesh filename="${mesh_dir}/RIGHT_HIP_YAW.STL" /></geometry><material name="Grey" /></visual>
+      <origin xyz="0.0010759524804974 -0.00102176499629938 ${-0.120345116027848 * leg_scale}" rpy="0 0 0" />
+      <mass value="${1.86647220449567 * leg_scale}" />
+      <inertia ixx="${0.00341588734528233 * leg_inertia_scale}" ixy="-1.17597783272228E-05" ixz="2.91733595327906E-05"
+               iyy="${0.00355990015451682 * leg_inertia_scale}" iyz="0.00011971567133214" izz="${0.00137525272174267 * leg_scale}" />
+    </inertial>
+    <visual><geometry><mesh filename="${mesh_dir}/RIGHT_HIP_YAW.STL" scale="1 1 ${leg_scale}"/></geometry><material name="Grey" /></visual>
     <collision name="right_hip_yaw_collision">
-      <origin xyz="0 0 -0.085" rpy="0 0 0" />
-      <geometry><cylinder radius="0.04" length="0.07" /></geometry>
+      <origin xyz="0 0 ${-0.085 * leg_scale}" rpy="0 0 0" />
+      <geometry><cylinder radius="0.04" length="${0.07 * leg_scale}" /></geometry>
     </collision>
   </link>
@@ -221,29 +212,27 @@
     <parent link="right_hip_roll_link" /><child link="right_hip_yaw_link" />
     <axis xyz="0 0 -1" />
-    <limit lower="-0.698" upper="0.698" effort="80" velocity="8" />
+    <limit lower="-0.698" upper="0.698" effort="${80 * effort_scale}" velocity="8" />
     <dynamics damping="0.038" friction="0" />
   </joint>
-  <!-- right_knee_link -->
   <link name="right_knee_link">
     <inertial>
-      <origin xyz="-0.000497587233719177 -0.000414757224949908 -0.112692693562372" rpy="0 0 0" />
-      <mass value="2.39110172735043" />
-      <inertia ixx="0.00962148213806552" ixy="-9.87527823922245E-06" ixz="-0.00064509471825313"
-               iyy="0.00975287238047396" iyz="7.98431367388265E-06" izz="0.0023309035826248" />
-    </inertial>
-    <visual><geometry><mesh filename="${mesh_dir}/RIGHT_KNEE.STL" /></geometry><material name="Grey" /></visual>
+      <origin xyz="-0.000497587233719177 -0.000414757224949908 ${-0.112692693562372 * leg_scale}" rpy="0 0 0" />
+      <mass value="${2.39110172735043 * leg_scale}" />
+      <inertia ixx="${0.00962148213806552 * leg_inertia_scale}" ixy="-9.87527823922245E-06" ixz="-0.00064509471825313"
+               iyy="${0.00975287238047396 * leg_inertia_scale}" iyz="7.98431367388265E-06" izz="${0.0023309035826248 * leg_scale}" />
+    </inertial>
+    <visual><geometry><mesh filename="${mesh_dir}/RIGHT_KNEE.STL" scale="1 1 ${leg_scale}"/></geometry><material name="Grey" /></visual>
     <collision name="right_knee_collision">
-      <origin xyz="0 0 -0.13" rpy="0 0 0" />
-      <geometry><cylinder radius="0.04" length="0.18" /></geometry>
+      <origin xyz="0 0 ${-0.13 * leg_scale}" rpy="0 0 0" />
+      <geometry><cylinder radius="0.04" length="${0.18 * leg_scale}" /></geometry>
     </collision>
   </link>
   <joint name="right_knee_joint" type="revolute">
-    <origin xyz="0 0 -0.195639999999998" rpy="0 0 0" />
+    <origin xyz="0 0 ${-0.195639999999998 * leg_scale}" rpy="0 0 0" />
     <parent link="right_hip_yaw_link" /><child link="right_knee_link" />
     <axis xyz="0 -1 0" />
-    <limit lower="-1.5" upper="0" effort="150" velocity="8" />
+    <limit lower="-1.5" upper="0" effort="${150 * effort_scale}" velocity="8" />
     <dynamics damping="0.0339552" friction="0" />
   </joint>
-  <!-- right_ankle_pitch_link -->
   <link name="right_ankle_pitch_link">
     <inertial>
@@ -256,11 +245,10 @@
   </link>
   <joint name="right_ankle_pitch_joint" type="revolute">
-    <origin xyz="0 0.0001 -0.294662336087023" rpy="0 0 0" />
+    <origin xyz="0 0.0001 ${-0.294662336087023 * leg_scale}" rpy="0 0 0" />
     <parent link="right_knee_link" /><child link="right_ankle_pitch_link" />
     <axis xyz="0 -1 0" />
-    <limit lower="-0.35" upper="0.35" effort="80" velocity="8" />
+    <limit lower="-0.35" upper="0.35" effort="${80 * effort_scale}" velocity="8" />
     <dynamics damping="0.0565056" friction="0" />
   </joint>
-  <!-- right_ankle_roll_link -->
   <link name="right_ankle_roll_link">
     <inertial>
@@ -276,8 +264,7 @@
     <parent link="right_ankle_pitch_link" /><child link="right_ankle_roll_link" />
     <axis xyz="-1 0 0" />
-    <limit lower="-0.1" upper="0.1" effort="50" velocity="8" />
+    <limit lower="-0.1" upper="0.1" effort="${50 * effort_scale}" velocity="8" />
     <dynamics damping="0.0565056" friction="0" />
   </joint>
-  <!-- right_toe_link -->
   <link name="right_toe_link">
     <inertial>
@@ -296,9 +283,7 @@
     <parent link="right_ankle_roll_link" /><child link="right_toe_link" />
     <axis xyz="0.0074685 -0.99997 0" />
-    <limit lower="-0.349" upper="1.047" effort="30" velocity="8" />
+    <limit lower="-0.349" upper="1.047" effort="${30 * effort_scale}" velocity="8" />
     <dynamics damping="0.001" friction="0.02" />
   </joint>
-  <!-- ========== UPPER BODY ========== -->
-  <!-- waist_yaw_link -->
   <link name="waist_yaw_link">
     <inertial>
@@ -389,6 +374,4 @@
     <origin xyz="0.126 -0.029 0.115" rpy="0 0 0" />
   </joint>
-  <!-- ========== RIGHT ARM (full inertials) ========== -->
-  <!-- right_shoulder_pitch_link -->
   <link name="right_shoulder_pitch_link">
     <inertial>
@@ -401,5 +384,5 @@
   </link>
   <joint name="right_shoulder_pitch_joint" type="revolute">
-    <origin xyz="-0.0262128253533167 -0.0964999999999998 0.261140483320038" rpy="0 -25 0" />
+    <origin xyz="-0.0262128253533167 -0.0964999999999998 0.261140483320038" rpy="0 -0.436332 0" />
     <parent link="waist_yaw_link" /><child link="right_shoulder_pitch_link" />
     <axis xyz="0 -1 0" />
@@ -407,5 +390,4 @@
     <dynamics damping="0.11" friction="0" />
   </joint>
-  <!-- right_shoulder_roll_link -->
   <link name="right_shoulder_roll_link">
     <inertial>
@@ -422,5 +404,5 @@
   </link>
   <joint name="right_shoulder_roll_joint" type="revolute">
-    <origin xyz="0 -0.0653532232325457 -6.33413504113611E-05" rpy="-0.25 0 0" />
+    <origin xyz="0 -0.0653532232325457 -6.33413504113611E-05" rpy="0 0 0" />
     <parent link="right_shoulder_pitch_link" />
     <child link="right_shoulder_roll_link" />
@@ -429,5 +411,4 @@
     <dynamics damping="0.0339552" friction="0" />
   </joint>
-  <!-- right_shoulder_yaw_link -->
   <link name="right_shoulder_yaw_link">
     <inertial>
@@ -446,5 +427,4 @@
     <dynamics damping="0.038" friction="0" />
   </joint>
-  <!-- right_elbow_link -->
   <link name="right_elbow_link">
     <inertial>
@@ -467,6 +447,4 @@
     <dynamics damping="0.0282528" friction="0" />
   </joint>
-  <!-- ========== LEFT ARM (mirrored) ========== -->
-  <!-- left_shoulder_pitch_link -->
   <link name="left_shoulder_pitch_link">
     <inertial>
@@ -479,5 +457,5 @@
   </link>
   <joint name="left_shoulder_pitch_joint" type="revolute">
-    <origin xyz="-0.0262128253533159 0.0965000000000001 0.261140483320038" rpy="0 -25 0" />
+    <origin xyz="-0.0262128253533159 0.0965000000000001 0.261140483320038" rpy="0 -0.436332 0" />
     <parent link="waist_yaw_link" /><child link="left_shoulder_pitch_link" />
     <axis xyz="0 1 0" />
@@ -485,5 +463,4 @@
     <dynamics damping="0.11" friction="0" />
   </joint>
-  <!-- left_shoulder_roll_link -->
   <link name="left_shoulder_roll_link">
     <inertial>
@@ -500,5 +477,5 @@
   </link>
   <joint name="left_shoulder_roll_joint" type="revolute">
-    <origin xyz="0.000100000000001779 0.0653532232325531 0" rpy="0.25 0 0" />
+    <origin xyz="0.000100000000001779 0.0653532232325531 0" rpy="0 0 0" />
     <parent link="left_shoulder_pitch_link" />
     <child link="left_shoulder_roll_link" />
@@ -507,5 +484,4 @@
     <dynamics damping="0.0339552" friction="0" />
   </joint>
-  <!-- left_shoulder_yaw_link -->
   <link name="left_shoulder_yaw_link">
     <inertial>
@@ -524,5 +500,4 @@
     <dynamics damping="0.038" friction="0" />
   </joint>
-  <!-- left_elbow_link -->
   <link name="left_elbow_link">
     <inertial>
@@ -544,26 +519,29 @@
     <limit lower="0" upper="2.443" effort="60" velocity="6" />
     <dynamics damping="0.0282528" friction="0" />
-  </joint><xacro:include filename="shadow_hand.xacro" />
+  </joint>
+  <xacro:include filename="shadow_hand.xacro" />
   <xacro:shadow_hand
       prefix="rh_"
       mesh_dir="${mesh_dir}"
-      forearm_visual_xyz="-0.02104 0.16338 -0.13304"
-      wrist_xyz="0.02104 0 -0.248456"   wrist_rpy="3.14159 0 1.5708"
+      forearm_visual_xyz="0.107504 0.162107 -0.113857"
+      wrist_xyz="-0.013287 0 -0.248456"
+      wrist_rpy="3.14159 0.1396263 0"
       mirror="false" />
   <joint name="right_elbow_to_forearm_glue" type="fixed">
     <parent link="right_elbow_link" />
     <child link="rh_forearm" />
-    <origin xyz="0 0 0" rpy="0 0 0" />
+    <origin xyz="0 0 0" rpy="0 -0.1396263 0" />
   </joint>
   <xacro:shadow_hand
       prefix="lh_"
       mesh_dir="${mesh_dir}"
-      forearm_visual_xyz="-0.02104 -0.16338 -0.13304"
-      wrist_xyz="0 0 -0.207"   wrist_rpy="3.14159 0 1.5708"
+      forearm_visual_xyz="0.107504 -0.162107 -0.113857"
+      wrist_xyz="-0.013287 0 -0.248456"
+      wrist_rpy="3.14159 -0.1396263 3.14159"
       mirror="true" />
   <joint name="left_elbow_to_forearm_glue" type="fixed">
     <parent link="left_elbow_link" />
     <child link="lh_forearm" />
-    <origin xyz="0 0 0" rpy="0 0 0" />
+    <origin xyz="0 0 0" rpy="0 -0.1396263 0" />
   </joint>
 </robot>

File: mechanical/revexbot.urdf (robot description, URDF)
Before this commit: robot RevEx_Full_Assembly, 95 links, 94 joints
Links:
- link left_hip_yaw_link: mass 1.86657016436158 -> 2.79985524654237; geometry collision cylinder length=0.10500000000000001 radius=0.04; visual mesh filename=C:/Projects/RevExBot/RevEx_Phase1_Hardware/mechanical/meshe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 scale=1 1 1.5
- link left_knee_link: mass 2.39114151033076 -> 3.58671226549614; geometry collision cylinder length=0.27 radius=0.04; visual mesh filename=C:/Projects/RevExBot/RevEx_Phase1_Hardware/mechanical/meshe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 scale=1 1 1.5
- link right_hip_yaw_link: mass 1.86647220449567 -> 2.799708306743505; geometry collision cylinder length=0.10500000000000001 radius=0.04; visual mesh filename=C:/Projects/RevExBot/RevEx_Phase1_Hardware/mechanical/meshe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 scale=1 1 1.5
- link right_knee_link: mass 2.39110172735043 -> 3.5866525910256453; geometry collision cylinder length=0.27 radius=0.04; visual mesh filename=C:/Projects/RevExBot/RevEx_Phase1_Hardware/mechanical/meshe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 scale=1 1 1.5
Joints:
- joint base_joint: origin xyz=0 0 0 rpy=0 0 0 -> xyz=0 0 0.24515 rpy=0 0 0
- joint left_ankle_pitch_joint: limit lower=-0.35 upper=0.35 effort=80 velocity=8 -> lower=-0.35 upper=0.35 effort=120.0 velocity=8; origin xyz=0 0 -0.294662336087024 rpy=0 0 0 -> xyz=0 0 -0.44199350413053606 rpy=0 0 0
- joint left_ankle_roll_joint: limit lower=-0.1 upper=0.1 effort=50 velocity=8 -> lower=-0.1 upper=0.1 effort=75.0 velocity=8
- joint left_elbow_to_forearm_glue: origin xyz=0 0 0 rpy=0 0 0 -> xyz=0 0 0 rpy=0 -0.1396263 0
- joint left_hip_pitch_joint: limit lower=-2.094 upper=1.047 effort=120 velocity=8 -> lower=-2.094 upper=1.047 effort=180.0 velocity=8
- joint left_hip_roll_joint: limit lower=-0.698 upper=0.698 effort=100 velocity=8 -> lower=-0.698 upper=0.698 effort=150.0 velocity=8
- joint left_hip_yaw_joint: limit lower=-0.698 upper=0.698 effort=80 velocity=8 -> lower=-0.698 upper=0.698 effort=120.0 velocity=8
- joint left_knee_joint: limit lower=0 upper=1.5 effort=150 velocity=8 -> lower=0 upper=1.5 effort=225.0 velocity=8; origin xyz=0 0 -0.195639999999998 rpy=0 0 0 -> xyz=0 0 -0.293459999999997 rpy=0 0 0
- joint left_shoulder_pitch_joint: origin xyz=-0.0262128253533159 0.0965000000000001 0.261140483320038 rpy=0 -25 0 -> xyz=-0.0262128253533159 0.0965000000000001 0.261140483320038 rpy=0 -0.436332 0
- joint left_shoulder_roll_joint: origin xyz=0.000100000000001779 0.0653532232325531 0 rpy=0.25 0 0 -> xyz=0.000100000000001779 0.0653532232325531 0 rpy=0 0 0
- joint left_toe_joint: limit lower=-1.047 upper=0.349 effort=30 velocity=8 -> lower=-1.047 upper=0.349 effort=45.0 velocity=8
- joint lh_WRJ2: origin xyz=-0.02104 -0.16338 -0.207 rpy=3.14159 1.5708 0 -> xyz=-0.013287 0 -0.248456 rpy=3.14159 -0.1396263 3.14159
- joint rh_WRJ2: origin xyz=-0.02104 0.16338 -0.207 rpy=3.14159 1.5708 0 -> xyz=-0.013287 0 -0.248456 rpy=3.14159 0.1396263 0
- joint right_ankle_pitch_joint: limit lower=-0.35 upper=0.35 effort=80 velocity=8 -> lower=-0.35 upper=0.35 effort=120.0 velocity=8; origin xyz=0 0.0001 -0.294662336087023 rpy=0 0 0 -> xyz=0 0.0001 -0.4419935041305345 rpy=0 0 0
- joint right_ankle_roll_joint: limit lower=-0.1 upper=0.1 effort=50 velocity=8 -> lower=-0.1 upper=0.1 effort=75.0 velocity=8
- joint right_elbow_to_forearm_glue: origin xyz=0 0 0 rpy=0 0 0 -> xyz=0 0 0 rpy=0 -0.1396263 0
- joint right_hip_pitch_joint: limit lower=-1.047 upper=2.094 effort=120 velocity=8 -> lower=-1.047 upper=2.094 effort=180.0 velocity=8
- joint right_hip_roll_joint: limit lower=-0.698 upper=0.698 effort=100 velocity=8 -> lower=-0.698 upper=0.698 effort=150.0 velocity=8
- joint right_hip_yaw_joint: limit lower=-0.698 upper=0.698 effort=80 velocity=8 -> lower=-0.698 upper=0.698 effort=120.0 velocity=8
- joint right_knee_joint: limit lower=-1.5 upper=0 effort=150 velocity=8 -> lower=-1.5 upper=0 effort=225.0 velocity=8; origin xyz=0 0 -0.195639999999998 rpy=0 0 0 -> xyz=0 0 -0.293459999999997 rpy=0 0 0
- joint right_shoulder_pitch_joint: origin xyz=-0.0262128253533167 -0.0964999999999998 0.261140483320038 rpy=0 -25 0 -> xyz=-0.0262128253533167 -0.0964999999999998 0.261140483320038 rpy=0 -0.436332 0
- joint right_shoulder_roll_joint: origin xyz=0 -0.0653532232325457 -6.33413504113611E-05 rpy=-0.25 0 0 -> xyz=0 -0.0653532232325457 -6.33413504113611E-05 rpy=0 0 0
- joint right_toe_joint: limit lower=-0.349 upper=1.047 effort=30 velocity=8 -> lower=-0.349 upper=1.047 effort=45.0 velocity=8
