Commit message: Fixed height of robot (increased), UPgraded and finalized the orientation

File: mechanical/master_assembly.xacro (robot description, xacro)
@@ -334,5 +334,5 @@
     <visual>
       <origin xyz="0 0 0" rpy="0 0 0" />
-      <geometry><mesh filename="${mesh_dir}/head.stl" /></geometry>
+      <geometry><mesh filename="${mesh_dir}/HEAD.STL" /></geometry>
       <material name="LightGrey" />
     </visual>
@@ -384,5 +384,5 @@
   </link>
   <joint name="right_shoulder_pitch_joint" type="revolute">
-    <origin xyz="-0.0262128253533167 -0.0964999999999998 0.261140483320038" rpy="0 -0.436332 0" />
+    <origin xyz="-0.0262128253533167 -0.0964999999999998 0.261140483320038" rpy="-0.261799 0 0" />
     <parent link="waist_yaw_link" /><child link="right_shoulder_pitch_link" />
     <axis xyz="0 -1 0" />
@@ -457,5 +457,5 @@
   </link>
   <joint name="left_shoulder_pitch_joint" type="revolute">
-    <origin xyz="-0.0262128253533159 0.0965000000000001 0.261140483320038" rpy="0 -0.436332 0" />
+    <origin xyz="-0.0262128253533159 0.0965000000000001 0.261140483320038" rpy="0.261799 0 0" />
     <parent link="waist_yaw_link" /><child link="left_shoulder_pitch_link" />
     <axis xyz="0 1 0" />

File: mechanical/revexbot.urdf (robot description, URDF)
Before this commit: robot RevEx_Full_Assembly, 95 links, 94 joints
Joints:
- joint left_shoulder_pitch_joint: origin xyz=-0.0262128253533159 0.0965000000000001 0.261140483320038 rpy=0 -0.436332 0 -> xyz=-0.0262128253533159 0.0965000000000001 0.261140483320038 rpy=0.261799 0 0
- joint lh_FFJ4: axis 0 -1 0 -> 0 1 0
- joint lh_LFJ4: axis 0 1 0 -> 0 -1 0
- joint lh_LFJ5: axis 1 0 0 -> -1 0 0
- joint lh_MFJ4: axis 0 -1 0 -> 0 1 0
- joint lh_RFJ4: axis 0 1 0 -> 0 -1 0
- joint right_shoulder_pitch_joint: origin xyz=-0.0262128253533167 -0.0964999999999998 0.261140483320038 rpy=0 -0.436332 0 -> xyz=-0.0262128253533167 -0.0964999999999998 0.261140483320038 rpy=-0.261799 0 0

File: mechanical/shadow_hand.xacro (robot description, xacro)
@@ -3,4 +3,5 @@
     <xacro:macro name="shadow_hand" params="prefix mesh_dir wrist_xyz wrist_rpy forearm_visual_xyz mirror:=false">
         <xacro:property name="f_x" value="${-1 if mirror else 1}" />
+        <xacro:property name="ab_x" value="${1 if mirror else -1}" />
         <link name="${prefix}forearm">
             <inertial>
@@ -98,49 +99,33 @@
             <collision>
                 <origin rpy="0 0 0" xyz="${0.011 * f_x} 0.0085 0.038" />
-                <geometry>
-                    <box size="0.062 0.007 0.098" />
-                </geometry>
+                <geometry><box size="0.062 0.007 0.098" /></geometry>
             </collision>
             <collision>
                 <origin rpy="0 0 0" xyz="${-0.002 * f_x} -0.0035 0.038" />
-                <geometry>
-                    <box size="0.036 0.017 0.098" />
-                </geometry>
+                <geometry><box size="0.036 0.017 0.098" /></geometry>
             </collision>
             <collision>
                 <origin rpy="0 0 0" xyz="${0.029 * f_x} -0.0035 0.082" />
-                <geometry>
-                    <box size="0.026 0.017 0.010" />
-                </geometry>
+                <geometry><box size="0.026 0.017 0.010" /></geometry>
             </collision>
             <collision>
                 <origin rpy="${0.2 * f_x} 0 ${0.25 * f_x}" xyz="${0.0265 * f_x} -0.001 0.070" />
-                <geometry>
-                    <box size="0.026 0.014 0.018" />
-                </geometry>
+                <geometry><box size="0.026 0.014 0.018" /></geometry>
             </collision>
             <collision>
                 <origin rpy="0 0 0" xyz="${0.0315 * f_x} -0.0085 0.001" />
-                <geometry>
-                    <box size="0.021 0.027 0.024" />
-                </geometry>
+                <geometry><box size="0.021 0.027 0.024" /></geometry>
             </collision>
             <collision>
                 <origin rpy="0 0 ${-0.48 * f_x}" xyz="${0.0125 * f_x} -0.015 0.009" />
-                <geometry>
-                    <box size="0.022 0.005 0.040" />
-                </geometry>
+                <geometry><box size="0.022 0.005 0.040" /></geometry>
             </collision>
             <collision>
                 <origin rpy="0 0 0" xyz="${0.011 * f_x} 0 0.089" />
-                <geometry>
-                    <box size="0.018 0.024 0.004" />
-                </geometry>
+                <geometry><box size="0.018 0.024 0.004" /></geometry>
             </collision>
             <collision>
                 <origin rpy="0 0 0" xyz="${-0.03 * f_x} 0 0.009" />
-                <geometry>
-                    <box size="0.020 0.024 0.040" />
-                </geometry>
+                <geometry><box size="0.020 0.024 0.040" /></geometry>
             </collision>
         </link>
@@ -173,5 +158,5 @@
             <parent link="${prefix}palm" /><child link="${prefix}ffknuckle" />
             <origin rpy="0 0 0" xyz="${0.033 * f_x} 0 0.095" />
-            <axis xyz="0 -1 0" />
+            <axis xyz="0 ${ab_x} 0" />
             <limit effort="2" lower="-0.3490658503988659" upper="0.3490658503988659" velocity="2.0" /><dynamics damping="0.1" />
         </joint>
@@ -201,5 +186,5 @@
         </joint>
         <link name="${prefix}ffdistal">
-            <inertial><mass value="0.012" /><origin xyz="0 0 0.012" /><inertia ixx="0.00000094" ixy="0.0" ixz="0.0" iyy="0.0000011" iyz="0.0" izz="0.00000053" /></inertial>
+            <inertial><mass value="0.012" /><origin xyz="0 0 0.012" /><inertia ixx="0.00000094" ixy="0.0" ixz="0.0" iyy="0.000011" iyz="0.0" izz="0.00000053" /></inertial>
             <visual><origin rpy="0 0 0" xyz="0 0 0" /><geometry><mesh filename="${mesh_dir}/${prefix}f_distal_pst.stl" /></geometry></visual>
             <collision><origin rpy="0 0 0" xyz="0 0 0" /><geometry><mesh filename="${mesh_dir}/${prefix}f_distal_pst.stl" /></geometry></collision>
@@ -221,5 +206,5 @@
             <parent link="${prefix}palm" /><child link="${prefix}mfknuckle" />
             <origin rpy="0 0 0" xyz="${0.011 * f_x} 0 0.099" />
-            <axis xyz="0 -1 0" />
+            <axis xyz="0 ${ab_x} 0" />
             <limit effort="2" lower="-0.3490658503988659" upper="0.3490658503988659" velocity="2.0" /><dynamics damping="0.1" />
         </joint>
@@ -269,5 +254,5 @@
             <parent link="${prefix}palm" /><child link="${prefix}rfknuckle" />
             <origin rpy="0 0 0" xyz="${-0.011 * f_x} 0 0.095" />
-            <axis xyz="0 1 0" />
+            <axis xyz="0 ${-ab_x} 0" />
             <limit effort="2" lower="-0.3490658503988659" upper="0.3490658503988659" velocity="2.0" /><dynamics damping="0.1" />
         </joint>
@@ -309,5 +294,5 @@
         <link name="${prefix}rftip"><inertial><mass value="0.001" /><inertia ixx="0.00001" ixy="0.0" ixz="0.0" iyy="0.00001" iyz="0.0" izz="0.00001" /></inertial></link>
         <joint name="${prefix}RFtip" type="fixed"><parent link="${prefix}rfdistal" /><child link="${prefix}rftip" /><origin rpy="0 0 0" xyz="0 0 0.026" /></joint>
-<link name="${prefix}lfmetacarpal">
+        <link name="${prefix}lfmetacarpal">
             <inertial>
                 <origin rpy="0 ${0.9599 * f_x} 0" xyz="${0.031748676 * f_x} 0 0.02235294" />
@@ -333,5 +318,5 @@
             <child link="${prefix}lfmetacarpal" />
             <origin rpy="0 ${-0.9599 * f_x} 0" xyz="${-0.033 * f_x} 0 0.02071" />
-            <axis xyz="1 0 0" />
+            <axis xyz="${-ab_x} 0 0" />
             <limit effort="2" lower="0" upper="0.7853981633974483" velocity="2.0" />
             <dynamics damping="0.1" />
@@ -361,13 +346,8 @@
             <child link="${prefix}lfknuckle" />
             <origin rpy="0 ${0.9599 * f_x} 0" xyz="${0.05397275 * f_x} 0 0.03779463" />
-            <axis xyz="0 1 0" />
+            <axis xyz="0 ${-ab_x} 0" />
             <limit effort="2" lower="-0.3490658503988659" upper="0.3490658503988659" velocity="2.0" />
             <dynamics damping="0.1" />
         </joint>
-        <link name="${prefix}lfknuckle">
-            <inertial><origin rpy="0 0 0" xyz="0 0 0" /><mass value="0.008" /><inertia ixx="0.00000026" ixy="0.0" ixz="0.0" iyy="0.00000026" iyz="0.0" izz="0.00000032" /></inertial>
-            <visual><origin rpy="0 0 0" xyz="0 0 0.0005" /><geometry><mesh filename="${mesh_dir}/${prefix}f_knuckle_E3M5.stl" /></geometry><material name="LightGrey" /></visual>
-            <collision><origin rpy="0 1.5708 0" xyz="0 0 0" /><geometry><cylinder length="0.014" radius="0.007" /></geometry></collision>
-        </link>
         <link name="${prefix}lfproximal">
             <inertial><mass value="0.030" /><origin xyz="0 0 0.0225" /><inertia ixx="0.0000098" ixy="0.0" ixz="0.0" iyy="0.00001" iyz="0.0" izz="0.0000018" /></inertial>
@@ -448,5 +428,8 @@
             <collision><origin rpy="0 0 0" xyz="0 0 0.012" /><geometry><cylinder length="0.018" radius="0.011" /></geometry></collision>
             <collision><origin rpy="0 0 0" xyz="0 0 0.019" /><geometry><sphere radius="0.011" /></geometry></collision>
-            <collision><origin rpy="0 1.5708 0" xyz="0 0 0.032" /><geometry><cylinder length="0.014" radius="0.010" /></geometry></collision>
+            <collision>
+                <origin rpy="0 ${1.5708 * f_x} 0" xyz="0 0 0.032" />
+                <geometry><cylinder length="0.014" radius="0.010" /></geometry>
+            </collision>
         </link>
         <joint name="${prefix}THJ2" type="revolute">
