Commit message: Re-scaled down. Fixed and finalized the complete orientation

File: mechanical/revexbot.urdf (robot description, URDF)
Before this commit: robot RevEx_Full_Assembly, 95 links, 94 joints
Links:
- link left_hip_yaw_link: mass 2.79985524654237 -> 1.86657016436158; geometry collision cylinder length=0.07 radius=0.04; visual mesh filename=C:/Projects/RevExBot/RevEx_Phase1_Hardware/mechanical/meshe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
- link left_knee_link: mass 3.58671226549614 -> 2.39114151033076; geometry collision cylinder length=0.18 radius=0.04; visual mesh filename=C:/Projects/RevExBot/RevEx_Phase1_Hardware/mechanical/meshe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
- link lh_ffdistal: geometry collision box size=0.015 0.015 0.024; visual mesh filename=C:/Projects/RevExBot/RevEx_Phase1_Hardware/mechanical/meshe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
- link lh_lfdistal: geometry collision box size=0.015 0.015 0.024; visual mesh filename=C:/Projects/RevExBot/RevEx_Phase1_Hardware/mechanical/meshe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
- link lh_mfdistal: geometry collision box size=0.015 0.015 0.024; visual mesh filename=C:/Projects/RevExBot/RevEx_Phase1_Hardware/mechanical/meshe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
- link lh_rfdistal: geometry collision box size=0.015 0.015 0.024; visual mesh filename=C:/Projects/RevExBot/RevEx_Phase1_Hardware/mechanical/meshe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
- link lh_thdistal: geometry collision box size=0.018 0.018 0.028; visual mesh filename=C:/Projects/RevExBot/RevEx_Phase1_Hardware/mechanical/meshe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
- link rh_ffdistal: geometry collision box size=0.015 0.015 0.024; visual mesh filename=C:/Projects/RevExBot/RevEx_Phase1_Hardware/mechanical/meshe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
- link rh_lfdistal: geometry collision box size=0.015 0.015 0.024; visual mesh filename=C:/Projects/RevExBot/RevEx_Phase1_Hardware/mechanical/meshe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
- link rh_mfdistal: geometry collision box size=0.015 0.015 0.024; visual mesh filename=C:/Projects/RevExBot/RevEx_Phase1_Hardware/mechanical/meshe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
- link rh_rfdistal: geometry collision box size=0.015 0.015 0.024; visual mesh filename=C:/Projects/RevExBot/RevEx_Phase1_Hardware/mechanical/meshe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
- link rh_thdistal: geometry collision box size=0.018 0.018 0.028; visual mesh filename=C:/Projects/RevExBot/RevEx_Phase1_Hardware/mechanical/meshe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
- link right_hip_yaw_link: mass 2.799708306743505 -> 1.86647220449567; geometry collision cylinder length=0.07 radius=0.04; visual mesh filename=C:/Projects/RevExBot/RevEx_Phase1_Hardware/mechanical/meshe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
- link right_knee_link: mass 3.5866525910256453 -> 2.39110172735043; geometry collision cylinder length=0.18 radius=0.04; visual mesh filename=C:/Projects/RevExBot/RevEx_Phase1_Hardware/mechanical/meshe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
Joints:
- joint base_joint: origin xyz=0 0 0.24515 rpy=0 0 0 -> xyz=0 0 0 rpy=0 0 0
- joint left_ankle_pitch_joint: limit lower=-0.35 upper=0.35 effort=120.0 velocity=8 -> lower=-0.35 upper=0.35 effort=80 velocity=8; origin xyz=0 0 -0.44199350413053606 rpy=0 0 0 -> xyz=0 0 -0.294662336087024 rpy=0 0 0
- joint left_ankle_roll_joint: limit lower=-0.1 upper=0.1 effort=75.0 velocity=8 -> lower=-0.1 upper=0.1 effort=50 velocity=8
- joint left_hip_pitch_joint: limit lower=-2.094 upper=1.047 effort=180.0 velocity=8 -> lower=-2.094 upper=1.047 effort=120 velocity=8
- joint left_hip_roll_joint: limit lower=-0.698 upper=0.698 effort=150.0 velocity=8 -> lower=-0.698 upper=0.698 effort=100 velocity=8
- joint left_hip_yaw_joint: limit lower=-0.698 upper=0.698 effort=120.0 velocity=8 -> lower=-0.698 upper=0.698 effort=80 velocity=8
- joint left_knee_joint: limit lower=0 upper=1.5 effort=225.0 velocity=8 -> lower=0 upper=1.5 effort=150 velocity=8; origin xyz=0 0 -0.293459999999997 rpy=0 0 0 -> xyz=0 0 -0.195639999999998 rpy=0 0 0
- joint left_toe_joint: limit lower=-1.047 upper=0.349 effort=45.0 velocity=8 -> lower=-1.047 upper=0.349 effort=30 velocity=8
- joint lh_WRJ2: origin xyz=-0.013287 0 -0.248456 rpy=3.14159 -0.1396263 3.14159 -> xyz=-0.013352 0.000739 -0.189317 rpy=3.14159 -0.1396263 3.14159
- joint rh_WRJ2: origin xyz=-0.013287 0 -0.248456 rpy=3.14159 0.1396263 0 -> xyz=-0.013352 -0.000739 -0.189317 rpy=3.14159 0.1396263 0
- joint right_ankle_pitch_joint: limit lower=-0.35 upper=0.35 effort=120.0 velocity=8 -> lower=-0.35 upper=0.35 effort=80 velocity=8; origin xyz=0 0.0001 -0.4419935041305345 rpy=0 0 0 -> xyz=0 0.0001 -0.294662336087023 rpy=0 0 0
- joint right_ankle_roll_joint: limit lower=-0.1 upper=0.1 effort=75.0 velocity=8 -> lower=-0.1 upper=0.1 effort=50 velocity=8
- joint right_hip_pitch_joint: limit lower=-1.047 upper=2.094 effort=180.0 velocity=8 -> lower=-1.047 upper=2.094 effort=120 velocity=8
- joint right_hip_roll_joint: limit lower=-0.698 upper=0.698 effort=150.0 velocity=8 -> lower=-0.698 upper=0.698 effort=100 velocity=8
- joint right_hip_yaw_joint: limit lower=-0.698 upper=0.698 effort=120.0 velocity=8 -> lower=-0.698 upper=0.698 effort=80 velocity=8
- joint right_knee_joint: limit lower=-1.5 upper=0 effort=225.0 velocity=8 -> lower=-1.5 upper=0 effort=150 velocity=8; origin xyz=0 0 -0.293459999999997 rpy=0 0 0 -> xyz=0 0 -0.195639999999998 rpy=0 0 0
- joint right_toe_joint: limit lower=-0.349 upper=1.047 effort=45.0 velocity=8 -> lower=-0.349 upper=1.047 effort=30 velocity=8

File: mechanical/urdf/master_assembly.xacro (robot description, xacro)
@@ -2,8 +2,4 @@
 <robot name="RevEx_Full_Assembly" xmlns:xacro="http://wiki.ros.org/xacro">
   <xacro:property name="mesh_dir" value="C:/Projects/RevExBot/RevEx_Phase1_Hardware/mechanical/meshes" />
-  <xacro:property name="leg_scale" value="1.5" />
-  <xacro:property name="leg_inertia_scale" value="${leg_scale * leg_scale}" />
-  <xacro:property name="effort_scale" value="${leg_scale}" />
-  <xacro:property name="pelvis_raise" value="0.24515" />
   <material name="Grey"><color rgba="0.6 0.6 0.6 1.0" /></material>
   <material name="DarkGrey"><color rgba="0.22 0.22 0.22 1.0" /></material>
@@ -13,5 +9,5 @@
     <parent link="base_link" />
     <child link="pelvis_link" />
-    <origin xyz="0 0 ${pelvis_raise}" rpy="0 0 0" />
+    <origin xyz="0 0 0" rpy="0 0 0" />
   </joint>
   <link name="pelvis_link">
@@ -49,6 +45,6 @@
     <parent link="pelvis_link" /><child link="left_hip_pitch_link" />
     <axis xyz="0 1 0" />
-    <limit lower="-2.094" upper="1.047" effort="${120 * effort_scale}" velocity="8" />
-    <dynamics damping="0.095625" friction="0" />
+    <limit lower="-2.094" upper="1.047" effort="120" velocity="8" />
+    <dynamics damping="0.095625" friction="0.15" />
   </joint>
   <link name="left_hip_roll_link">
@@ -65,18 +61,18 @@
     <parent link="left_hip_pitch_link" /><child link="left_hip_roll_link" />
     <axis xyz="1 0 0" />
-    <limit lower="-0.698" upper="0.698" effort="${100 * effort_scale}" velocity="8" />
-    <dynamics damping="0.11" friction="0" />
+    <limit lower="-0.698" upper="0.698" effort="100" velocity="8" />
+    <dynamics damping="0.11" friction="0.15" />
   </joint>
   <link name="left_hip_yaw_link">
     <inertial>
-      <origin xyz="0.00107948196019631 0.00102490074879569 ${-0.120338859084698 * leg_scale}" rpy="0 0 0" />
-      <mass value="${1.86657016436158 * leg_scale}" />
-      <inertia ixx="${0.00341632805787578 * leg_inertia_scale}" ixy="1.12872344062739E-05" ixz="2.89779048114687E-05"
-               iyy="${0.00356015908770306 * leg_inertia_scale}" iyz="-0.000119761895425219" izz="${0.00137524372110325 * leg_scale}" />
-    </inertial>
-    <visual><geometry><mesh filename="${mesh_dir}/LEFT_HIP_YAW.STL" scale="1 1 ${leg_scale}"/></geometry><material name="Grey" /></visual>
+      <origin xyz="0.00107948196019631 0.00102490074879569 -0.120338859084698" rpy="0 0 0" />
+      <mass value="1.86657016436158" />
+      <inertia ixx="0.00341632805787578" ixy="1.12872344062739E-05" ixz="2.89779048114687E-05"
+               iyy="0.00356015908770306" iyz="-0.000119761895425219" izz="0.00137524372110325" />
+    </inertial>
+    <visual><geometry><mesh filename="${mesh_dir}/LEFT_HIP_YAW.STL" /></geometry><material name="Grey" /></visual>
     <collision name="left_hip_yaw_collision">
-      <origin xyz="0 0 ${-0.085 * leg_scale}" rpy="0 0 0" />
-      <geometry><cylinder radius="0.04" length="${0.07 * leg_scale}" /></geometry>
+      <origin xyz="0 0 -0.085" rpy="0 0 0" />
+      <geometry><cylinder radius="0.04" length="0.07" /></geometry>
     </collision>
   </link>
@@ -85,26 +81,26 @@
     <parent link="left_hip_roll_link" /><child link="left_hip_yaw_link" />
     <axis xyz="0 0 -1" />
-    <limit lower="-0.698" upper="0.698" effort="${80 * effort_scale}" velocity="8" />
-    <dynamics damping="0.038" friction="0" />
+    <limit lower="-0.698" upper="0.698" effort="80" velocity="8" />
+    <dynamics damping="0.038" friction="0.15" />
   </joint>
   <link name="left_knee_link">
     <inertial>
-      <origin xyz="-0.000500664455004187 0.000509289489479564 ${-0.11269288769412 * leg_scale}" rpy="0 0 0" />
-      <mass value="${2.39114151033076 * leg_scale}" />
-      <inertia ixx="${0.00962172060189828 * leg_inertia_scale}" ixy="9.87646392241852E-06" ixz="-0.000645140055016828"
-               iyy="${0.00975314356560942 * leg_inertia_scale}" iyz="-7.94058135611557E-06" izz="${0.00233095236940007 * leg_scale}" />
-    </inertial>
-    <visual><geometry><mesh filename="${mesh_dir}/LEFT_KNEE.STL" scale="1 1 ${leg_scale}"/></geometry><material name="Grey" /></visual>
+      <origin xyz="-0.000500664455004187 0.000509289489479564 -0.11269288769412" rpy="0 0 0" />
+      <mass value="2.39114151033076" />
+      <inertia ixx="0.00962172060189828" ixy="9.87646392241852E-06" ixz="-0.000645140055016828"
+               iyy="0.00975314356560942" iyz="-7.94058135611557E-06" izz="0.00233095236940007" />
+    </inertial>
+    <visual><geometry><mesh filename="${mesh_dir}/LEFT_KNEE.STL" /></geometry><material name="Grey" /></visual>
     <collision name="left_knee_collision">
-      <origin xyz="0 0 ${-0.13 * leg_scale}" rpy="0 0 0" />
-      <geometry><cylinder radius="0.04" length="${0.18 * leg_scale}" /></geometry>
+      <origin xyz="0 0 -0.13" rpy="0 0 0" />
+      <geometry><cylinder radius="0.04" length="0.18" /></geometry>
     </collision>
   </link>
   <joint name="left_knee_joint" type="revolute">
-    <origin xyz="0 0 ${-0.195639999999998 * leg_scale}" rpy="0 0 0" />
+    <origin xyz="0 0 -0.195639999999998" rpy="0 0 0" />
     <parent link="left_hip_yaw_link" /><child link="left_knee_link" />
     <axis xyz="0 1 0" />
-    <limit lower="0" upper="1.5" effort="${150 * effort_scale}" velocity="8" />
-    <dynamics damping="0.0339552" friction="0" />
+    <limit lower="0" upper="1.5" effort="150" velocity="8" />
+    <dynamics damping="0.0339552" friction="0.15" />
   </joint>
   <link name="left_ankle_pitch_link">
@@ -118,9 +114,9 @@
   </link>
   <joint name="left_ankle_pitch_joint" type="revolute">
-    <origin xyz="0 0 ${-0.294662336087024 * leg_scale}" rpy="0 0 0" />
+    <origin xyz="0 0 -0.294662336087024" rpy="0 0 0" />
     <parent link="left_knee_link" /><child link="left_ankle_pitch_link" />
     <axis xyz="0 1 0" />
-    <limit lower="-0.35" upper="0.35" effort="${80 * effort_scale}" velocity="8" />
-    <dynamics damping="0.0565056" friction="0" />
+    <limit lower="-0.35" upper="0.35" effort="80" velocity="8" />
+    <dynamics damping="0.0565056" friction="0.15" />
   </joint>
   <link name="left_ankle_roll_link">
@@ -137,6 +133,6 @@
     <parent link="left_ankle_pitch_link" /><child link="left_ankle_roll_link" />
     <axis xyz="-1 0 0" />
-    <limit lower="-0.1" upper="0.1" effort="${50 * effort_scale}" velocity="8" />
-    <dynamics damping="0.0565056" friction="0" />
+    <limit lower="-0.1" upper="0.1" effort="50" velocity="8" />
+    <dynamics damping="0.0565056" friction="0.15" />
   </joint>
   <link name="left_toe_link">
@@ -156,5 +152,5 @@
     <parent link="left_ankle_roll_link" /><child link="left_toe_link" />
     <axis xyz="0.010532 0.99994 0" />
-    <limit lower="-1.047" upper="0.349" effort="${30 * effort_scale}" velocity="8" />
+    <limit lower="-1.047" upper="0.349" effort="30" velocity="8" />
     <dynamics damping="0.001" friction="0.02" />
   </joint>
@@ -176,6 +172,6 @@
     <parent link="pelvis_link" /><child link="right_hip_pitch_link" />
     <axis xyz="0 -1 0" />
-    <limit lower="-1.047" upper="2.094" effort="${120 * effort_scale}" velocity="8" />
-    <dynamics damping="0.095625" friction="0" />
+    <limit lower="-1.047" upper="2.094" effort="120" velocity="8" />
+    <dynamics damping="0.095625" friction="0.15" />
   </joint>
   <link name="right_hip_roll_link">
@@ -192,18 +188,18 @@
     <parent link="right_hip_pitch_link" /><child link="right_hip_roll_link" />
     <axis xyz="1 0 0" />
-    <limit lower="-0.698" upper="0.698" effort="${100 * effort_scale}" velocity="8" />
-    <dynamics damping="0.11" friction="0" />
+    <limit lower="-0.698" upper="0.698" effort="100" velocity="8" />
+    <dynamics damping="0.11" friction="0.15" />
   </joint>
   <link name="right_hip_yaw_link">
     <inertial>
-      <origin xyz="0.0010759524804974 -0.00102176499629938 ${-0.120345116027848 * leg_scale}" rpy="0 0 0" />
-      <mass value="${1.86647220449567 * leg_scale}" />
-      <inertia ixx="${0.00341588734528233 * leg_inertia_scale}" ixy="-1.17597783272228E-05" ixz="2.91733595327906E-05"
-               iyy="${0.00355990015451682 * leg_inertia_scale}" iyz="0.00011971567133214" izz="${0.00137525272174267 * leg_scale}" />
-    </inertial>
-    <visual><geometry><mesh filename="${mesh_dir}/RIGHT_HIP_YAW.STL" scale="1 1 ${leg_scale}"/></geometry><material name="Grey" /></visual>
+      <origin xyz="0.0010759524804974 -0.00102176499629938 -0.120345116027848" rpy="0 0 0" />
+      <mass value="1.86647220449567" />
+      <inertia ixx="0.00341588734528233" ixy="-1.17597783272228E-05" ixz="2.91733595327906E-05"
+               iyy="0.00355990015451682" iyz="0.00011971567133214" izz="0.00137525272174267" />
+    </inertial>
+    <visual><geometry><mesh filename="${mesh_dir}/RIGHT_HIP_YAW.STL" /></geometry><material name="Grey" /></visual>
     <collision name="right_hip_yaw_collision">
-      <origin xyz="0 0 ${-0.085 * leg_scale}" rpy="0 0 0" />
-      <geometry><cylinder radius="0.04" length="${0.07 * leg_scale}" /></geometry>
+      <origin xyz="0 0 -0.085" rpy="0 0 0" />
+      <geometry><cylinder radius="0.04" length="0.07" /></geometry>
     </collision>
   </link>
@@ -212,26 +208,26 @@
     <parent link="right_hip_roll_link" /><child link="right_hip_yaw_link" />
     <axis xyz="0 0 -1" />
-    <limit lower="-0.698" upper="0.698" effort="${80 * effort_scale}" velocity="8" />
-    <dynamics damping="0.038" friction="0" />
+    <limit lower="-0.698" upper="0.698" effort="80" velocity="8" />
+    <dynamics damping="0.038" friction="0.15" />
   </joint>
   <link name="right_knee_link">
     <inertial>
-      <origin xyz="-0.000497587233719177 -0.000414757224949908 ${-0.112692693562372 * leg_scale}" rpy="0 0 0" />
-      <mass value="${2.39110172735043 * leg_scale}" />
-      <inertia ixx="${0.00962148213806552 * leg_inertia_scale}" ixy="-9.87527823922245E-06" ixz="-0.00064509471825313"
-               iyy="${0.00975287238047396 * leg_inertia_scale}" iyz="7.98431367388265E-06" izz="${0.0023309035826248 * leg_scale}" />
-    </inertial>
-    <visual><geometry><mesh filename="${mesh_dir}/RIGHT_KNEE.STL" scale="1 1 ${leg_scale}"/></geometry><material name="Grey" /></visual>
+      <origin xyz="-0.000497587233719177 -0.000414757224949908 -0.112692693562372" rpy="0 0 0" />
+      <mass value="2.39110172735043" />
+      <inertia ixx="0.00962148213806552" ixy="-9.87527823922245E-06" ixz="-0.00064509471825313"
+               iyy="0.00975287238047396" iyz="7.98431367388265E-06" izz="0.0023309035826248" />
+    </inertial>
+    <visual><geometry><mesh filename="${mesh_dir}/RIGHT_KNEE.STL" /></geometry><material name="Grey" /></visual>
     <collision name="right_knee_collision">
-      <origin xyz="0 0 ${-0.13 * leg_scale}" rpy="0 0 0" />
-      <geometry><cylinder radius="0.04" length="${0.18 * leg_scale}" /></geometry>
+      <origin xyz="0 0 -0.13" rpy="0 0 0" />
+      <geometry><cylinder radius="0.04" length="0.18" /></geometry>
     </collision>
   </link>
   <joint name="right_knee_joint" type="revolute">
-    <origin xyz="0 0 ${-0.195639999999998 * leg_scale}" rpy="0 0 0" />
+    <origin xyz="0 0 -0.195639999999998" rpy="0 0 0" />
     <parent link="right_hip_yaw_link" /><child link="right_knee_link" />
     <axis xyz="0 -1 0" />
-    <limit lower="-1.5" upper="0" effort="${150 * effort_scale}" velocity="8" />
-    <dynamics damping="0.0339552" friction="0" />
+    <limit lower="-1.5" upper="0" effort="150" velocity="8" />
+    <dynamics damping="0.0339552" friction="0.15" />
   </joint>
   <link name="right_ankle_pitch_link">
@@ -245,9 +241,9 @@
   </link>
   <joint name="right_ankle_pitch_joint" type="revolute">
-    <origin xyz="0 0.0001 ${-0.294662336087023 * leg_scale}" rpy="0 0 0" />
+    <origin xyz="0 0.0001 -0.294662336087023" rpy="0 0 0" />
     <parent link="right_knee_link" /><child link="right_ankle_pitch_link" />
     <axis xyz="0 -1 0" />
-    <limit lower="-0.35" upper="0.35" effort="${80 * effort_scale}" velocity="8" />
-    <dynamics damping="0.0565056" friction="0" />
+    <limit lower="-0.35" upper="0.35" effort="80" velocity="8" />
+    <dynamics damping="0.0565056" friction="0.15" />
   </joint>
   <link name="right_ankle_roll_link">
@@ -264,6 +260,6 @@
     <parent link="right_ankle_pitch_link" /><child link="right_ankle_roll_link" />
     <axis xyz="-1 0 0" />
-    <limit lower="-0.1" upper="0.1" effort="${50 * effort_scale}" velocity="8" />
-    <dynamics damping="0.0565056" friction="0" />
+    <limit lower="-0.1" upper="0.1" effort="50" velocity="8" />
+    <dynamics damping="0.0565056" friction="0.15" />
   </joint>
   <link name="right_toe_link">
@@ -283,5 +279,5 @@
     <parent link="right_ankle_roll_link" /><child link="right_toe_link" />
     <axis xyz="0.0074685 -0.99997 0" />
-    <limit lower="-0.349" upper="1.047" effort="${30 * effort_scale}" velocity="8" />
+    <limit lower="-0.349" upper="1.047" effort="30" velocity="8" />
     <dynamics damping="0.001" friction="0.02" />
   </joint>
@@ -304,5 +300,5 @@
     <axis xyz="0 0 1" />
     <limit lower="-1.047" upper="1.047" effort="150" velocity="5" />
-    <dynamics damping="0.095625" friction="0" />
+    <dynamics damping="0.095625" friction="0.15" />
   </joint>
   <link name="neck_yaw_link">
@@ -324,5 +320,5 @@
     <axis xyz="0 0 1" />
     <limit lower="-1.571" upper="1.571" effort="20" velocity="5" />
-    <dynamics damping="0.0565" friction="0" />
+    <dynamics damping="0.0565" friction="0.08" />
   </joint>
   <link name="head_link">
@@ -334,5 +330,5 @@
     <visual>
       <origin xyz="0 0 0" rpy="0 0 0" />
-      <geometry><mesh filename="${mesh_dir}/HEAD.STL" /></geometry>
+      <geometry><mesh filename="${mesh_dir}/head.stl" /></geometry>
       <material name="LightGrey" />
     </visual>
@@ -348,5 +344,5 @@
     <axis xyz="0 1 0" />
     <limit lower="-0.5" upper="0.5" effort="20" velocity="5" />
-    <dynamics damping="0.0565" friction="0" />
+    <dynamics damping="0.0565" friction="0.08" />
   </joint>
   <link name="left_eye_camera_link" />
@@ -388,5 +384,5 @@
     <axis xyz="0 -1 0" />
     <limit lower="-0.872" upper="3.141" effort="80" velocity="6" />
-    <dynamics damping="0.11" friction="0" />
+    <dynamics damping="0.11" friction="0.08" />
   </joint>
   <link name="right_shoulder_roll_link">
@@ -409,5 +405,5 @@
     <axis xyz="-1 0 0" />
     <limit lower="0" upper="1.571" effort="80" velocity="6" />
-    <dynamics damping="0.0339552" friction="0" />
+    <dynamics damping="0.0339552" friction="0.08" />
   </joint>
   <link name="right_shoulder_yaw_link">
@@ -425,5 +421,5 @@
     <axis xyz="0 0 -1" />
     <limit lower="-1.571" upper="1.571" effort="60" velocity="6" />
-    <dynamics damping="0.038" friction="0" />
+    <dynamics damping="0.038" friction="0.08" />
   </joint>
   <link name="right_elbow_link">
@@ -445,5 +441,5 @@
     <axis xyz="0 1 0" />
     <limit lower="-2.443" upper="0" effort="60" velocity="6" />
-    <dynamics damping="0.0282528" friction="0" />
+    <dynamics damping="0.0282528" friction="0.08" />
   </joint>
   <link name="left_shoulder_pitch_link">
@@ -461,5 +457,5 @@
     <axis xyz="0 1 0" />
     <limit lower="-3.141" upper="0.872" effort="80" velocity="6" />
-    <dynamics damping="0.11" friction="0" />
+    <dynamics damping="0.11" friction="0.08" />
   </joint>
   <link name="left_shoulder_roll_link">
@@ -482,5 +478,5 @@
     <axis xyz="-1 0 0" />
     <limit lower="-1.571" upper="0" effort="80" velocity="6" />
-    <dynamics damping="0.0339552" friction="0" />
+    <dynamics damping="0.0339552" friction="0.08" />
   </joint>
   <link name="left_shoulder_yaw_link">
@@ -498,5 +494,5 @@
     <axis xyz="0 0 -1" />
     <limit lower="-1.571" upper="1.571" effort="60" velocity="6" />
-    <dynamics damping="0.038" friction="0" />
+    <dynamics damping="0.038" friction="0.08" />
   </joint>
   <link name="left_elbow_link">
@@ -518,12 +514,12 @@
     <axis xyz="0 -1 0" />
     <limit lower="0" upper="2.443" effort="60" velocity="6" />
-    <dynamics damping="0.0282528" friction="0" />
+    <dynamics damping="0.0282528" friction="0.08" />
   </joint>
   <xacro:include filename="shadow_hand.xacro" />
-  <xacro:shadow_hand
+<xacro:shadow_hand
       prefix="rh_"
       mesh_dir="${mesh_dir}"
-      forearm_visual_xyz="0.107504 0.162107 -0.113857"
-      wrist_xyz="-0.013287 0 -0.248456"
+      forearm_visual_xyz="0.0 0.0 0.0"
+      wrist_xyz="-0.013352 -0.000739 -0.189317"
       wrist_rpy="3.14159 0.1396263 0"
       mirror="false" />
@@ -536,6 +532,6 @@
       prefix="lh_"
       mesh_dir="${mesh_dir}"
-      forearm_visual_xyz="0.107504 -0.162107 -0.113857"
-      wrist_xyz="-0.013287 0 -0.248456"
+      forearm_visual_xyz="0.0 0.0 0.0"
+      wrist_xyz="-0.013352 0.000739 -0.189317"
       wrist_rpy="3.14159 -0.1396263 3.14159"
       mirror="true" />
