Commit message: Re-scaled down. Fixed and finalized the complete orientation

File: mechanical/urdf/shadow_hand.xacro (robot description, xacro)
@@ -2,6 +2,10 @@
 <robot xmlns:xacro="http://wiki.ros.org/xacro" name="shadow_hand">
     <xacro:macro name="shadow_hand" params="prefix mesh_dir wrist_xyz wrist_rpy forearm_visual_xyz mirror:=false">
+        <!-- Mirroring helpers -->
         <xacro:property name="f_x" value="${-1 if mirror else 1}" />
         <xacro:property name="ab_x" value="${1 if mirror else -1}" />
+        <!-- ================================================================ -->
+        <!-- FOREARM                                                         -->
+        <!-- ================================================================ -->
         <link name="${prefix}forearm">
             <inertial>
@@ -12,5 +16,5 @@
             <visual>
                 <origin rpy="0 0 0" xyz="${forearm_visual_xyz}" />
-                <geometry name="${prefix}forearm_visual">
+                <geometry>
                     <mesh filename="${mesh_dir}/${prefix}forearm.stl" />
                 </geometry>
@@ -21,5 +25,5 @@
             <collision>
                 <origin rpy="0 0 0" xyz="${forearm_visual_xyz}" />
-                <geometry name="${prefix}forearm_collision">
+                <geometry>
                     <mesh filename="${mesh_dir}/${prefix}forearm.stl" />
                 </geometry>
@@ -32,4 +36,7 @@
             </collision>
         </link>
+        <!-- ================================================================ -->
+        <!-- WRIST                                                           -->
+        <!-- ================================================================ -->
         <link name="${prefix}wrist">
             <inertial>
@@ -84,4 +91,7 @@
             <dynamics damping="0.1" />
         </joint>
+        <!-- ================================================================ -->
+        <!-- PALM                                                            -->
+        <!-- ================================================================ -->
         <link name="${prefix}palm">
             <inertial>
@@ -150,4 +160,7 @@
             <origin rpy="${-1.5707963 * f_x} 3.141592 0.0" xyz="${0.01785 * f_x} 0.00765 0.049125" />
         </joint>
+        <!-- ================================================================ -->
+        <!-- INDEX FINGER (FF)                                                -->
+        <!-- ================================================================ -->
         <link name="${prefix}ffknuckle">
             <inertial><origin rpy="0 0 0" xyz="0 0 0" /><mass value="0.008" /><inertia ixx="0.00000026" ixy="0.0" ixz="0.0" iyy="0.00000026" iyz="0.0" izz="0.00000032" /></inertial>
@@ -186,7 +199,10 @@
         </joint>
         <link name="${prefix}ffdistal">
-            <inertial><mass value="0.012" /><origin xyz="0 0 0.012" /><inertia ixx="0.00000094" ixy="0.0" ixz="0.0" iyy="0.000011" iyz="0.0" izz="0.00000053" /></inertial>
+            <inertial><mass value="0.012" /><origin xyz="0 0 0.012" /><inertia ixx="0.00000094" ixy="0.0" ixz="0.0" iyy="0.0000011" iyz="0.0" izz="0.00000053" /></inertial>
             <visual><origin rpy="0 0 0" xyz="0 0 0" /><geometry><mesh filename="${mesh_dir}/${prefix}f_distal_pst.stl" /></geometry></visual>
-            <collision><origin rpy="0 0 0" xyz="0 0 0" /><geometry><mesh filename="${mesh_dir}/${prefix}f_distal_pst.stl" /></geometry></collision>
+            <collision>
+                <origin rpy="0 0 0" xyz="0 0 0.012" />
+                <geometry><box size="0.015 0.015 0.024" /></geometry>
+            </collision>
         </link>
         <joint name="${prefix}FFJ1" type="revolute">
@@ -198,4 +214,7 @@
         <link name="${prefix}fftip"><inertial><mass value="0.001" /><inertia ixx="0.00001" ixy="0.0" ixz="0.0" iyy="0.00001" iyz="0.0" izz="0.00001" /></inertial></link>
         <joint name="${prefix}FFtip" type="fixed"><parent link="${prefix}ffdistal" /><child link="${prefix}fftip" /><origin rpy="0 0 0" xyz="0 0 0.026" /></joint>
+        <!-- ================================================================ -->
+        <!-- MIDDLE FINGER (MF)                                               -->
+        <!-- ================================================================ -->
         <link name="${prefix}mfknuckle">
             <inertial><origin rpy="0 0 0" xyz="0 0 0" /><mass value="0.008" /><inertia ixx="0.00000026" ixy="0.0" ixz="0.0" iyy="0.00000026" iyz="0.0" izz="0.00000032" /></inertial>
@@ -236,5 +255,8 @@
             <inertial><mass value="0.012" /><origin xyz="0 0 0.012" /><inertia ixx="0.00000094" ixy="0.0" ixz="0.0" iyy="0.0000011" iyz="0.0" izz="0.00000053" /></inertial>
             <visual><origin rpy="0 0 0" xyz="0 0 0" /><geometry><mesh filename="${mesh_dir}/${prefix}f_distal_pst.stl" /></geometry></visual>
-            <collision><origin rpy="0 0 0" xyz="0 0 0" /><geometry><mesh filename="${mesh_dir}/${prefix}f_distal_pst.stl" /></geometry></collision>
+            <collision>
+                <origin rpy="0 0 0" xyz="0 0 0.012" />
+                <geometry><box size="0.015 0.015 0.024" /></geometry>
+            </collision>
         </link>
         <joint name="${prefix}MFJ1" type="revolute">
@@ -246,4 +268,7 @@
         <link name="${prefix}mftip"><inertial><mass value="0.001" /><inertia ixx="0.00001" ixy="0.0" ixz="0.0" iyy="0.00001" iyz="0.0" izz="0.00001" /></inertial></link>
         <joint name="${prefix}MFtip" type="fixed"><parent link="${prefix}mfdistal" /><child link="${prefix}mftip" /><origin rpy="0 0 0" xyz="0 0 0.026" /></joint>
+        <!-- ================================================================ -->
+        <!-- RING FINGER (RF)                                                 -->
+        <!-- ================================================================ -->
         <link name="${prefix}rfknuckle">
             <inertial><origin rpy="0 0 0" xyz="0 0 0" /><mass value="0.008" /><inertia ixx="0.00000026" ixy="0.0" ixz="0.0" iyy="0.00000026" iyz="0.0" izz="0.00000032" /></inertial>
@@ -284,5 +309,8 @@
             <inertial><mass value="0.012" /><origin xyz="0 0 0.012" /><inertia ixx="0.00000094" ixy="0.0" ixz="0.0" iyy="0.0000011" iyz="0.0" izz="0.00000053" /></inertial>
             <visual><origin rpy="0 0 0" xyz="0 0 0" /><geometry><mesh filename="${mesh_dir}/${prefix}f_distal_pst.stl" /></geometry></visual>
-            <collision><origin rpy="0 0 0" xyz="0 0 0" /><geometry><mesh filename="${mesh_dir}/${prefix}f_distal_pst.stl" /></geometry></collision>
+            <collision>
+                <origin rpy="0 0 0" xyz="0 0 0.012" />
+                <geometry><box size="0.015 0.015 0.024" /></geometry>
+            </collision>
         </link>
         <joint name="${prefix}RFJ1" type="revolute">
@@ -294,4 +322,7 @@
         <link name="${prefix}rftip"><inertial><mass value="0.001" /><inertia ixx="0.00001" ixy="0.0" ixz="0.0" iyy="0.00001" iyz="0.0" izz="0.00001" /></inertial></link>
         <joint name="${prefix}RFtip" type="fixed"><parent link="${prefix}rfdistal" /><child link="${prefix}rftip" /><origin rpy="0 0 0" xyz="0 0 0.026" /></joint>
+        <!-- ================================================================ -->
+        <!-- LITTLE FINGER (LF) – duplicate lfknuckle removed                 -->
+        <!-- ================================================================ -->
         <link name="${prefix}lfmetacarpal">
             <inertial>
@@ -322,4 +353,5 @@
             <dynamics damping="0.1" />
         </joint>
+        <!-- Only one lfknuckle definition (kept here) -->
         <link name="${prefix}lfknuckle">
             <inertial>
@@ -377,5 +409,8 @@
             <inertial><mass value="0.012" /><origin xyz="0 0 0.012" /><inertia ixx="0.00000094" ixy="0.0" ixz="0.0" iyy="0.0000011" iyz="0.0" izz="0.00000053" /></inertial>
             <visual><origin rpy="0 0 0" xyz="0 0 0" /><geometry><mesh filename="${mesh_dir}/${prefix}f_distal_pst.stl" /></geometry></visual>
-            <collision><origin rpy="0 0 0" xyz="0 0 0" /><geometry><mesh filename="${mesh_dir}/${prefix}f_distal_pst.stl" /></geometry></collision>
+            <collision>
+                <origin rpy="0 0 0" xyz="0 0 0.012" />
+                <geometry><box size="0.015 0.015 0.024" /></geometry>
+            </collision>
         </link>
         <joint name="${prefix}LFJ1" type="revolute">
@@ -387,4 +422,7 @@
         <link name="${prefix}lftip"><inertial><mass value="0.001" /><inertia ixx="0.00001" ixy="0.0" ixz="0.0" iyy="0.00001" iyz="0.0" izz="0.00001" /></inertial></link>
         <joint name="${prefix}LFtip" type="fixed"><parent link="${prefix}lfdistal" /><child link="${prefix}lftip" /><origin rpy="0 0 0" xyz="0 0 0.026" /></joint>
+        <!-- ================================================================ -->
+        <!-- THUMB                                                           -->
+        <!-- ================================================================ -->
         <link name="${prefix}thbase">
             <inertial><mass value="0.010" /><origin rpy="0 0 0" xyz="0 0 0" /><inertia ixx="0.00000016" ixy="0.0" ixz="0.0" iyy="0.00000016" iyz="0.0" izz="0.00000016" /></inertial>
@@ -428,4 +466,5 @@
             <collision><origin rpy="0 0 0" xyz="0 0 0.012" /><geometry><cylinder length="0.018" radius="0.011" /></geometry></collision>
             <collision><origin rpy="0 0 0" xyz="0 0 0.019" /><geometry><sphere radius="0.011" /></geometry></collision>
+            <!-- Mirrored cylinder orientation -->
             <collision>
                 <origin rpy="0 ${1.5708 * f_x} 0" xyz="0 0 0.032" />
@@ -442,5 +481,8 @@
             <inertial><mass value="0.016" /><origin rpy="0 0 0" xyz="0 0 0.01375" /><inertia ixx="0.0000021" ixy="0.0" ixz="0.0" iyy="0.0000022" iyz="0.0" izz="0.000001" /></inertial>
             <visual><origin rpy="0 0 0" xyz="0 0 0" /><geometry><mesh filename="${mesh_dir}/${prefix}th_distal_pst.stl" /></geometry><material name="shadow_thmiddle_material"><color rgba="0.2 0.2 0.2 1.0" /></material></visual>
-            <collision><origin rpy="0 0 0" xyz="0 0 0" /><geometry><mesh filename="${mesh_dir}/${prefix}th_distal_pst.stl" /></geometry></collision>
+            <collision>
+                <origin rpy="0 0 0" xyz="0 0 0.01375" />
+                <geometry><box size="0.018 0.018 0.028" /></geometry>
+            </collision>
         </link>
         <joint name="${prefix}THJ1" type="revolute">
