Commit message: Updated weights and maths in the xacro blueprints

File: assets/urdf/revexbot1.urdf (robot description, URDF)
Before this commit: robot RevEx_Full_Assembly, 62 links, 61 joints
Links:
- link lh_index_dp: mass 0.004 -> 0.02
- link lh_index_mp: mass 0.006 -> 0.02
- link lh_index_pp: mass 0.008 -> 0.02
- link lh_middle_dp: mass 0.004 -> 0.02
- link lh_middle_mp: mass 0.006 -> 0.02
- link lh_middle_pp: mass 0.008 -> 0.02
- link lh_pinky_dp: mass 0.004 -> 0.02
- link lh_pinky_mp: mass 0.006 -> 0.02
- link lh_pinky_pp: mass 0.008 -> 0.02
- link lh_ring_dp: mass 0.004 -> 0.02
- link lh_ring_mp: mass 0.006 -> 0.02
- link lh_ring_pp: mass 0.008 -> 0.02
- link lh_thumb_base: mass 0.012 -> 0.02
- link lh_thumb_dp: mass 0.005 -> 0.02
- link lh_thumb_mp: mass 0.008 -> 0.02
- link lh_thumb_pp: mass 0.01 -> 0.02
- link rh_index_dp: mass 0.004 -> 0.02
- link rh_index_mp: mass 0.006 -> 0.02
- link rh_index_pp: mass 0.008 -> 0.02
- link rh_middle_dp: mass 0.004 -> 0.02
- link rh_middle_mp: mass 0.006 -> 0.02
- link rh_middle_pp: mass 0.008 -> 0.02
- link rh_pinky_dp: mass 0.004 -> 0.02
- link rh_pinky_mp: mass 0.006 -> 0.02
- link rh_pinky_pp: mass 0.008 -> 0.02
- link rh_ring_dp: mass 0.004 -> 0.02
- link rh_ring_mp: mass 0.006 -> 0.02
- link rh_ring_pp: mass 0.008 -> 0.02
- link rh_thumb_base: mass 0.012 -> 0.02
- link rh_thumb_dp: mass 0.005 -> 0.02
- link rh_thumb_mp: mass 0.008 -> 0.02
- link rh_thumb_pp: mass 0.01 -> 0.02

File: assets/xacro/faive_hand.xacro (robot description, xacro)
@@ -2,14 +2,10 @@
 <robot xmlns:xacro="http://wiki.ros.org/xacro" name="faive_hand">
     <xacro:macro name="faive_hand" params="prefix mesh_dir mirror_factor:=1">
-        <!-- Uniform scaling for the hand -->
         <xacro:property name="s" value="1.0" />
         <xacro:property name="mass_scale" value="${s * s * s}" />
         <xacro:property name="inertia_scale" value="${s * s * s * s * s}" />
-        <!-- Mirror across Y axis (1 = right, -1 = left) -->
         <xacro:property name="f_y" value="${mirror_factor}" />
-        <!-- Offsets (in meters) -->
         <xacro:property name="palm_offset"  value="0.02" />
         <xacro:property name="thumb_offset" value="0.00" />
-        <!-- ==================== PALM ==================== -->
         <link name="${prefix}palm">
             <visual>
@@ -23,16 +19,13 @@
             <inertial>
                 <origin xyz="0 0 0"/>
-                <!-- GAP 4 FIX: Increased mass to 0.3kg for stability -->
                 <mass value="${0.3 * mass_scale}"/>
-                <!-- GAP 2 FIX: Inflated inertia floor -->
                 <inertia ixx="${0.0001 * inertia_scale}" ixy="0" ixz="0" iyy="${0.0001 * inertia_scale}" iyz="0" izz="${0.0001 * inertia_scale}"/>
             </inertial>
         </link>
-        <!-- ==================== THUMB ==================== -->
         <xacro:property name="thumb_shift" value="0.02" />
         <link name="${prefix}thumb_base">
             <visual><origin xyz="${0.02945 * s} ${(-0.06159 * s + thumb_shift) * f_y} ${0.00627 * s}" rpy="0 0 0"/><geometry><mesh filename="${mesh_dir}/${prefix}thumb_base.stl" scale="${s} ${s} ${s}"/></geometry></visual>
             <collision><origin xyz="0 ${thumb_shift * f_y} 0" rpy="0 1.5708 0"/><geometry><cylinder radius="${0.01 * s}" length="${0.02 * s}"/></geometry></collision>
-            <inertial><mass value="${0.012 * mass_scale}"/><inertia ixx="${0.0001 * inertia_scale}" ixy="0" ixz="0" iyy="${0.0001 * inertia_scale}" iyz="0" izz="${0.0001 * inertia_scale}"/></inertial>
+            <inertial><mass value="${0.02 * mass_scale}"/><inertia ixx="${0.0001 * inertia_scale}" ixy="0" ixz="0" iyy="${0.0001 * inertia_scale}" iyz="0" izz="${0.0001 * inertia_scale}"/></inertial>
         </link>
         <joint name="${prefix}thumb_base_joint" type="revolute">
@@ -41,5 +34,4 @@
             <child link="${prefix}thumb_base"/>
             <axis xyz="0.297249628842018 ${-0.700414486434294 * f_y} -0.648893061564281"/>
-            <!-- GAP 1 FIX: Reduced effort to 0.5 Nm -->
             <limit lower="0" upper="2.27" effort="0.5" velocity="8"/>
             <dynamics damping="0.1" friction="0.03" armature="0.001"/>
@@ -48,5 +40,5 @@
             <visual><origin xyz="${0.04371 * s} ${(-0.05927 * s + thumb_shift) * f_y} ${0.01030 * s}" rpy="0 0 0"/><geometry><mesh filename="${mesh_dir}/${prefix}thumb_pp.stl" scale="${s} ${s} ${s}"/></geometry></visual>
             <collision><origin xyz="${-0.01 * s} ${thumb_shift * f_y} 0" rpy="0 1.5708 0"/><geometry><cylinder radius="${0.01 * s}" length="${0.025 * s}"/></geometry></collision>
-            <inertial><mass value="${0.01 * mass_scale}"/><inertia ixx="${0.0001 * inertia_scale}" ixy="0" ixz="0" iyy="${0.0001 * inertia_scale}" iyz="0" izz="${0.0001 * inertia_scale}"/></inertial>
+            <inertial><mass value="${0.02 * mass_scale}"/><inertia ixx="${0.0001 * inertia_scale}" ixy="0" ixz="0" iyy="${0.0001 * inertia_scale}" iyz="0" izz="${0.0001 * inertia_scale}"/></inertial>
         </link>
         <joint name="${prefix}thumb_pp_joint" type="revolute">
@@ -61,5 +53,5 @@
             <visual><origin xyz="${0.09026 * s} ${(-0.04514 * s + thumb_shift) * f_y} ${0.02114 * s}" rpy="0 0 0"/><geometry><mesh filename="${mesh_dir}/${prefix}thumb_mp.stl" scale="${s} ${s} ${s}"/></geometry></visual>
             <collision><origin xyz="${-0.015 * s} ${thumb_shift * f_y} 0" rpy="0 1.5708 0"/><geometry><cylinder radius="${0.01 * s}" length="${0.035 * s}"/></geometry></collision>
-            <inertial><mass value="${0.008 * mass_scale}"/><inertia ixx="${0.0001 * inertia_scale}" ixy="0" ixz="0" iyy="${0.0001 * inertia_scale}" iyz="0" izz="${0.0001 * inertia_scale}"/></inertial>
+            <inertial><mass value="${0.02 * mass_scale}"/><inertia ixx="${0.0001 * inertia_scale}" ixy="0" ixz="0" iyy="${0.0001 * inertia_scale}" iyz="0" izz="${0.0001 * inertia_scale}"/></inertial>
         </link>
         <joint name="${prefix}thumb_mp_joint" type="revolute">
@@ -68,5 +60,4 @@
             <child link="${prefix}thumb_mp"/>
             <axis xyz="0.284429826078874 ${-0.088618171481011 * f_y} -0.954592318070968"/>
-            <!-- GAP 1 FIX: Reduced effort to 0.3 Nm -->
             <limit lower="0" upper="0.96" effort="0.3" velocity="8"/>
             <dynamics damping="0.1" friction="0.03" armature="0.001"/>
@@ -75,5 +66,5 @@
             <visual><origin xyz="${0.12386 * s} ${(-0.03879 * s + thumb_shift) * f_y} ${0.03068 * s}" rpy="0 0 0"/><geometry><mesh filename="${mesh_dir}/${prefix}thumb_dp.stl" scale="${s} ${s} ${s}"/></geometry></visual>
             <collision><origin xyz="${-0.01 * s} ${thumb_shift * f_y} 0" rpy="0 1.5708 0"/><geometry><cylinder radius="${0.01 * s}" length="${0.02 * s}"/></geometry></collision>
-            <inertial><mass value="${0.005 * mass_scale}"/><inertia ixx="${0.0001 * inertia_scale}" ixy="0" ixz="0" iyy="${0.0001 * inertia_scale}" iyz="0" izz="${0.0001 * inertia_scale}"/></inertial>
+            <inertial><mass value="${0.02 * mass_scale}"/><inertia ixx="${0.0001 * inertia_scale}" ixy="0" ixz="0" iyy="${0.0001 * inertia_scale}" iyz="0" izz="${0.0001 * inertia_scale}"/></inertial>
         </link>
         <joint name="${prefix}thumb_dp_joint" type="revolute">
@@ -82,14 +73,12 @@
             <child link="${prefix}thumb_dp"/>
             <axis xyz="0.284429826078874 ${-0.088618171481011 * f_y} -0.954592318070968"/>
-            <!-- GAP 1 FIX: Reduced effort to 0.2 Nm -->
-            <limit lower="0" upper="0.68" effort="0.2" velocity="8"/>
-            <dynamics damping="0.1" friction="0.03" armature="0.001"/>
-        </joint>
-        <!-- ==================== INDEX FINGER ==================== -->
+            <limit lower="0" upper="0.68" effort="0.2" velocity="8"/>
+            <dynamics damping="0.1" friction="0.03" armature="0.001"/>
+        </joint>
         <xacro:property name="index_x_shift" value="0.001825" />
         <link name="${prefix}index_pp">
             <visual><origin xyz="${0.03138 * s + index_x_shift} ${-0.13319 * s * f_y} ${-0.02008 * s}" rpy="0 0 0"/><geometry><mesh filename="${mesh_dir}/${prefix}index_pp.stl" scale="${s} ${s} ${s}"/></geometry></visual>
             <collision><origin xyz="${index_x_shift} ${0.02 * s * f_y} 0" rpy="1.5708 0 0"/><geometry><cylinder radius="${0.01 * s}" length="${0.04 * s}"/></geometry></collision>
-            <inertial><mass value="${0.008 * mass_scale}"/><inertia ixx="${0.0001 * inertia_scale}" ixy="0" ixz="0" iyy="${0.0001 * inertia_scale}" iyz="0" izz="${0.0001 * inertia_scale}"/></inertial>
+            <inertial><mass value="${0.02 * mass_scale}"/><inertia ixx="${0.0001 * inertia_scale}" ixy="0" ixz="0" iyy="${0.0001 * inertia_scale}" iyz="0" izz="${0.0001 * inertia_scale}"/></inertial>
         </link>
         <joint name="${prefix}index_pp_joint" type="revolute">
@@ -104,5 +93,5 @@
             <visual><origin xyz="${0.03631 * s + index_x_shift} ${-0.17559 * s * f_y} ${-0.02523 * s}" rpy="0 0 0"/><geometry><mesh filename="${mesh_dir}/${prefix}index_mp.stl" scale="${s} ${s} ${s}"/></geometry></visual>
             <collision><origin xyz="${index_x_shift} ${0.016 * s * f_y} 0" rpy="1.5708 0 0"/><geometry><cylinder radius="${0.01 * s}" length="${0.032 * s}"/></geometry></collision>
-            <inertial><mass value="${0.006 * mass_scale}"/><inertia ixx="${0.0001 * inertia_scale}" ixy="0" ixz="0" iyy="${0.0001 * inertia_scale}" iyz="0" izz="${0.0001 * inertia_scale}"/></inertial>
+            <inertial><mass value="${0.02 * mass_scale}"/><inertia ixx="${0.0001 * inertia_scale}" ixy="0" ixz="0" iyy="${0.0001 * inertia_scale}" iyz="0" izz="${0.0001 * inertia_scale}"/></inertial>
         </link>
         <joint name="${prefix}index_mp_joint" type="revolute">
@@ -117,5 +106,5 @@
             <visual><origin xyz="${0.04004 * s + index_x_shift} ${-0.20764 * s * f_y} ${-0.02912 * s}" rpy="0 0 0"/><geometry><mesh filename="${mesh_dir}/${prefix}index_dp.stl" scale="${s} ${s} ${s}"/></geometry></visual>
             <collision><origin xyz="${index_x_shift} ${0.01 * s * f_y} 0" rpy="1.5708 0 0"/><geometry><cylinder radius="${0.01 * s}" length="${0.02 * s}"/></geometry></collision>
-            <inertial><mass value="${0.004 * mass_scale}"/><inertia ixx="${0.0001 * inertia_scale}" ixy="0" ixz="0" iyy="${0.0001 * inertia_scale}" iyz="0" izz="${0.0001 * inertia_scale}"/></inertial>
+            <inertial><mass value="${0.02 * mass_scale}"/><inertia ixx="${0.0001 * inertia_scale}" ixy="0" ixz="0" iyy="${0.0001 * inertia_scale}" iyz="0" izz="${0.0001 * inertia_scale}"/></inertial>
         </link>
         <joint name="${prefix}index_dp_joint" type="revolute">
@@ -127,9 +116,8 @@
             <dynamics damping="0.1" friction="0.03" armature="0.001"/>
         </joint>
-        <!-- ==================== MIDDLE FINGER ==================== -->
         <link name="${prefix}middle_pp">
             <visual><origin xyz="${0.00550 * s} ${-0.13548 * s * f_y} ${-0.02188 * s}" rpy="0 0 0"/><geometry><mesh filename="${mesh_dir}/${prefix}middle_pp.stl" scale="${s} ${s} ${s}"/></geometry></visual>
             <collision><origin xyz="0 ${0.02 * s * f_y} 0" rpy="1.5708 0 0"/><geometry><cylinder radius="${0.01 * s}" length="${0.04 * s}"/></geometry></collision>
-            <inertial><mass value="${0.008 * mass_scale}"/><inertia ixx="${0.0001 * inertia_scale}" ixy="0" ixz="0" iyy="${0.0001 * inertia_scale}" iyz="0" izz="${0.0001 * inertia_scale}"/></inertial>
+            <inertial><mass value="${0.02 * mass_scale}"/><inertia ixx="${0.0001 * inertia_scale}" ixy="0" ixz="0" iyy="${0.0001 * inertia_scale}" iyz="0" izz="${0.0001 * inertia_scale}"/></inertial>
         </link>
         <joint name="${prefix}middle_pp_joint" type="revolute">
@@ -144,5 +132,5 @@
             <visual><origin xyz="${0.00550 * s} ${-0.18213 * s * f_y} ${-0.02761 * s}" rpy="0 0 0"/><geometry><mesh filename="${mesh_dir}/${prefix}middle_mp.stl" scale="${s} ${s} ${s}"/></geometry></visual>
             <collision><origin xyz="0 ${0.017 * s * f_y} 0" rpy="1.5708 0 0"/><geometry><cylinder radius="${0.01 * s}" length="${0.034 * s}"/></geometry></collision>
-            <inertial><mass value="${0.006 * mass_scale}"/><inertia ixx="${0.0001 * inertia_scale}" ixy="0" ixz="0" iyy="${0.0001 * inertia_scale}" iyz="0" izz="${0.0001 * inertia_scale}"/></inertial>
+            <inertial><mass value="${0.02 * mass_scale}"/><inertia ixx="${0.0001 * inertia_scale}" ixy="0" ixz="0" iyy="${0.0001 * inertia_scale}" iyz="0" izz="${0.0001 * inertia_scale}"/></inertial>
         </link>
         <joint name="${prefix}middle_mp_joint" type="revolute">
@@ -157,5 +145,5 @@
             <visual><origin xyz="${0.00550 * s} ${-0.21637 * s * f_y} ${-0.03181 * s}" rpy="0 0 0"/><geometry><mesh filename="${mesh_dir}/${prefix}middle_dp.stl" scale="${s} ${s} ${s}"/></geometry></visual>
             <collision><origin xyz="0 ${0.01 * s * f_y} 0" rpy="1.5708 0 0"/><geometry><cylinder radius="${0.01 * s}" length="${0.02 * s}"/></geometry></collision>
-            <inertial><mass value="${0.004 * mass_scale}"/><inertia ixx="${0.0001 * inertia_scale}" ixy="0" ixz="0" iyy="${0.0001 * inertia_scale}" iyz="0" izz="${0.0001 * inertia_scale}"/></inertial>
+            <inertial><mass value="${0.02 * mass_scale}"/><inertia ixx="${0.0001 * inertia_scale}" ixy="0" ixz="0" iyy="${0.0001 * inertia_scale}" iyz="0" izz="${0.0001 * inertia_scale}"/></inertial>
         </link>
         <joint name="${prefix}middle_dp_joint" type="revolute">
@@ -167,10 +155,9 @@
             <dynamics damping="0.1" friction="0.03" armature="0.001"/>
         </joint>
-        <!-- ==================== RING FINGER ==================== -->
         <xacro:property name="ring_x_shift" value="-0.001825" />
         <link name="${prefix}ring_pp">
             <visual><origin xyz="${-0.02015 * s + ring_x_shift} ${-0.13023 * s * f_y} ${-0.02037 * s}" rpy="0 0 0"/><geometry><mesh filename="${mesh_dir}/${prefix}ring_pp.stl" scale="${s} ${s} ${s}"/></geometry></visual>
             <collision><origin xyz="${ring_x_shift} ${0.02 * s * f_y} 0" rpy="1.5708 0 0"/><geometry><cylinder radius="${0.01 * s}" length="${0.04 * s}"/></geometry></collision>
-            <inertial><mass value="${0.008 * mass_scale}"/><inertia ixx="${0.0001 * inertia_scale}" ixy="0" ixz="0" iyy="${0.0001 * inertia_scale}" iyz="0" izz="${0.0001 * inertia_scale}"/></inertial>
+            <inertial><mass value="${0.02 * mass_scale}"/><inertia ixx="${0.0001 * inertia_scale}" ixy="0" ixz="0" iyy="${0.0001 * inertia_scale}" iyz="0" izz="${0.0001 * inertia_scale}"/></inertial>
         </link>
         <joint name="${prefix}ring_pp_joint" type="revolute">
@@ -185,5 +172,5 @@
             <visual><origin xyz="${-0.02508 * s + ring_x_shift} ${-0.17263 * s * f_y} ${-0.02552 * s}" rpy="0 0 0"/><geometry><mesh filename="${mesh_dir}/${prefix}ring_mp.stl" scale="${s} ${s} ${s}"/></geometry></visual>
             <collision><origin xyz="${ring_x_shift} ${0.016 * s * f_y} 0" rpy="1.5708 0 0"/><geometry><cylinder radius="${0.01 * s}" length="${0.032 * s}"/></geometry></collision>
-            <inertial><mass value="${0.006 * mass_scale}"/><inertia ixx="${0.0001 * inertia_scale}" ixy="0" ixz="0" iyy="${0.0001 * inertia_scale}" iyz="0" izz="${0.0001 * inertia_scale}"/></inertial>
+            <inertial><mass value="${0.02 * mass_scale}"/><inertia ixx="${0.0001 * inertia_scale}" ixy="0" ixz="0" iyy="${0.0001 * inertia_scale}" iyz="0" izz="${0.0001 * inertia_scale}"/></inertial>
         </link>
         <joint name="${prefix}ring_mp_joint" type="revolute">
@@ -198,5 +185,5 @@
             <visual><origin xyz="${-0.02881 * s + ring_x_shift} ${-0.20468 * s * f_y} ${-0.02941 * s}" rpy="0 0 0"/><geometry><mesh filename="${mesh_dir}/${prefix}ring_dp.stl" scale="${s} ${s} ${s}"/></geometry></visual>
             <collision><origin xyz="${ring_x_shift} ${0.01 * s * f_y} 0" rpy="1.5708 0 0"/><geometry><cylinder radius="${0.01 * s}" length="${0.02 * s}"/></geometry></collision>
-            <inertial><mass value="${0.004 * mass_scale}"/><inertia ixx="${0.0001 * inertia_scale}" ixy="0" ixz="0" iyy="${0.0001 * inertia_scale}" iyz="0" izz="${0.0001 * inertia_scale}"/></inertial>
+            <inertial><mass value="${0.02 * mass_scale}"/><inertia ixx="${0.0001 * inertia_scale}" ixy="0" ixz="0" iyy="${0.0001 * inertia_scale}" iyz="0" izz="${0.0001 * inertia_scale}"/></inertial>
         </link>
         <joint name="${prefix}ring_dp_joint" type="revolute">
@@ -208,10 +195,9 @@
             <dynamics damping="0.1" friction="0.03" armature="0.001"/>
         </joint>
-        <!-- ==================== PINKY FINGER ==================== -->
         <xacro:property name="pinky_x_shift" value="-0.0044225" />
         <link name="${prefix}pinky_pp">
             <visual><origin xyz="${-0.04565 * s + pinky_x_shift} ${-0.11920 * s * f_y} ${-0.01504 * s}" rpy="0 0 0"/><geometry><mesh filename="${mesh_dir}/${prefix}pinky_pp.stl" scale="${s} ${s} ${s}"/></geometry></visual>
             <collision><origin xyz="${pinky_x_shift} ${0.018 * s * f_y} 0" rpy="1.5708 0 0"/><geometry><cylinder radius="${0.01 * s}" length="${0.037 * s}"/></geometry></collision>
-            <inertial><mass value="${0.008 * mass_scale}"/><inertia ixx="${0.0001 * inertia_scale}" ixy="0" ixz="0" iyy="${0.0001 * inertia_scale}" iyz="0" izz="${0.0001 * inertia_scale}"/></inertial>
+            <inertial><mass value="${0.02 * mass_scale}"/><inertia ixx="${0.0001 * inertia_scale}" ixy="0" ixz="0" iyy="${0.0001 * inertia_scale}" iyz="0" izz="${0.0001 * inertia_scale}"/></inertial>
         </link>
         <joint name="${prefix}pinky_pp_joint" type="revolute">
@@ -226,5 +212,5 @@
             <visual><origin xyz="${-0.05536 * s + pinky_x_shift} ${-0.15676 * s * f_y} ${-0.01904 * s}" rpy="0 0 0"/><geometry><mesh filename="${mesh_dir}/${prefix}pinky_mp.stl" scale="${s} ${s} ${s}"/></geometry></visual>
             <collision><origin xyz="${pinky_x_shift} ${0.013 * s * f_y} 0" rpy="1.5708 0 0"/><geometry><cylinder radius="${0.01 * s}" length="${0.027 * s}"/></geometry></collision>
-            <inertial><mass value="${0.006 * mass_scale}"/><inertia ixx="${0.0001 * inertia_scale}" ixy="0" ixz="0" iyy="${0.0001 * inertia_scale}" iyz="0" izz="${0.0001 * inertia_scale}"/></inertial>
+            <inertial><mass value="${0.02 * mass_scale}"/><inertia ixx="${0.0001 * inertia_scale}" ixy="0" ixz="0" iyy="${0.0001 * inertia_scale}" iyz="0" izz="${0.0001 * inertia_scale}"/></inertial>
         </link>
         <joint name="${prefix}pinky_mp_joint" type="revolute">
@@ -239,5 +225,5 @@
             <visual><origin xyz="${-0.06245 * s + pinky_x_shift} ${-0.18421 * s * f_y} ${-0.02196 * s}" rpy="0 0 0"/><geometry><mesh filename="${mesh_dir}/${prefix}pinky_dp.stl" scale="${s} ${s} ${s}"/></geometry></visual>
             <collision><origin xyz="${pinky_x_shift} ${0.01 * s * f_y} 0" rpy="1.5708 0 0"/><geometry><cylinder radius="${0.01 * s}" length="${0.02 * s}"/></geometry></collision>
-            <inertial><mass value="${0.004 * mass_scale}"/><inertia ixx="${0.0001 * inertia_scale}" ixy="0" ixz="0" iyy="${0.0001 * inertia_scale}" iyz="0" izz="${0.0001 * inertia_scale}"/></inertial>
+            <inertial><mass value="${0.02 * mass_scale}"/><inertia ixx="${0.0001 * inertia_scale}" ixy="0" ixz="0" iyy="${0.0001 * inertia_scale}" iyz="0" izz="${0.0001 * inertia_scale}"/></inertial>
         </link>
         <joint name="${prefix}pinky_dp_joint" type="revolute">
