Commit message: Hand changed.

File: assets/urdf/revexbot1.urdf (robot description, URDF)
Before this commit: robot RevEx_Full_Assembly, 62 links, 61 joints
Links:
- removed link lh_index_dp
- removed link lh_index_mp
- removed link lh_index_pp
- removed link lh_middle_dp
- removed link lh_middle_mp
- removed link lh_middle_pp
- removed link lh_palm
- removed link lh_pinky_dp
- removed link lh_pinky_mp
- removed link lh_pinky_pp
- removed link lh_ring_dp
- removed link lh_ring_mp
- removed link lh_ring_pp
- removed link lh_thumb_base
- removed link lh_thumb_dp
- removed link lh_thumb_mp
- removed link lh_thumb_pp
- removed link rh_index_dp
- removed link rh_index_mp
- removed link rh_index_pp
- removed link rh_middle_dp
- removed link rh_middle_mp
- removed link rh_middle_pp
- removed link rh_palm
- removed link rh_pinky_dp
- removed link rh_pinky_mp
- removed link rh_pinky_pp
- removed link rh_ring_dp
- removed link rh_ring_mp
- removed link rh_ring_pp
- removed link rh_thumb_base
- removed link rh_thumb_dp
- removed link rh_thumb_mp
- removed link rh_thumb_pp
- added link lh_ee_index_link
- added link lh_ee_little_link
- added link lh_ee_middle_link
- added link lh_ee_ring_link
- added link lh_ee_thumb_link
- added link lh_hand_palm, mass 0.09; collision mesh filename=../meshes/F03_AL_palm.stl scale=0.001 0.001 0.001; visual mesh filename=../meshes/F03_AL_palm.stl scale=0.001 0.001 0.001
- added link lh_index_DIP, mass 0.0025; collision box size=0.01 0.01 0.02; visual mesh filename=../meshes/F03_AL_link_DIP.stl scale=0.001 0.001 0.001
- added link lh_index_MCP, mass 0.0125; collision box size=0.015 0.015 0.035; visual mesh filename=../meshes/F03_AL_link_MCP.stl scale=0.001 0.001 0.001
- added link lh_index_PIP, mass 0.0125; collision box size=0.012 0.012 0.025; visual mesh filename=../meshes/F03_AL_link_PIP.stl scale=0.001 0.001 0.001
- added link lh_knuckle_index, mass 0.01; visual mesh filename=../meshes/F03_Finger_base.stl scale=0.001 0.001 0.001
- added link lh_knuckle_little, mass 0.01; visual mesh filename=../meshes/F03_Finger_base.stl scale=0.001 0.001 0.001
- added link lh_knuckle_middle, mass 0.01; visual mesh filename=../meshes/F03_Finger_base.stl scale=0.001 0.001 0.001
- added link lh_knuckle_ring, mass 0.01; visual mesh filename=../meshes/F03_Finger_base.stl scale=0.001 0.001 0.001
- added link lh_knuckle_thumb, mass 0.01; visual mesh filename=../meshes/F03_Thumb_base.stl scale=0.001 0.001 0.001
- added link lh_little_DIP, mass 0.0025; collision box size=0.01 0.01 0.02; visual mesh filename=../meshes/F03_AL_link_DIP.stl scale=0.001 0.001 0.001
- added link lh_little_MCP, mass 0.0125; collision box size=0.015 0.015 0.035; visual mesh filename=../meshes/F03_AL_link_MCP.stl scale=0.001 0.001 0.001
- added link lh_little_PIP, mass 0.0125; collision box size=0.012 0.012 0.025; visual mesh filename=../meshes/F03_AL_link_PIP.stl scale=0.001 0.001 0.001
- added link lh_middle_DIP, mass 0.0025; collision box size=0.01 0.01 0.02; visual mesh filename=../meshes/F03_AL_link_DIP.stl scale=0.001 0.001 0.001
- added link lh_middle_MCP, mass 0.0125; collision box size=0.015 0.015 0.035; visual mesh filename=../meshes/F03_AL_link_MCP.stl scale=0.001 0.001 0.001
- added link lh_middle_PIP, mass 0.0125; collision box size=0.012 0.012 0.025; visual mesh filename=../meshes/F03_AL_link_PIP.stl scale=0.001 0.001 0.001
- added link lh_motor_index, mass 0.015; visual box size=0.016 0.035 0.02
- added link lh_motor_little, mass 0.015; visual box size=0.016 0.035 0.02
- added link lh_motor_middle, mass 0.015; visual box size=0.016 0.035 0.02
- added link lh_motor_ring, mass 0.015; visual box size=0.016 0.035 0.02
- added link lh_motor_thumb_DIP, mass 0.0025; visual box size=0.016 0.035 0.02
- added link lh_motor_thumb_jo, mass 0.015; visual box size=0.016 0.035 0.02
- added link lh_pris_index, mass 0.015; visual box size=0.005 0.005 0.025
- added link lh_pris_little, mass 0.015; visual box size=0.005 0.005 0.025
- added link lh_pris_middle, mass 0.015; visual box size=0.005 0.005 0.025
- added link lh_pris_ring, mass 0.015; visual box size=0.005 0.005 0.025
- added link lh_pris_thumb_DIP, mass 0.015; visual box size=0.005 0.005 0.025
- added link lh_pris_thumb_jo, mass 0.015; visual box size=0.005 0.005 0.025
- added link lh_ring_DIP, mass 0.0025; collision box size=0.01 0.01 0.02; visual mesh filename=../meshes/F03_AL_link_DIP.stl scale=0.001 0.001 0.001
- added link lh_ring_MCP, mass 0.0125; collision box size=0.015 0.015 0.035; visual mesh filename=../meshes/F03_AL_link_MCP.stl scale=0.001 0.001 0.001
- added link lh_ring_PIP, mass 0.0125; collision box size=0.012 0.012 0.025; visual mesh filename=../meshes/F03_AL_link_PIP.stl scale=0.001 0.001 0.001
- added link lh_thumb_DIP, mass 0.0025; collision box size=0.01 0.01 0.02; visual mesh filename=../meshes/F03_AL_link_DIP.stl scale=0.001 0.001 0.001
- added link lh_thumb_MCP, mass 0.0125; collision box size=0.015 0.015 0.035; visual mesh filename=../meshes/F03_AL_link_MCP.stl scale=0.001 0.001 0.001
- added link lh_thumb_joint, mass 0.015; collision box size=0.015 0.015 0.02; visual mesh filename=../meshes/F03_Thumb_joint.stl scale=0.001 0.001 0.001
- added link lh_wrist_plate; collision mesh filename=../meshes/F03_AL_link_hand_wrist_part.stl scale=0.001 0.001 0.001; visual mesh filename=../meshes/F03_AL_link_hand_wrist_part.stl scale=0.001 0.001 0.001
- added link rh_ee_index_link
- added link rh_ee_little_link
- added link rh_ee_middle_link
- added link rh_ee_ring_link
- added link rh_ee_thumb_link
- added link rh_hand_palm, mass 0.09; collision mesh filename=../meshes/F03_AL_palm.stl scale=0.001 0.001 0.001; visual mesh filename=../meshes/F03_AL_palm.stl scale=0.001 0.001 0.001
- added link rh_index_DIP, mass 0.0025; collision box size=0.01 0.01 0.02; visual mesh filename=../meshes/F03_AL_link_DIP.stl scale=0.001 0.001 0.001
- added link rh_index_MCP, mass 0.0125; collision box size=0.015 0.015 0.035; visual mesh filename=../meshes/F03_AL_link_MCP.stl scale=0.001 0.001 0.001
- added link rh_index_PIP, mass 0.0125; collision box size=0.012 0.012 0.025; visual mesh filename=../meshes/F03_AL_link_PIP.stl scale=0.001 0.001 0.001
- added link rh_knuckle_index, mass 0.01; visual mesh filename=../meshes/F03_Finger_base.stl scale=0.001 0.001 0.001
- added link rh_knuckle_little, mass 0.01; visual mesh filename=../meshes/F03_Finger_base.stl scale=0.001 0.001 0.001
- added link rh_knuckle_middle, mass 0.01; visual mesh filename=../meshes/F03_Finger_base.stl scale=0.001 0.001 0.001
- added link rh_knuckle_ring, mass 0.01; visual mesh filename=../meshes/F03_Finger_base.stl scale=0.001 0.001 0.001
- added link rh_knuckle_thumb, mass 0.01; visual mesh filename=../meshes/F03_Thumb_base.stl scale=0.001 0.001 0.001
- added link rh_little_DIP, mass 0.0025; collision box size=0.01 0.01 0.02; visual mesh filename=../meshes/F03_AL_link_DIP.stl scale=0.001 0.001 0.001
- added link rh_little_MCP, mass 0.0125; collision box size=0.015 0.015 0.035; visual mesh filename=../meshes/F03_AL_link_MCP.stl scale=0.001 0.001 0.001
- added link rh_little_PIP, mass 0.0125; collision box size=0.012 0.012 0.025; visual mesh filename=../meshes/F03_AL_link_PIP.stl scale=0.001 0.001 0.001
- added link rh_middle_DIP, mass 0.0025; collision box size=0.01 0.01 0.02; visual mesh filename=../meshes/F03_AL_link_DIP.stl scale=0.001 0.001 0.001
- added link rh_middle_MCP, mass 0.0125; collision box size=0.015 0.015 0.035; visual mesh filename=../meshes/F03_AL_link_MCP.stl scale=0.001 0.001 0.001
- added link rh_middle_PIP, mass 0.0125; collision box size=0.012 0.012 0.025; visual mesh filename=../meshes/F03_AL_link_PIP.stl scale=0.001 0.001 0.001
- added link rh_motor_index, mass 0.015; visual box size=0.016 0.035 0.02
- added link rh_motor_little, mass 0.015; visual box size=0.016 0.035 0.02
- added link rh_motor_middle, mass 0.015; visual box size=0.016 0.035 0.02
- added link rh_motor_ring, mass 0.015; visual box size=0.016 0.035 0.02
- added link rh_motor_thumb_DIP, mass 0.0025; visual box size=0.016 0.035 0.02
- added link rh_motor_thumb_jo, mass 0.015; visual box size=0.016 0.035 0.02
- added link rh_pris_index, mass 0.015; visual box size=0.005 0.005 0.025
- added link rh_pris_little, mass 0.015; visual box size=0.005 0.005 0.025
- added link rh_pris_middle, mass 0.015; visual box size=0.005 0.005 0.025
- added link rh_pris_ring, mass 0.015; visual box size=0.005 0.005 0.025
- added link rh_pris_thumb_DIP, mass 0.015; visual box size=0.005 0.005 0.025
- added link rh_pris_thumb_jo, mass 0.015; visual box size=0.005 0.005 0.025
- added link rh_ring_DIP, mass 0.0025; collision box size=0.01 0.01 0.02; visual mesh filename=../meshes/F03_AL_link_DIP.stl scale=0.001 0.001 0.001
- added link rh_ring_MCP, mass 0.0125; collision box size=0.015 0.015 0.035; visual mesh filename=../meshes/F03_AL_link_MCP.stl scale=0.001 0.001 0.001
- added link rh_ring_PIP, mass 0.0125; collision box size=0.012 0.012 0.025; visual mesh filename=../meshes/F03_AL_link_PIP.stl scale=0.001 0.001 0.001
- added link rh_thumb_DIP, mass 0.0025; collision box size=0.01 0.01 0.02; visual mesh filename=../meshes/F03_AL_link_DIP.stl scale=0.001 0.001 0.001
- added link rh_thumb_MCP, mass 0.0125; collision box size=0.015 0.015 0.035; visual mesh filename=../meshes/F03_AL_link_MCP.stl scale=0.001 0.001 0.001
- added link rh_thumb_joint, mass 0.015; collision box size=0.015 0.015 0.02; visual mesh filename=../meshes/F03_Thumb_joint.stl scale=0.001 0.001 0.001
- added link rh_wrist_plate; collision mesh filename=../meshes/F03_AL_link_hand_wrist_part.stl scale=0.001 0.001 0.001; visual mesh filename=../meshes/F03_AL_link_hand_wrist_part.stl scale=0.001 0.001 0.001
Joints:
- removed joint left_wrist_to_hand
- removed joint lh_index_dp_joint
- removed joint lh_index_mp_joint
- removed joint lh_index_pp_joint
- removed joint lh_middle_dp_joint
- removed joint lh_middle_mp_joint
- removed joint lh_middle_pp_joint
- removed joint lh_pinky_dp_joint
- removed joint lh_pinky_mp_joint
- removed joint lh_pinky_pp_joint
- removed joint lh_ring_dp_joint
- removed joint lh_ring_mp_joint
- removed joint lh_ring_pp_joint
- removed joint lh_thumb_base_joint
- removed joint lh_thumb_dp_joint
- removed joint lh_thumb_mp_joint
- removed joint lh_thumb_pp_joint
- removed joint rh_index_dp_joint
- removed joint rh_index_mp_joint
- removed joint rh_index_pp_joint
- removed joint rh_middle_dp_joint
- removed joint rh_middle_mp_joint
- removed joint rh_middle_pp_joint
- removed joint rh_pinky_dp_joint
- removed joint rh_pinky_mp_joint
- removed joint rh_pinky_pp_joint
- removed joint rh_ring_dp_joint
- removed joint rh_ring_mp_joint
- removed joint rh_ring_pp_joint
- removed joint rh_thumb_base_joint
- removed joint rh_thumb_dp_joint
- removed joint rh_thumb_mp_joint
- removed joint rh_thumb_pp_joint
- removed joint right_wrist_to_hand
- added joint lh_ee_index_joint: type fixed, parent lh_index_DIP, child lh_ee_index_link, origin xyz=0.0 0.0 0.025725 rpy=0.0 0.0 0.0
- added joint lh_ee_little_joint: type fixed, parent lh_little_DIP, child lh_ee_little_link, origin xyz=0.0 0.0 0.025725 rpy=0.0 0.0 0.0
- added joint lh_ee_middle_joint: type fixed, parent lh_middle_DIP, child lh_ee_middle_link, origin xyz=0.0 0.0 0.025725 rpy=0.0 0.0 0.0
- added joint lh_ee_ring_joint: type fixed, parent lh_ring_DIP, child lh_ee_ring_link, origin xyz=0.0 0.0 0.025725 rpy=0.0 0.0 0.0
- added joint lh_ee_th_joint: type fixed, parent lh_thumb_DIP, child lh_ee_thumb_link, origin xyz=-0.025725 0.0 0.0  rpy=0.0 0.0 0.0
- added joint lh_hand_wrist_plate_to_hand_palm: type fixed, parent lh_wrist_plate, child lh_hand_palm, origin xyz=0 0 .026
- added joint lh_index_DIP_joint: type revolute, parent lh_index_PIP, child lh_index_DIP, origin xyz=0.0 0.0 0.0233, axis -1 0 0, limit lower=0.0 upper=1.0 effort=10.0 velocity=1.0, mimic joint=lh_pris_index_joint multiplier=100.00 offset=0.0
- added joint lh_index_MCP_joint: type revolute, parent lh_knuckle_index, child lh_index_MCP, origin xyz=-0.0002 -0.00677 0.0538, axis -1 0 0, limit lower=0.0 upper=1.3 effort=10.0 velocity=1.0, mimic joint=lh_pris_index_joint multiplier=100.00 offset=0.0
- added joint lh_index_PIP_joint: type revolute, parent lh_index_MCP, child lh_index_PIP, origin xyz=0.0 -0.00208 0.02677, axis -1 0 0, limit lower=0.0 upper=1.0 effort=10.0 velocity=1.0, mimic joint=lh_pris_index_joint multiplier=100.00 offset=0.0
- added joint lh_knuckle_index_joint: type fixed, parent lh_hand_palm, child lh_knuckle_index, origin xyz=-0.0313 0.0160 0.0295
- added joint lh_knuckle_little_joint: type fixed, parent lh_hand_palm, child lh_knuckle_little, origin xyz=0.0317 0.0160 0.0295
- added joint lh_knuckle_middle_joint: type fixed, parent lh_hand_palm, child lh_knuckle_middle, origin xyz=-0.0103 0.0160 0.0295
- added joint lh_knuckle_ring_joint: type fixed, parent lh_hand_palm, child lh_knuckle_ring, origin xyz=0.010700000000000001 0.0160 0.0295
- added joint lh_knuckle_thumb_joint: type fixed, parent lh_hand_palm, child lh_knuckle_thumb, origin xyz=0.0345 0.0162 0.0186
- added joint lh_little_DIP_joint: type revolute, parent lh_little_PIP, child lh_little_DIP, origin xyz=0.0 0.0 0.0233, axis -1 0 0, limit lower=0.0 upper=1.0 effort=10.0 velocity=1.0, mimic joint=lh_pris_little_joint multiplier=100.00 offset=0.0
- added joint lh_little_MCP_joint: type revolute, parent lh_knuckle_little, child lh_little_MCP, origin xyz=-0.0002 -0.00677 0.0538, axis -1 0 0, limit lower=0.0 upper=1.3 effort=10.0 velocity=1.0, mimic joint=lh_pris_little_joint multiplier=100.00 offset=0.0
- added joint lh_little_PIP_joint: type revolute, parent lh_little_MCP, child lh_little_PIP, origin xyz=0.0 -0.00208 0.02677, axis -1 0 0, limit lower=0.0 upper=1.0 effort=10.0 velocity=1.0, mimic joint=lh_pris_little_joint multiplier=100.00 offset=0.0
- added joint lh_middle_DIP_joint: type revolute, parent lh_middle_PIP, child lh_middle_DIP, origin xyz=0.0 0.0 0.0233, axis -1 0 0, limit lower=0.0 upper=1.0 effort=10.0 velocity=1.0, mimic joint=lh_pris_middle_joint multiplier=100.00 offset=0.0
- added joint lh_middle_MCP_joint: type revolute, parent lh_knuckle_middle, child lh_middle_MCP, origin xyz=-0.0002 -0.00677 0.0538, axis -1 0 0, limit lower=0.0 upper=1.3 effort=10.0 velocity=1.0, mimic joint=lh_pris_middle_joint multiplier=100.00 offset=0.0
- added joint lh_middle_PIP_joint: type revolute, parent lh_middle_MCP, child lh_middle_PIP, origin xyz=0.0 -0.00208 0.02677, axis -1 0 0, limit lower=0.0 upper=1.0 effort=10.0 velocity=1.0, mimic joint=lh_pris_middle_joint multiplier=100.00 offset=0.0
- added joint lh_motor_index_joint: type fixed, parent lh_knuckle_index, child lh_motor_index, origin xyz=0.0 -0.0145 0.006 rpy=1.57 0 0, axis 1 0 0
- added joint lh_motor_little_joint: type fixed, parent lh_knuckle_little, child lh_motor_little, origin xyz=0.0 -0.0145 0.006 rpy=1.57 0 0, axis 1 0 0
- added joint lh_motor_middle_joint: type fixed, parent lh_knuckle_middle, child lh_motor_middle, origin xyz=0.0 -0.0145 0.006 rpy=1.57 0 0, axis 1 0 0
- added joint lh_motor_ring_joint: type fixed, parent lh_knuckle_ring, child lh_motor_ring, origin xyz=0.0 -0.0145 0.006 rpy=1.57 0 0, axis 1 0 0
- added joint lh_motor_thumb_DIP_joint: type fixed, parent lh_thumb_joint, child lh_motor_thumb_DIP, origin xyz=0.0125 -0.0055 -0.015 rpy=3.14 3.14 -1.57, axis 1 0 0
- added joint lh_motor_thumb_jo_joint: type fixed, parent lh_knuckle_thumb, child lh_motor_thumb_jo, origin xyz=-0.008 -0.015 0.0 rpy=1.57 -1.57 0, axis 1 0 0
- added joint lh_pris_index_joint: type prismatic, parent lh_motor_index, child lh_pris_index, origin xyz=0.0 0.03 0.0 rpy=1.57 0 0, axis 0 0 -1, limit lower=0.0 upper=0.0103 effort=10.0 velocity=0.1
- added joint lh_pris_little_joint: type prismatic, parent lh_motor_little, child lh_pris_little, origin xyz=0.0 0.03 0.0 rpy=1.57 0 0, axis 0 0 -1, limit lower=0.0 upper=0.0103 effort=10.0 velocity=0.1
- added joint lh_pris_middle_joint: type prismatic, parent lh_motor_middle, child lh_pris_middle, origin xyz=0.0 0.03 0.0 rpy=1.57 0 0, axis 0 0 -1, limit lower=0.0 upper=0.0103 effort=10.0 velocity=0.1
- added joint lh_pris_ring_joint: type prismatic, parent lh_motor_ring, child lh_pris_ring, origin xyz=0.0 0.03 0.0 rpy=1.57 0 0, axis 0 0 -1, limit lower=0.0 upper=0.0103 effort=10.0 velocity=0.1
- added joint lh_pris_thumb_DIP_joint: type prismatic, parent lh_motor_thumb_DIP, child lh_pris_thumb_DIP, origin xyz=0.0 -0.015 0.0 rpy=1.57 0 0, axis 0 0 -1, limit lower=0.0 upper=0.0103 effort=10.0 velocity=0.1
- added joint lh_pris_thumb_jo_joint: type prismatic, parent lh_motor_thumb_jo, child lh_pris_thumb_jo, origin xyz=0.0 -0.015 0.0 rpy=1.57 0 0, axis 0 0 -1, limit lower=0.0 upper=0.0103 effort=10.0 velocity=0.1
- added joint lh_ring_DIP_joint: type revolute, parent lh_ring_PIP, child lh_ring_DIP, origin xyz=0.0 0.0 0.0233, axis -1 0 0, limit lower=0.0 upper=1.0 effort=10.0 velocity=1.0, mimic joint=lh_pris_ring_joint multiplier=100.00 offset=0.0
- added joint lh_ring_MCP_joint: type revolute, parent lh_knuckle_ring, child lh_ring_MCP, origin xyz=-0.0002 -0.00677 0.0538, axis -1 0 0, limit lower=0.0 upper=1.3 effort=10.0 velocity=1.0, mimic joint=lh_pris_ring_joint multiplier=100.00 offset=0.0
- added joint lh_ring_PIP_joint: type revolute, parent lh_ring_MCP, child lh_ring_PIP, origin xyz=0.0 -0.00208 0.02677, axis -1 0 0, limit lower=0.0 upper=1.0 effort=10.0 velocity=1.0, mimic joint=lh_pris_ring_joint multiplier=100.00 offset=0.0
- added joint lh_thumb_DIP_joint: type revolute, parent lh_thumb_MCP, child lh_thumb_DIP, origin xyz=-0.0298 0.0 -0.0042 rpy=0.0 0.0 0.0, axis 0 1 0, limit lower=0.0 upper=0.8 effort=10.0 velocity=1.0, mimic joint=lh_pris_thumb_DIP_joint multiplier=100.00 offset=0.0
- added joint lh_thumb_MCP_joint: type revolute, parent lh_thumb_joint, child lh_thumb_MCP, origin xyz=-0.031 -0.0055 0.0 rpy=0.0 0.4538 0.0, axis 0 1 0, limit lower=0.0 upper=1.0 effort=10.0 velocity=1.0, mimic joint=lh_pris_thumb_DIP_joint multiplier=100.00 offset=0.0
- added joint lh_thumb_jo_joint: type revolute, parent lh_knuckle_thumb, child lh_thumb_joint, origin xyz=-0.0558 -0.00675 0.0 rpy=0.0 0.0 -0.6021, axis 0 0 -1, limit lower=0.0 upper=1.8 effort=10.0 velocity=1.0, mimic joint=lh_pris_thumb_jo_joint multiplier=100.00 offset=0.0
- added joint lh_wrist_plate_joint: type fixed, parent left_wrist_yaw_link, child lh_wrist_plate, origin xyz=0 0 0 rpy=-0.7854 3.14159 -1.5708
- added joint rh_ee_index_joint: type fixed, parent rh_index_DIP, child rh_ee_index_link, origin xyz=0.0 0.0 0.025725 rpy=0.0 0.0 0.0
- added joint rh_ee_little_joint: type fixed, parent rh_little_DIP, child rh_ee_little_link, origin xyz=0.0 0.0 0.025725 rpy=0.0 0.0 0.0
- added joint rh_ee_middle_joint: type fixed, parent rh_middle_DIP, child rh_ee_middle_link, origin xyz=0.0 0.0 0.025725 rpy=0.0 0.0 0.0
- added joint rh_ee_ring_joint: type fixed, parent rh_ring_DIP, child rh_ee_ring_link, origin xyz=0.0 0.0 0.025725 rpy=0.0 0.0 0.0
- added joint rh_ee_th_joint: type fixed, parent rh_thumb_DIP, child rh_ee_thumb_link, origin xyz=-0.025725 0.0 0.0  rpy=0.0 0.0 0.0
- added joint rh_hand_wrist_plate_to_hand_palm: type fixed, parent rh_wrist_plate, child rh_hand_palm, origin xyz=0 0 .026
- added joint rh_index_DIP_joint: type revolute, parent rh_index_PIP, child rh_index_DIP, origin xyz=0.0 0.0 0.0233, axis -1 0 0, limit lower=0.0 upper=1.0 effort=10.0 velocity=1.0, mimic joint=rh_pris_index_joint multiplier=100.00 offset=0.0
- added joint rh_index_MCP_joint: type revolute, parent rh_knuckle_index, child rh_index_MCP, origin xyz=-0.0002 -0.00677 0.0538, axis -1 0 0, limit lower=0.0 upper=1.3 effort=10.0 velocity=1.0, mimic joint=rh_pris_index_joint multiplier=100.00 offset=0.0
- added joint rh_index_PIP_joint: type revolute, parent rh_index_MCP, child rh_index_PIP, origin xyz=0.0 -0.00208 0.02677, axis -1 0 0, limit lower=0.0 upper=1.0 effort=10.0 velocity=1.0, mimic joint=rh_pris_index_joint multiplier=100.00 offset=0.0
- added joint rh_knuckle_index_joint: type fixed, parent rh_hand_palm, child rh_knuckle_index, origin xyz=-0.0313 0.0160 0.0295
- added joint rh_knuckle_little_joint: type fixed, parent rh_hand_palm, child rh_knuckle_little, origin xyz=0.0317 0.0160 0.0295
- added joint rh_knuckle_middle_joint: type fixed, parent rh_hand_palm, child rh_knuckle_middle, origin xyz=-0.0103 0.0160 0.0295
- added joint rh_knuckle_ring_joint: type fixed, parent rh_hand_palm, child rh_knuckle_ring, origin xyz=0.010700000000000001 0.0160 0.0295
- added joint rh_knuckle_thumb_joint: type fixed, parent rh_hand_palm, child rh_knuckle_thumb, origin xyz=0.0345 0.0162 0.0186
- added joint rh_little_DIP_joint: type revolute, parent rh_little_PIP, child rh_little_DIP, origin xyz=0.0 0.0 0.0233, axis -1 0 0, limit lower=0.0 upper=1.0 effort=10.0 velocity=1.0, mimic joint=rh_pris_little_joint multiplier=100.00 offset=0.0
- added joint rh_little_MCP_joint: type revolute, parent rh_knuckle_little, child rh_little_MCP, origin xyz=-0.0002 -0.00677 0.0538, axis -1 0 0, limit lower=0.0 upper=1.3 effort=10.0 velocity=1.0, mimic joint=rh_pris_little_joint multiplier=100.00 offset=0.0
- added joint rh_little_PIP_joint: type revolute, parent rh_little_MCP, child rh_little_PIP, origin xyz=0.0 -0.00208 0.02677, axis -1 0 0, limit lower=0.0 upper=1.0 effort=10.0 velocity=1.0, mimic joint=rh_pris_little_joint multiplier=100.00 offset=0.0
- added joint rh_middle_DIP_joint: type revolute, parent rh_middle_PIP, child rh_middle_DIP, origin xyz=0.0 0.0 0.0233, axis -1 0 0, limit lower=0.0 upper=1.0 effort=10.0 velocity=1.0, mimic joint=rh_pris_middle_joint multiplier=100.00 offset=0.0
- added joint rh_middle_MCP_joint: type revolute, parent rh_knuckle_middle, child rh_middle_MCP, origin xyz=-0.0002 -0.00677 0.0538, axis -1 0 0, limit lower=0.0 upper=1.3 effort=10.0 velocity=1.0, mimic joint=rh_pris_middle_joint multiplier=100.00 offset=0.0
- added joint rh_middle_PIP_joint: type revolute, parent rh_middle_MCP, child rh_middle_PIP, origin xyz=0.0 -0.00208 0.02677, axis -1 0 0, limit lower=0.0 upper=1.0 effort=10.0 velocity=1.0, mimic joint=rh_pris_middle_joint multiplier=100.00 offset=0.0
- added joint rh_motor_index_joint: type fixed, parent rh_knuckle_index, child rh_motor_index, origin xyz=0.0 -0.0145 0.006 rpy=1.57 0 0, axis 1 0 0
- added joint rh_motor_little_joint: type fixed, parent rh_knuckle_little, child rh_motor_little, origin xyz=0.0 -0.0145 0.006 rpy=1.57 0 0, axis 1 0 0
- added joint rh_motor_middle_joint: type fixed, parent rh_knuckle_middle, child rh_motor_middle, origin xyz=0.0 -0.0145 0.006 rpy=1.57 0 0, axis 1 0 0
- added joint rh_motor_ring_joint: type fixed, parent rh_knuckle_ring, child rh_motor_ring, origin xyz=0.0 -0.0145 0.006 rpy=1.57 0 0, axis 1 0 0
- added joint rh_motor_thumb_DIP_joint: type fixed, parent rh_thumb_joint, child rh_motor_thumb_DIP, origin xyz=0.0125 -0.0055 -0.015 rpy=3.14 3.14 -1.57, axis 1 0 0
- added joint rh_motor_thumb_jo_joint: type fixed, parent rh_knuckle_thumb, child rh_motor_thumb_jo, origin xyz=-0.008 -0.015 0.0 rpy=1.57 -1.57 0, axis 1 0 0
- added joint rh_pris_index_joint: type prismatic, parent rh_motor_index, child rh_pris_index, origin xyz=0.0 0.03 0.0 rpy=1.57 0 0, axis 0 0 -1, limit lower=0.0 upper=0.0103 effort=10.0 velocity=0.1
- added joint rh_pris_little_joint: type prismatic, parent rh_motor_little, child rh_pris_little, origin xyz=0.0 0.03 0.0 rpy=1.57 0 0, axis 0 0 -1, limit lower=0.0 upper=0.0103 effort=10.0 velocity=0.1
- added joint rh_pris_middle_joint: type prismatic, parent rh_motor_middle, child rh_pris_middle, origin xyz=0.0 0.03 0.0 rpy=1.57 0 0, axis 0 0 -1, limit lower=0.0 upper=0.0103 effort=10.0 velocity=0.1
- added joint rh_pris_ring_joint: type prismatic, parent rh_motor_ring, child rh_pris_ring, origin xyz=0.0 0.03 0.0 rpy=1.57 0 0, axis 0 0 -1, limit lower=0.0 upper=0.0103 effort=10.0 velocity=0.1
- added joint rh_pris_thumb_DIP_joint: type prismatic, parent rh_motor_thumb_DIP, child rh_pris_thumb_DIP, origin xyz=0.0 -0.015 0.0 rpy=1.57 0 0, axis 0 0 -1, limit lower=0.0 upper=0.0103 effort=10.0 velocity=0.1
- added joint rh_pris_thumb_jo_joint: type prismatic, parent rh_motor_thumb_jo, child rh_pris_thumb_jo, origin xyz=0.0 -0.015 0.0 rpy=1.57 0 0, axis 0 0 -1, limit lower=0.0 upper=0.0103 effort=10.0 velocity=0.1
- added joint rh_ring_DIP_joint: type revolute, parent rh_ring_PIP, child rh_ring_DIP, origin xyz=0.0 0.0 0.0233, axis -1 0 0, limit lower=0.0 upper=1.0 effort=10.0 velocity=1.0, mimic joint=rh_pris_ring_joint multiplier=100.00 offset=0.0
- added joint rh_ring_MCP_joint: type revolute, parent rh_knuckle_ring, child rh_ring_MCP, origin xyz=-0.0002 -0.00677 0.0538, axis -1 0 0, limit lower=0.0 upper=1.3 effort=10.0 velocity=1.0, mimic joint=rh_pris_ring_joint multiplier=100.00 offset=0.0
- added joint rh_ring_PIP_joint: type revolute, parent rh_ring_MCP, child rh_ring_PIP, origin xyz=0.0 -0.00208 0.02677, axis -1 0 0, limit lower=0.0 upper=1.0 effort=10.0 velocity=1.0, mimic joint=rh_pris_ring_joint multiplier=100.00 offset=0.0
- added joint rh_thumb_DIP_joint: type revolute, parent rh_thumb_MCP, child rh_thumb_DIP, origin xyz=-0.0298 0.0 -0.0042 rpy=0.0 0.0 0.0, axis 0 1 0, limit lower=0.0 upper=0.8 effort=10.0 velocity=1.0, mimic joint=rh_pris_thumb_DIP_joint multiplier=100.00 offset=0.0
- added joint rh_thumb_MCP_joint: type revolute, parent rh_thumb_joint, child rh_thumb_MCP, origin xyz=-0.031 -0.0055 0.0 rpy=0.0 0.4538 0.0, axis 0 1 0, limit lower=0.0 upper=1.0 effort=10.0 velocity=1.0, mimic joint=rh_pris_thumb_DIP_joint multiplier=100.00 offset=0.0
- added joint rh_thumb_jo_joint: type revolute, parent rh_knuckle_thumb, child rh_thumb_joint, origin xyz=-0.0558 -0.00675 0.0 rpy=0.0 0.0 -0.6021, axis 0 0 -1, limit lower=0.0 upper=1.8 effort=10.0 velocity=1.0, mimic joint=rh_pris_thumb_jo_joint multiplier=100.00 offset=0.0
- added joint rh_wrist_plate_joint: type fixed, parent right_wrist_yaw_link, child rh_wrist_plate, origin xyz=0 0 0 rpy=0.7854 3.14159 -1.5708
