Commit message: Hand changed.

File: assets/xacro/master_assembly.xacro (robot description, xacro)
@@ -524,20 +524,16 @@
     <dynamics damping="0.0282528" friction="0.08" armature="0.001" />
   </joint>
-  <xacro:include filename="faive_hand.xacro" />
-  <!-- Right hand -->
-  <xacro:faive_hand prefix="rh_" mesh_dir="${mesh_dir}" mirror_factor="1" />
-  <!-- Left hand (mirrored) -->
-  <xacro:faive_hand prefix="lh_" mesh_dir="${mesh_dir}" mirror_factor="-1" />
-  <!-- Right hand attachment: pitch +90°, yaw +90° -->
-  <joint name="right_wrist_to_hand" type="fixed">
-      <parent link="right_wrist_yaw_link" />
-      <child link="rh_palm" />
-      <origin xyz="-0.035 -0.000182 0.032" rpy="0.7854 3.14159 -1.5708" />
-  </joint>
-  <!-- Left hand attachment: pitch -90°, yaw +90° -->
-  <joint name="left_wrist_to_hand" type="fixed">
-      <parent link="left_wrist_yaw_link" />
-      <child link="lh_palm" />
-      <origin xyz="-0.035 0.000182 0.032" rpy="-0.7854 3.14159 1.5708" />
-  </joint>
+<xacro:include filename="hri_hand.xacro" />
+  <xacro:hri_hand
+      prefix="rh_"
+      parent="right_wrist_yaw_link"
+      mesh_dir="../meshes">
+      <origin xyz="0 0 0" rpy="0.7854 3.14159 -1.5708" />
+  </xacro:hri_hand>
+  <xacro:hri_hand
+      prefix="lh_"
+      parent="left_wrist_yaw_link"
+      mesh_dir="../meshes">
+      <origin xyz="0 0 0" rpy="-0.7854 3.14159 -1.5708" />
+  </xacro:hri_hand>
 </robot>

Commit message: Implemented combination of modified hands with body

File: assets/urdf/revexbot1.urdf (robot description, URDF)
Before this commit: robot RevEx_Full_Assembly, 106 links, 105 joints
Links:
- link lh_hand_palm: geometry collision mesh filename=../meshes/lh_f03_al_palm.stl scale=1.0 1.0 1.0; visual mesh filename=../meshes/lh_f03_al_palm.stl scale=1.0 1.0 1.0
- link lh_index_DIP: geometry collision box size=0.01 0.01 0.02; visual mesh filename=../meshes/lh_f03_al_link_dip.stl scale=1.0 1.0 1.0
- link lh_index_MCP: geometry collision box size=0.015 0.015 0.035; visual mesh filename=../meshes/lh_f03_al_link_mcp.stl scale=1.0 1.0 1.0
- link lh_index_PIP: geometry collision box size=0.012 0.012 0.025; visual mesh filename=../meshes/lh_f03_al_link_pip.stl scale=1.0 1.0 1.0
- link lh_knuckle_index: geometry visual mesh filename=../meshes/lh_f03_finger_base.stl scale=1.0 1.0 1.0
- link lh_knuckle_little: geometry visual mesh filename=../meshes/lh_f03_finger_base.stl scale=1.0 1.0 1.0
- link lh_knuckle_middle: geometry visual mesh filename=../meshes/lh_f03_finger_base.stl scale=1.0 1.0 1.0
- link lh_knuckle_ring: geometry visual mesh filename=../meshes/lh_f03_finger_base.stl scale=1.0 1.0 1.0
- link lh_knuckle_thumb: geometry visual mesh filename=../meshes/lh_f03_thumb_base.stl scale=1.0 1.0 1.0
- link lh_little_DIP: geometry collision box size=0.01 0.01 0.02; visual mesh filename=../meshes/lh_f03_al_link_dip.stl scale=1.0 1.0 1.0
- link lh_little_MCP: geometry collision box size=0.015 0.015 0.035; visual mesh filename=../meshes/lh_f03_al_link_mcp.stl scale=1.0 1.0 1.0
- link lh_little_PIP: geometry collision box size=0.012 0.012 0.025; visual mesh filename=../meshes/lh_f03_al_link_pip.stl scale=1.0 1.0 1.0
- link lh_middle_DIP: geometry collision box size=0.01 0.01 0.02; visual mesh filename=../meshes/lh_f03_al_link_dip.stl scale=1.0 1.0 1.0
- link lh_middle_MCP: geometry collision box size=0.015 0.015 0.035; visual mesh filename=../meshes/lh_f03_al_link_mcp.stl scale=1.0 1.0 1.0
- link lh_middle_PIP: geometry collision box size=0.012 0.012 0.025; visual mesh filename=../meshes/lh_f03_al_link_pip.stl scale=1.0 1.0 1.0
- link lh_ring_DIP: geometry collision box size=0.01 0.01 0.02; visual mesh filename=../meshes/lh_f03_al_link_dip.stl scale=1.0 1.0 1.0
- link lh_ring_MCP: geometry collision box size=0.015 0.015 0.035; visual mesh filename=../meshes/lh_f03_al_link_mcp.stl scale=1.0 1.0 1.0
- link lh_ring_PIP: geometry collision box size=0.012 0.012 0.025; visual mesh filename=../meshes/lh_f03_al_link_pip.stl scale=1.0 1.0 1.0
- link lh_thumb_DIP: geometry collision box size=0.01 0.01 0.02; visual mesh filename=../meshes/lh_f03_al_link_dip.stl scale=1.0 1.0 1.0
- link lh_thumb_MCP: geometry collision box size=0.015 0.015 0.035; visual mesh filename=../meshes/lh_f03_al_link_mcp.stl scale=1.0 1.0 1.0
- link lh_thumb_joint: geometry collision box size=0.015 0.015 0.02; visual mesh filename=../meshes/lh_f03_thumb_joint.stl scale=1.0 1.0 1.0
- link lh_wrist_plate: geometry collision mesh filename=../meshes/lh_f03_al_link_hand_wrist_part.stl scale=1.0 1.0 1.0; visual mesh filename=../meshes/lh_f03_al_link_hand_wrist_part.stl scale=1.0 1.0 1.0
- link rh_hand_palm: geometry collision mesh filename=../meshes/rh_f03_al_palm.stl scale=1.0 1.0 1.0; visual mesh filename=../meshes/rh_f03_al_palm.stl scale=1.0 1.0 1.0
- link rh_index_DIP: geometry collision box size=0.01 0.01 0.02; visual mesh filename=../meshes/rh_f03_al_link_dip.stl scale=1.0 1.0 1.0
- link rh_index_MCP: geometry collision box size=0.015 0.015 0.035; visual mesh filename=../meshes/rh_f03_al_link_mcp.stl scale=1.0 1.0 1.0
- link rh_index_PIP: geometry collision box size=0.012 0.012 0.025; visual mesh filename=../meshes/rh_f03_al_link_pip.stl scale=1.0 1.0 1.0
- link rh_knuckle_index: geometry visual mesh filename=../meshes/rh_f03_finger_base.stl scale=1.0 1.0 1.0
- link rh_knuckle_little: geometry visual mesh filename=../meshes/rh_f03_finger_base.stl scale=1.0 1.0 1.0
- link rh_knuckle_middle: geometry visual mesh filename=../meshes/rh_f03_finger_base.stl scale=1.0 1.0 1.0
- link rh_knuckle_ring: geometry visual mesh filename=../meshes/rh_f03_finger_base.stl scale=1.0 1.0 1.0
- link rh_knuckle_thumb: geometry visual mesh filename=../meshes/rh_f03_thumb_base.stl scale=1.0 1.0 1.0
- link rh_little_DIP: geometry collision box size=0.01 0.01 0.02; visual mesh filename=../meshes/rh_f03_al_link_dip.stl scale=1.0 1.0 1.0
- link rh_little_MCP: geometry collision box size=0.015 0.015 0.035; visual mesh filename=../meshes/rh_f03_al_link_mcp.stl scale=1.0 1.0 1.0
- link rh_little_PIP: geometry collision box size=0.012 0.012 0.025; visual mesh filename=../meshes/rh_f03_al_link_pip.stl scale=1.0 1.0 1.0
- link rh_middle_DIP: geometry collision box size=0.01 0.01 0.02; visual mesh filename=../meshes/rh_f03_al_link_dip.stl scale=1.0 1.0 1.0
- link rh_middle_MCP: geometry collision box size=0.015 0.015 0.035; visual mesh filename=../meshes/rh_f03_al_link_mcp.stl scale=1.0 1.0 1.0
- link rh_middle_PIP: geometry collision box size=0.012 0.012 0.025; visual mesh filename=../meshes/rh_f03_al_link_pip.stl scale=1.0 1.0 1.0
- link rh_ring_DIP: geometry collision box size=0.01 0.01 0.02; visual mesh filename=../meshes/rh_f03_al_link_dip.stl scale=1.0 1.0 1.0
- link rh_ring_MCP: geometry collision box size=0.015 0.015 0.035; visual mesh filename=../meshes/rh_f03_al_link_mcp.stl scale=1.0 1.0 1.0
- link rh_ring_PIP: geometry collision box size=0.012 0.012 0.025; visual mesh filename=../meshes/rh_f03_al_link_pip.stl scale=1.0 1.0 1.0
- link rh_thumb_DIP: geometry collision box size=0.01 0.01 0.02; visual mesh filename=../meshes/rh_f03_al_link_dip.stl scale=1.0 1.0 1.0
- link rh_thumb_MCP: geometry collision box size=0.015 0.015 0.035; visual mesh filename=../meshes/rh_f03_al_link_mcp.stl scale=1.0 1.0 1.0
- link rh_thumb_joint: geometry collision box size=0.015 0.015 0.02; visual mesh filename=../meshes/rh_f03_thumb_joint.stl scale=1.0 1.0 1.0
- link rh_wrist_plate: geometry collision mesh filename=../meshes/rh_f03_al_link_hand_wrist_part.stl scale=1.0 1.0 1.0; visual mesh filename=../meshes/rh_f03_al_link_hand_wrist_part.stl scale=1.0 1.0 1.0
Joints:
- joint lh_index_MCP_joint: origin xyz=-0.0002 -0.00677 0.0538 -> xyz=-0.0002 0.00677 0.0538
- joint lh_index_PIP_joint: origin xyz=0.0 -0.00208 0.02677 -> xyz=0.0 0.00208 0.02677
- joint lh_knuckle_index_joint: origin xyz=-0.0313 0.0160 0.0295 -> xyz=-0.0313 -0.016 0.0295
- joint lh_knuckle_little_joint: origin xyz=0.0317 0.0160 0.0295 -> xyz=0.0317 -0.016 0.0295
- joint lh_knuckle_middle_joint: origin xyz=-0.0103 0.0160 0.0295 -> xyz=-0.0103 -0.016 0.0295
- joint lh_knuckle_ring_joint: origin xyz=0.010700000000000001 0.0160 0.0295 -> xyz=0.010700000000000001 -0.016 0.0295
- joint lh_knuckle_thumb_joint: origin xyz=0.0345 0.0162 0.0186 -> xyz=0.0345 -0.0162 0.0186
- joint lh_little_MCP_joint: origin xyz=-0.0002 -0.00677 0.0538 -> xyz=-0.0002 0.00677 0.0538
- joint lh_little_PIP_joint: origin xyz=0.0 -0.00208 0.02677 -> xyz=0.0 0.00208 0.02677
- joint lh_middle_MCP_joint: origin xyz=-0.0002 -0.00677 0.0538 -> xyz=-0.0002 0.00677 0.0538
- joint lh_middle_PIP_joint: origin xyz=0.0 -0.00208 0.02677 -> xyz=0.0 0.00208 0.02677
- joint lh_motor_index_joint: axis 1 0 0 -> (none); origin xyz=0.0 -0.0145 0.006 rpy=1.57 0 0 -> xyz=0.0 0.0145 0.006 rpy=1.57 0 0
- joint lh_motor_little_joint: axis 1 0 0 -> (none); origin xyz=0.0 -0.0145 0.006 rpy=1.57 0 0 -> xyz=0.0 0.0145 0.006 rpy=1.57 0 0
- joint lh_motor_middle_joint: axis 1 0 0 -> (none); origin xyz=0.0 -0.0145 0.006 rpy=1.57 0 0 -> xyz=0.0 0.0145 0.006 rpy=1.57 0 0
- joint lh_motor_ring_joint: axis 1 0 0 -> (none); origin xyz=0.0 -0.0145 0.006 rpy=1.57 0 0 -> xyz=0.0 0.0145 0.006 rpy=1.57 0 0
- joint lh_motor_thumb_DIP_joint: axis 1 0 0 -> (none); origin xyz=0.0125 -0.0055 -0.015 rpy=3.14 3.14 -1.57 -> xyz=0.0125 0.0055 -0.015 rpy=3.14 3.14 1.57
- joint lh_motor_thumb_jo_joint: axis 1 0 0 -> (none); origin xyz=-0.008 -0.015 0.0 rpy=1.57 -1.57 0 -> xyz=-0.008 0.015 0.0 rpy=-1.57 -1.57 0
- joint lh_pris_index_joint: origin xyz=0.0 0.03 0.0 rpy=1.57 0 0 -> xyz=0.0 -0.03 0.0 rpy=-1.57 0 0
- joint lh_pris_little_joint: origin xyz=0.0 0.03 0.0 rpy=1.57 0 0 -> xyz=0.0 -0.03 0.0 rpy=-1.57 0 0
- joint lh_pris_middle_joint: origin xyz=0.0 0.03 0.0 rpy=1.57 0 0 -> xyz=0.0 -0.03 0.0 rpy=-1.57 0 0
- joint lh_pris_ring_joint: origin xyz=0.0 0.03 0.0 rpy=1.57 0 0 -> xyz=0.0 -0.03 0.0 rpy=-1.57 0 0
- joint lh_pris_thumb_DIP_joint: origin xyz=0.0 -0.015 0.0 rpy=1.57 0 0 -> xyz=0.0 0.015 0.0 rpy=-1.57 0 0
- joint lh_pris_thumb_jo_joint: origin xyz=0.0 -0.015 0.0 rpy=1.57 0 0 -> xyz=0.0 0.015 0.0 rpy=-1.57 0 0
- joint lh_ring_MCP_joint: origin xyz=-0.0002 -0.00677 0.0538 -> xyz=-0.0002 0.00677 0.0538
- joint lh_ring_PIP_joint: origin xyz=0.0 -0.00208 0.02677 -> xyz=0.0 0.00208 0.02677
- joint lh_thumb_MCP_joint: origin xyz=-0.031 -0.0055 0.0 rpy=0.0 0.4538 0.0 -> xyz=-0.031 0.0055 0.0 rpy=0.0 0.4538 0.0
- joint lh_thumb_jo_joint: origin xyz=-0.0558 -0.00675 0.0 rpy=0.0 0.0 -0.6021 -> xyz=-0.0558 0.00675 0.0 rpy=0.0 0.0 0.6021
- joint lh_wrist_plate_joint: origin xyz=0 0 0 rpy=-0.7854 3.14159 -1.5708 -> xyz=0 0 0 rpy=0.7854 3.14159 1.5708
- joint rh_knuckle_index_joint: origin xyz=-0.0313 0.0160 0.0295 -> xyz=-0.0313 0.016 0.0295
- joint rh_knuckle_little_joint: origin xyz=0.0317 0.0160 0.0295 -> xyz=0.0317 0.016 0.0295
- joint rh_knuckle_middle_joint: origin xyz=-0.0103 0.0160 0.0295 -> xyz=-0.0103 0.016 0.0295
- joint rh_knuckle_ring_joint: origin xyz=0.010700000000000001 0.0160 0.0295 -> xyz=0.010700000000000001 0.016 0.0295
- joint rh_motor_index_joint: axis 1 0 0 -> (none)
- joint rh_motor_little_joint: axis 1 0 0 -> (none)
- joint rh_motor_middle_joint: axis 1 0 0 -> (none)
- joint rh_motor_ring_joint: axis 1 0 0 -> (none)
- joint rh_motor_thumb_DIP_joint: axis 1 0 0 -> (none)
- joint rh_motor_thumb_jo_joint: axis 1 0 0 -> (none)
- joint rh_wrist_plate_joint: origin xyz=0 0 0 rpy=0.7854 3.14159 -1.5708 -> xyz=0 0 0 rpy=-0.7854 3.14159 -1.5708
