Commit message: Updated xacros for isaaclab

File: assets/urdf/revexbot1.urdf (robot description, URDF)
Before this commit: robot RevEx_Full_Assembly, 106 links, 105 joints
Links:
- link head_link: mass 0.5 -> 1.0; geometry collision box size=0.2 0.16 0.12; visual mesh filename=../meshes/HEAD.STL
- link left_wrist_yaw_link: mass 0.15 -> 0.058058790654763
- link lh_ee_index_link: mass None -> 0.001
- link lh_ee_little_link: mass None -> 0.001
- link lh_ee_middle_link: mass None -> 0.001
- link lh_ee_ring_link: mass None -> 0.001
- link lh_ee_thumb_link: mass None -> 0.001
- link lh_hand_palm: geometry collision box size=0.09 0.03 0.06; visual mesh filename=../meshes/lh_f03_al_palm.stl scale=1.0 1.0 1.0
- link lh_wrist_plate: mass None -> 0.015; geometry collision box size=0.04 0.04 0.01; visual mesh filename=../meshes/lh_f03_al_link_hand_wrist_part.stl scale=1.0 1.0 1.0
- link neck_yaw_link: mass 0.1 -> 0.693
- link rh_ee_index_link: mass None -> 0.001
- link rh_ee_little_link: mass None -> 0.001
- link rh_ee_middle_link: mass None -> 0.001
- link rh_ee_ring_link: mass None -> 0.001
- link rh_ee_thumb_link: mass None -> 0.001
- link rh_hand_palm: geometry collision box size=0.09 0.03 0.06; visual mesh filename=../meshes/rh_f03_al_palm.stl scale=1.0 1.0 1.0
- link rh_wrist_plate: mass None -> 0.015; geometry collision box size=0.04 0.04 0.01; visual mesh filename=../meshes/rh_f03_al_link_hand_wrist_part.stl scale=1.0 1.0 1.0
- link right_wrist_yaw_link: mass 0.15 -> 0.0580595106779709
Joints:
- joint lh_index_DIP_joint: limit lower=0.0 upper=1.0 effort=10.0 velocity=1.0 -> lower=0.0 upper=1.0 effort=3.0 velocity=1.0
- joint lh_index_MCP_joint: limit lower=0.0 upper=1.3 effort=10.0 velocity=1.0 -> lower=0.0 upper=1.3 effort=3.0 velocity=1.0
- joint lh_index_PIP_joint: limit lower=0.0 upper=1.0 effort=10.0 velocity=1.0 -> lower=0.0 upper=1.0 effort=3.0 velocity=1.0
- joint lh_little_DIP_joint: limit lower=0.0 upper=1.0 effort=10.0 velocity=1.0 -> lower=0.0 upper=1.0 effort=3.0 velocity=1.0
- joint lh_little_MCP_joint: limit lower=0.0 upper=1.3 effort=10.0 velocity=1.0 -> lower=0.0 upper=1.3 effort=3.0 velocity=1.0
- joint lh_little_PIP_joint: limit lower=0.0 upper=1.0 effort=10.0 velocity=1.0 -> lower=0.0 upper=1.0 effort=3.0 velocity=1.0
- joint lh_middle_DIP_joint: limit lower=0.0 upper=1.0 effort=10.0 velocity=1.0 -> lower=0.0 upper=1.0 effort=3.0 velocity=1.0
- joint lh_middle_MCP_joint: limit lower=0.0 upper=1.3 effort=10.0 velocity=1.0 -> lower=0.0 upper=1.3 effort=3.0 velocity=1.0
- joint lh_middle_PIP_joint: limit lower=0.0 upper=1.0 effort=10.0 velocity=1.0 -> lower=0.0 upper=1.0 effort=3.0 velocity=1.0
- joint lh_pris_index_joint: limit lower=0.0 upper=0.0103 effort=10.0 velocity=0.1 -> lower=0.0 upper=0.0103 effort=3.0 velocity=0.1
- joint lh_pris_little_joint: limit lower=0.0 upper=0.0103 effort=10.0 velocity=0.1 -> lower=0.0 upper=0.0103 effort=3.0 velocity=0.1
- joint lh_pris_middle_joint: limit lower=0.0 upper=0.0103 effort=10.0 velocity=0.1 -> lower=0.0 upper=0.0103 effort=3.0 velocity=0.1
- joint lh_pris_ring_joint: limit lower=0.0 upper=0.0103 effort=10.0 velocity=0.1 -> lower=0.0 upper=0.0103 effort=3.0 velocity=0.1
- joint lh_pris_thumb_DIP_joint: limit lower=0.0 upper=0.0103 effort=10.0 velocity=0.1 -> lower=0.0 upper=0.0103 effort=3.0 velocity=0.1
- joint lh_pris_thumb_jo_joint: limit lower=0.0 upper=0.0103 effort=10.0 velocity=0.1 -> lower=0.0 upper=0.0103 effort=3.0 velocity=0.1
- joint lh_ring_DIP_joint: limit lower=0.0 upper=1.0 effort=10.0 velocity=1.0 -> lower=0.0 upper=1.0 effort=3.0 velocity=1.0
- joint lh_ring_MCP_joint: limit lower=0.0 upper=1.3 effort=10.0 velocity=1.0 -> lower=0.0 upper=1.3 effort=3.0 velocity=1.0
- joint lh_ring_PIP_joint: limit lower=0.0 upper=1.0 effort=10.0 velocity=1.0 -> lower=0.0 upper=1.0 effort=3.0 velocity=1.0
- joint lh_thumb_DIP_joint: limit lower=0.0 upper=0.8 effort=10.0 velocity=1.0 -> lower=0.0 upper=0.8 effort=3.0 velocity=1.0
- joint lh_thumb_MCP_joint: limit lower=0.0 upper=1.0 effort=10.0 velocity=1.0 -> lower=0.0 upper=1.0 effort=3.0 velocity=1.0
- joint lh_thumb_jo_joint: limit lower=0.0 upper=1.8 effort=10.0 velocity=1.0 -> lower=0.0 upper=1.8 effort=3.0 velocity=1.0
- joint neck_pitch_joint: limit lower=-0.5 upper=0.5 effort=20 velocity=5 -> lower=-0.785398 upper=0.785398 effort=20 velocity=5
- joint rh_index_DIP_joint: limit lower=0.0 upper=1.0 effort=10.0 velocity=1.0 -> lower=0.0 upper=1.0 effort=3.0 velocity=1.0
- joint rh_index_MCP_joint: limit lower=0.0 upper=1.3 effort=10.0 velocity=1.0 -> lower=0.0 upper=1.3 effort=3.0 velocity=1.0
- joint rh_index_PIP_joint: limit lower=0.0 upper=1.0 effort=10.0 velocity=1.0 -> lower=0.0 upper=1.0 effort=3.0 velocity=1.0
- joint rh_little_DIP_joint: limit lower=0.0 upper=1.0 effort=10.0 velocity=1.0 -> lower=0.0 upper=1.0 effort=3.0 velocity=1.0
- joint rh_little_MCP_joint: limit lower=0.0 upper=1.3 effort=10.0 velocity=1.0 -> lower=0.0 upper=1.3 effort=3.0 velocity=1.0
- joint rh_little_PIP_joint: limit lower=0.0 upper=1.0 effort=10.0 velocity=1.0 -> lower=0.0 upper=1.0 effort=3.0 velocity=1.0
- joint rh_middle_DIP_joint: limit lower=0.0 upper=1.0 effort=10.0 velocity=1.0 -> lower=0.0 upper=1.0 effort=3.0 velocity=1.0
- joint rh_middle_MCP_joint: limit lower=0.0 upper=1.3 effort=10.0 velocity=1.0 -> lower=0.0 upper=1.3 effort=3.0 velocity=1.0
- joint rh_middle_PIP_joint: limit lower=0.0 upper=1.0 effort=10.0 velocity=1.0 -> lower=0.0 upper=1.0 effort=3.0 velocity=1.0
- joint rh_pris_index_joint: limit lower=0.0 upper=0.0103 effort=10.0 velocity=0.1 -> lower=0.0 upper=0.0103 effort=3.0 velocity=0.1
- joint rh_pris_little_joint: limit lower=0.0 upper=0.0103 effort=10.0 velocity=0.1 -> lower=0.0 upper=0.0103 effort=3.0 velocity=0.1
- joint rh_pris_middle_joint: limit lower=0.0 upper=0.0103 effort=10.0 velocity=0.1 -> lower=0.0 upper=0.0103 effort=3.0 velocity=0.1
- joint rh_pris_ring_joint: limit lower=0.0 upper=0.0103 effort=10.0 velocity=0.1 -> lower=0.0 upper=0.0103 effort=3.0 velocity=0.1
- joint rh_pris_thumb_DIP_joint: limit lower=0.0 upper=0.0103 effort=10.0 velocity=0.1 -> lower=0.0 upper=0.0103 effort=3.0 velocity=0.1
- joint rh_pris_thumb_jo_joint: limit lower=0.0 upper=0.0103 effort=10.0 velocity=0.1 -> lower=0.0 upper=0.0103 effort=3.0 velocity=0.1
- joint rh_ring_DIP_joint: limit lower=0.0 upper=1.0 effort=10.0 velocity=1.0 -> lower=0.0 upper=1.0 effort=3.0 velocity=1.0
- joint rh_ring_MCP_joint: limit lower=0.0 upper=1.3 effort=10.0 velocity=1.0 -> lower=0.0 upper=1.3 effort=3.0 velocity=1.0
- joint rh_ring_PIP_joint: limit lower=0.0 upper=1.0 effort=10.0 velocity=1.0 -> lower=0.0 upper=1.0 effort=3.0 velocity=1.0
- joint rh_thumb_DIP_joint: limit lower=0.0 upper=0.8 effort=10.0 velocity=1.0 -> lower=0.0 upper=0.8 effort=3.0 velocity=1.0
- joint rh_thumb_MCP_joint: limit lower=0.0 upper=1.0 effort=10.0 velocity=1.0 -> lower=0.0 upper=1.0 effort=3.0 velocity=1.0
- joint rh_thumb_jo_joint: limit lower=0.0 upper=1.8 effort=10.0 velocity=1.0 -> lower=0.0 upper=1.8 effort=3.0 velocity=1.0

File: assets/xacro/hri_hand.xacro (robot description, xacro)
@@ -26,7 +26,11 @@
       </visual>
       <collision>
-        <geometry><mesh filename="${mesh_dir}/${prefix}f03_al_link_hand_wrist_part.stl" scale="1.0 1.0 1.0"/></geometry>
-        <origin xyz="0.0 0.0 0.0" rpy="${1.57 * reflect} 0.0 0.0"/>
+        <geometry><box size="0.04 0.04 0.01"/></geometry>
+        <origin xyz="0.0 0.0 0.0" rpy="0 0 0"/>
       </collision>
+      <inertial>
+        <mass value="0.015"/>
+        <inertia ixx="1.0e-05" ixy="0.0" ixz="0.0" iyy="1.0e-05" iyz="0.0" izz="1.0e-05" />
+      </inertial>
     </link>
     <joint name="${prefix}wrist_plate_joint" type="fixed">
@@ -42,6 +46,6 @@
       </visual>
       <collision>
-        <geometry><mesh filename="${mesh_dir}/${prefix}f03_al_palm.stl" scale="1.0 1.0 1.0"/></geometry>
-        <origin xyz="0.0 ${0.0162 * reflect} 0.030" rpy="${3.14 * reflect} 4.71 0.0"/>
+        <geometry><box size="0.09 0.03 0.06"/></geometry>
+        <origin xyz="0.0 ${0.0162 * reflect} 0.030" rpy="0 0 0"/>
       </collision>
       <inertial>
@@ -64,5 +68,5 @@
         <inertial>
           <mass value="${knucle_mass}"/>
-          <inertia ixx="1.0e-03" ixy="0.0" ixz="0.0" iyy="1.0e-03" iyz="0.0" izz="1.0e-03" />
+          <inertia ixx="1.0e-05" ixy="0.0" ixz="0.0" iyy="1.0e-05" iyz="0.0" izz="1.0e-05" />
         </inertial>
       </link>
@@ -75,8 +79,10 @@
         <visual><geometry><mesh filename="${mesh_dir}/${prefix}f03_al_link_mcp.stl" scale="1.0 1.0 1.0"/></geometry><origin xyz="0.0 ${0.00415 * reflect} -0.00955" rpy="0.0 -1.57 ${3.14 * reflect}"/><material name="white"/></visual>
         <collision><geometry><box size="0.015 0.015 0.035"/></geometry><origin xyz="0.0 0.0 0.015" rpy="0 0 0"/></collision>
-        <inertial><mass value="${MCP_mass}"/><inertia ixx="1.0e-03" ixy="0.0" ixz="0.0" iyy="1.0e-03" iyz="0.0" izz="1.0e-03" /></inertial>
+        <inertial><mass value="${MCP_mass}"/><inertia ixx="1.0e-05" ixy="0.0" ixz="0.0" iyy="1.0e-05" iyz="0.0" izz="1.0e-05" /></inertial>
       </link>
       <joint name="${prefix}${finger_name}_MCP_joint" type="revolute">
-        <axis xyz="-1 0 0"/><limit effort="10.0" lower="0.0" upper="1.3" velocity="1.0"/>
+        <axis xyz="-1 0 0"/>
+        <limit effort="3.0" lower="0.0" upper="1.3" velocity="1.0"/>
+        <dynamics damping="0.5" friction="0.1"/>
         <parent link="${prefix}knuckle_${finger_name}"/><child link="${prefix}${finger_name}_MCP"/>
         <origin xyz="-0.0002 ${-0.00677 * reflect} 0.0538"/>
@@ -86,8 +92,10 @@
         <visual><geometry><mesh filename="${mesh_dir}/${prefix}f03_al_link_pip.stl" scale="1.0 1.0 1.0"/></geometry><origin xyz="-0.0002 ${0.0093 * reflect} -0.00242" rpy="0.0 -1.57 ${3.14 * reflect}"/><material name="white"/></visual>
         <collision><geometry><box size="0.012 0.012 0.025"/></geometry><origin xyz="0.0 0.0 0.01" rpy="0 0 0"/></collision>
-        <inertial><mass value="${PIP_mass}"/><inertia ixx="1.0e-03" ixy="0.0" ixz="0.0" iyy="1.0e-03" iyz="0.0" izz="1.0e-03" /></inertial>
+        <inertial><mass value="${PIP_mass}"/><inertia ixx="1.0e-05" ixy="0.0" ixz="0.0" iyy="1.0e-05" iyz="0.0" izz="1.0e-05" /></inertial>
       </link>
       <joint name="${prefix}${finger_name}_PIP_joint" type="revolute">
-        <axis xyz="-1 0 0"/><limit effort="10.0" lower="0.0" upper="1.0" velocity="1.0"/>
+        <axis xyz="-1 0 0"/>
+        <limit effort="3.0" lower="0.0" upper="1.0" velocity="1.0"/>
+        <dynamics damping="0.5" friction="0.1"/>
         <parent link="${prefix}${finger_name}_MCP"/><child link="${prefix}${finger_name}_PIP"/>
         <origin xyz="0.0 ${-0.00208 * reflect} 0.02677"/>
@@ -97,13 +105,20 @@
         <visual><geometry><mesh filename="${mesh_dir}/${prefix}f03_al_link_dip.stl" scale="1.0 1.0 1.0"/></geometry><origin xyz="0.0 ${0.0075 * reflect} -0.0025" rpy="0.0 -1.57 ${3.14 * reflect}"/><material name="lightyellow"><color rgba="1.0 1.0 0.3 1.0"/></material></visual>
         <collision><geometry><box size="0.01 0.01 0.02"/></geometry><origin xyz="0.0 0.0 0.01" rpy="0 0 0"/></collision>
-        <inertial><mass value="${DIP_mass}"/><inertia ixx="1.0e-03" ixy="0.0" ixz="0.0" iyy="1.0e-03" iyz="0.0" izz="1.0e-03" /></inertial>
+        <inertial><mass value="${DIP_mass}"/><inertia ixx="1.0e-06" ixy="0.0" ixz="0.0" iyy="1.0e-06" iyz="0.0" izz="1.0e-06" /></inertial>
       </link>
       <joint name="${prefix}${finger_name}_DIP_joint" type="revolute">
-        <axis xyz="-1 0 0"/><limit effort="10.0" lower="0.0" upper="1.0" velocity="1.0"/>
+        <axis xyz="-1 0 0"/>
+        <limit effort="3.0" lower="0.0" upper="1.0" velocity="1.0"/>
+        <dynamics damping="0.5" friction="0.1"/>
         <parent link="${prefix}${finger_name}_PIP"/><child link="${prefix}${finger_name}_DIP"/>
         <origin xyz="0.0 0.0 0.0233"/>
         <mimic joint="${prefix}pris_${finger_name}_joint" multiplier="100.00" offset="0.0" />
       </joint>
-      <link name="${prefix}ee_${finger_name}_link"/>
+      <link name="${prefix}ee_${finger_name}_link">
+        <inertial>
+          <mass value="0.001"/>
+          <inertia ixx="1.0e-07" ixy="0.0" ixz="0.0" iyy="1.0e-07" iyz="0.0" izz="1.0e-07" />
+        </inertial>
+      </link>
       <joint name="${prefix}ee_${finger_name}_joint" type="fixed">
         <parent link="${prefix}${finger_name}_DIP"/><child link="${prefix}ee_${finger_name}_link"/>
@@ -112,5 +127,5 @@
       <link name="${prefix}motor_${finger_name}">
         <visual><geometry><box size="${motor_x} ${motor_y} ${motor_z}"/></geometry><origin xyz="0 ${0.02 * reflect} 0"/><material name="black"><color rgba="0.25 0.25 0.25 1"/></material></visual>
-        <inertial><mass value="${motor_mass}"/><inertia ixx="1.0e-03" ixy="0.0" ixz="0.0" iyy="1.0e-03" iyz="0.0" izz="1.0e-03" /></inertial>
+        <inertial><mass value="${motor_mass}"/><inertia ixx="1.0e-05" ixy="0.0" ixz="0.0" iyy="1.0e-05" iyz="0.0" izz="1.0e-05" /></inertial>
       </link>
       <joint name="${prefix}motor_${finger_name}_joint" type="fixed">
@@ -120,8 +135,8 @@
       <link name="${prefix}pris_${finger_name}">
         <visual><geometry><box size="${pris_x} ${pris_y} ${pris_z}"/></geometry><origin xyz="0 0 0"/><material name="black"/></visual>
-        <inertial><mass value="${safe_dummy_mass}"/><inertia ixx="1.0e-03" ixy="0.0" ixz="0.0" iyy="1.0e-03" iyz="0.0" izz="1.0e-03" /></inertial>
+        <inertial><mass value="${safe_dummy_mass}"/><inertia ixx="1.0e-05" ixy="0.0" ixz="0.0" iyy="1.0e-05" iyz="0.0" izz="1.0e-05" /></inertial>
       </link>
       <joint name="${prefix}pris_${finger_name}_joint" type="prismatic">
-        <axis xyz="0 0 -1"/><limit effort="10.0" lower="0.0" upper="${motor_max_upper}" velocity="0.1"/>
+        <axis xyz="0 0 -1"/><limit effort="3.0" lower="0.0" upper="${motor_max_upper}" velocity="0.1"/>
         <parent link="${prefix}motor_${finger_name}"/><child link="${prefix}pris_${finger_name}"/>
         <origin xyz="0.0 ${(motor_joint_y + 0.0445) * reflect} 0.0" rpy="${1.57 * reflect} 0 0"/>
@@ -138,5 +153,5 @@
         <material name="white"/>
       </visual>
-      <inertial><mass value="${knucle_mass}"/><inertia ixx="1.0e-03" ixy="0.0" ixz="0.0" iyy="1.0e-03" iyz="0.0" izz="1.0e-03" /></inertial>
+      <inertial><mass value="${knucle_mass}"/><inertia ixx="1.0e-05" ixy="0.0" ixz="0.0" iyy="1.0e-05" iyz="0.0" izz="1.0e-05" /></inertial>
     </link>
     <joint name="${prefix}knuckle_thumb_joint" type="fixed">
@@ -147,8 +162,10 @@
       <visual><geometry><mesh filename="${mesh_dir}/${prefix}f03_thumb_joint.stl" scale="1.0 1.0 1.0"/></geometry><origin xyz="0 0 -0.005" rpy="0 0 ${3.14 * reflect}"/><material name="white"/></visual>
       <collision><geometry><box size="0.015 0.015 0.02"/></geometry><origin xyz="0 0 0" rpy="0 0 0"/></collision>
-      <inertial><mass value="${motor_mass}"/><inertia ixx="1.0e-03" ixy="0.0" ixz="0.0" iyy="1.0e-03" iyz="0.0" izz="1.0e-03" /></inertial>
+      <inertial><mass value="${motor_mass}"/><inertia ixx="1.0e-05" ixy="0.0" ixz="0.0" iyy="1.0e-05" iyz="0.0" izz="1.0e-05" /></inertial>
     </link>
     <joint name="${prefix}thumb_jo_joint" type="revolute">
-      <axis xyz="0 0 -1"/><limit effort="10.0" lower="0.0" upper="1.8" velocity="1.0"/>
+      <axis xyz="0 0 -1"/>
+      <limit effort="3.0" lower="0.0" upper="1.8" velocity="1.0"/>
+      <dynamics damping="0.5" friction="0.1"/>
       <parent link="${prefix}knuckle_thumb"/><child link="${prefix}thumb_joint"/>
       <origin xyz="-0.0558 ${-0.00675 * reflect} 0.0" rpy="0.0 0.0 ${-0.6021 * reflect}" />
@@ -158,8 +175,10 @@
       <visual><geometry><mesh filename="${mesh_dir}/${prefix}f03_al_link_mcp.stl" scale="1.0 1.0 1.0"/></geometry><origin xyz="0.00955 0.0 0.00415" rpy="${-1.57 * reflect} 0 ${3.14 * reflect}"/><material name="white"/></visual>
       <collision><geometry><box size="0.015 0.015 0.035"/></geometry><origin xyz="0 0 0" rpy="0 0 0"/></collision>
-      <inertial><mass value="${MCP_mass}"/><inertia ixx="1.0e-03" ixy="0.0" ixz="0.0" iyy="1.0e-03" iyz="0.0" izz="1.0e-03" /></inertial>
+      <inertial><mass value="${MCP_mass}"/><inertia ixx="1.0e-05" ixy="0.0" ixz="0.0" iyy="1.0e-05" iyz="0.0" izz="1.0e-05" /></inertial>
     </link>
     <joint name="${prefix}thumb_MCP_joint" type="revolute">
-      <axis xyz="0 1 0"/><limit effort="10.0" lower="0.0" upper="1.0" velocity="1.0"/>
+      <axis xyz="0 1 0"/>
+      <limit effort="3.0" lower="0.0" upper="1.0" velocity="1.0"/>
+      <dynamics damping="0.5" friction="0.1"/>
       <parent link="${prefix}thumb_joint"/><child link="${prefix}thumb_MCP"/>
       <origin xyz="-0.031 ${-0.0055 * reflect} 0.0" rpy="0.0 0.4538 0.0"/>
@@ -169,13 +188,20 @@
       <visual><geometry><mesh filename="${mesh_dir}/${prefix}f03_al_link_dip.stl" scale="1.0 1.0 1.0"/></geometry><origin xyz="0.00255 0.0 0.00726" rpy="${-1.57 * reflect} 0 ${3.14 * reflect}"/><material name="lightyellow"><color rgba="1.0 1.0 0.3 1.0"/></material></visual>
       <collision><geometry><box size="0.01 0.01 0.02"/></geometry><origin xyz="0 0 0" rpy="0 0 0"/></collision>
-      <inertial><mass value="${DIP_mass}"/><inertia ixx="1.0e-03" ixy="0.0" ixz="0.0" iyy="1.0e-03" iyz="0.0" izz="1.0e-03" /></inertial>
+      <inertial><mass value="${DIP_mass}"/><inertia ixx="1.0e-06" ixy="0.0" ixz="0.0" iyy="1.0e-06" iyz="0.0" izz="1.0e-06" /></inertial>
     </link>
     <joint name="${prefix}thumb_DIP_joint" type="revolute">
-      <axis xyz="0 1 0"/><limit effort="10.0" lower="0.0" upper="0.8" velocity="1.0"/>
+      <axis xyz="0 1 0"/>
+      <limit effort="3.0" lower="0.0" upper="0.8" velocity="1.0"/>
+      <dynamics damping="0.5" friction="0.1"/>
       <parent link="${prefix}thumb_MCP"/><child link="${prefix}thumb_DIP"/>
       <origin xyz="-0.0298 0.0 -0.0042" rpy="0.0 0.0 0.0"/>
       <mimic joint="${prefix}pris_thumb_DIP_joint" multiplier="100.00" offset="0.0" />
     </joint>
-    <link name="${prefix}ee_thumb_link"/>
+    <link name="${prefix}ee_thumb_link">
+      <inertial>
+        <mass value="0.001"/>
+        <inertia ixx="1.0e-07" ixy="0.0" ixz="0.0" iyy="1.0e-07" iyz="0.0" izz="1.0e-07" />
+      </inertial>
+    </link>
     <joint name="${prefix}ee_th_joint" type="fixed">
       <parent link="${prefix}thumb_DIP"/><child link="${prefix}ee_thumb_link"/>
@@ -184,5 +210,5 @@
     <link name="${prefix}motor_thumb_jo">
       <visual><geometry><box size="${motor_x} ${motor_y} ${motor_z}"/></geometry><origin xyz="0 ${0.02 * reflect} 0"/><material name="black"/></visual>
-      <inertial><mass value="${motor_mass}"/><inertia ixx="1.0e-03" ixy="0.0" ixz="0.0" iyy="1.0e-03" iyz="0.0" izz="1.0e-03" /></inertial>
+      <inertial><mass value="${motor_mass}"/><inertia ixx="1.0e-05" ixy="0.0" ixz="0.0" iyy="1.0e-05" iyz="0.0" izz="1.0e-05" /></inertial>
     </link>
     <joint name="${prefix}motor_thumb_jo_joint" type="fixed">
@@ -192,8 +218,8 @@
     <link name="${prefix}pris_thumb_jo">
       <visual><geometry><box size="${pris_x} ${pris_y} ${pris_z}"/></geometry><origin xyz="0 0 0"/><material name="black"/></visual>
-      <inertial><mass value="${safe_dummy_mass}"/><inertia ixx="1.0e-03" ixy="0.0" ixz="0.0" iyy="1.0e-03" iyz="0.0" izz="1.0e-03" /></inertial>
+      <inertial><mass value="${safe_dummy_mass}"/><inertia ixx="1.0e-05" ixy="0.0" ixz="0.0" iyy="1.0e-05" iyz="0.0" izz="1.0e-05" /></inertial>
     </link>
     <joint name="${prefix}pris_thumb_jo_joint" type="prismatic">
-      <axis xyz="0 0 -1"/><limit effort="10.0" lower="0.0" upper="${motor_max_upper}" velocity="0.1"/>
+      <axis xyz="0 0 -1"/><limit effort="3.0" lower="0.0" upper="${motor_max_upper}" velocity="0.1"/>
       <parent link="${prefix}motor_thumb_jo"/><child link="${prefix}pris_thumb_jo"/>
       <origin xyz="0.0 ${-0.015 * reflect} 0.0" rpy="${1.57 * reflect} 0 0"/>
@@ -201,5 +227,5 @@
     <link name="${prefix}motor_thumb_DIP">
       <visual><geometry><box size="${motor_x} ${motor_y} ${motor_z}"/></geometry><origin xyz="0 ${0.02 * reflect} 0"/><material name="black"/></visual>
-      <inertial><mass value="${DIP_mass}"/><inertia ixx="1.0e-03" ixy="0.0" ixz="0.0" iyy="1.0e-03" iyz="0.0" izz="1.0e-03" /></inertial>
+      <inertial><mass value="${DIP_mass}"/><inertia ixx="1.0e-06" ixy="0.0" ixz="0.0" iyy="1.0e-06" iyz="0.0" izz="1.0e-06" /></inertial>
     </link>
     <joint name="${prefix}motor_thumb_DIP_joint" type="fixed">
@@ -209,8 +235,8 @@
     <link name="${prefix}pris_thumb_DIP">
       <visual><geometry><box size="${pris_x} ${pris_y} ${pris_z}"/></geometry><origin xyz="0 0 0"/><material name="black"/></visual>
-      <inertial><mass value="${safe_dummy_mass}"/><inertia ixx="1.0e-03" ixy="0.0" ixz="0.0" iyy="1.0e-03" iyz="0.0" izz="1.0e-03" /></inertial>
+      <inertial><mass value="${safe_dummy_mass}"/><inertia ixx="1.0e-05" ixy="0.0" ixz="0.0" iyy="1.0e-05" iyz="0.0" izz="1.0e-05" /></inertial>
     </link>
     <joint name="${prefix}pris_thumb_DIP_joint" type="prismatic">
-      <axis xyz="0 0 -1"/><limit effort="10.0" lower="0.0" upper="${motor_max_upper}" velocity="0.1"/>
+      <axis xyz="0 0 -1"/><limit effort="3.0" lower="0.0" upper="${motor_max_upper}" velocity="0.1"/>
       <parent link="${prefix}motor_thumb_DIP"/><child link="${prefix}pris_thumb_DIP"/>
       <origin xyz="0.0 ${-0.015 * reflect} 0.0" rpy="${1.57 * reflect} 0 0"/>
