Commit message: Updated xacros for isaaclab

File: assets/xacro/master_assembly.xacro (robot description, xacro)
@@ -5,5 +5,4 @@
   <material name="DarkGrey"><color rgba="0.22 0.22 0.22 1.0" /></material>
   <material name="LightGrey"><color rgba="0.8 0.8 0.8 1.0" /></material>
-  <!-- ========== PELVIS ========== -->
   <link name="pelvis_link">
     <inertial>
@@ -23,5 +22,4 @@
     </collision>
   </link>
-  <!-- ========== LEFT LEG ========== -->
   <link name="left_hip_pitch_link">
     <inertial>
@@ -42,5 +40,4 @@
     <axis xyz="0 1 0" />
     <limit lower="-2.094" upper="1.0" effort="120" velocity="8" />
-    <!-- GAP 1 FIX: Added armature for gearbox inertia -->
     <dynamics damping="0.095625" friction="0.15" armature="0.02" />
   </joint>
@@ -140,5 +137,4 @@
     </inertial>
     <visual><origin xyz="0 0.008 0" rpy="0 0 0" /><geometry><mesh filename="${mesh_dir}/LEFT_TOE.STL" /></geometry><material name="DarkGrey" /></visual>
-    <!-- GAP 3 FIX: Padded collision box to prevent floor clipping -->
     <collision name="left_toe_collision">
       <origin xyz="0.025 0 0.006" rpy="0 0 0" />
@@ -153,5 +149,4 @@
     <dynamics damping="0.001" friction="0.02" armature="0.001" />
   </joint>
-  <!-- ========== RIGHT LEG ========== -->
   <link name="right_hip_pitch_link">
     <inertial>
@@ -269,5 +264,4 @@
     </inertial>
     <visual><origin xyz="0 -0.008 0" rpy="0 0 0" /><geometry><mesh filename="${mesh_dir}/RIGHT_TOE.STL" /></geometry><material name="DarkGrey" /></visual>
-    <!-- GAP 3 FIX: Padded collision box to prevent floor clipping -->
     <collision name="right_toe_collision">
       <origin xyz="0.025 0 0.006" rpy="0 0 0" />
@@ -282,5 +276,4 @@
     <dynamics damping="0.001" friction="0.02" armature="0.001" />
   </joint>
-  <!-- ========== UPPER BODY ========== -->
   <link name="waist_yaw_link">
     <inertial>
@@ -303,10 +296,10 @@
     <dynamics damping="0.095625" friction="0.15" armature="0.02" />
   </joint>
-  <!-- ========== NECK & HEAD ========== -->
   <link name="neck_yaw_link">
     <inertial>
-      <origin xyz="0 0 0.01" rpy="0 0 0" />
-      <mass value="0.1" />
-      <inertia ixx="0.001" ixy="0" ixz="0" iyy="0.001" iyz="0" izz="0.001" />
+      <origin xyz="-0.000232155049410487 -0.000686932388815892 0.0356746841654919" rpy="0 0 0" />
+      <mass value="0.693" />
+      <inertia ixx="0.000343" ixy="-4.52e-12" ixz="1.57e-05"
+               iyy="0.000324" iyz="-1.15e-10" izz="0.000263" />
     </inertial>
     <visual>
@@ -326,14 +319,15 @@
     <inertial>
       <origin xyz="0 0 0.05" rpy="0 0 0" />
-      <mass value="0.5" />
-      <inertia ixx="0.01" ixy="0" ixz="0" iyy="0.01" iyz="0" izz="0.01" />
+      <mass value="1.0" />
+      <inertia ixx="0.004" ixy="0" ixz="0"
+               iyy="0.004" iyz="0" izz="0.004" />
     </inertial>
     <visual>
       <origin xyz="0 0 0" rpy="0 0 0" />
-      <geometry><mesh filename="${mesh_dir}/head.stl" /></geometry>
+      <geometry><mesh filename="${mesh_dir}/HEAD.STL" /></geometry>
       <material name="LightGrey" />
     </visual>
     <collision>
-      <origin xyz="0 0 0.05" rpy="0 0 0" />
+      <origin xyz="0.03 0 0.02" rpy="0 0 0" />
       <geometry><box size="0.2 0.16 0.12" /></geometry>
     </collision>
@@ -343,8 +337,7 @@
     <parent link="neck_yaw_link" /><child link="head_link" />
     <axis xyz="0 1 0" />
-    <limit lower="-0.5" upper="0.5" effort="20" velocity="5" />
+    <limit lower="-0.785398" upper="0.785398" effort="20" velocity="5" />
     <dynamics damping="0.0565" friction="0.08" armature="0.001" />
   </joint>
-  <!-- ========== RIGHT ARM ========== -->
   <link name="right_shoulder_pitch_link">
     <inertial>
@@ -419,10 +412,10 @@
     <dynamics damping="0.0282528" friction="0.08" armature="0.01" />
   </joint>
-  <!-- GAP 2 FIX: Inflated wrist mass and inertia for stability -->
   <link name="right_wrist_yaw_link">
     <inertial>
       <origin xyz="0.00382289129248181 8.36540312021405E-09 -0.00320778585722904" rpy="0 0 0" />
-      <mass value="0.15" />
-      <inertia ixx="0.0001" ixy="0" ixz="0" iyy="0.0001" iyz="0" izz="0.0001" />
+      <mass value="0.0580595106779709" />
+      <inertia ixx="1.18803001723724E-05" ixy="3.73796867740447E-08" ixz="-3.06346018877142E-06"
+               iyy="8.8546080362749E-06" iyz="4.45423430732884E-08" izz="1.07999391749915E-05" />
     </inertial>
     <visual><geometry><mesh filename="${mesh_dir}/RIGHT_WRIST_YAW.STL" /></geometry><material name="Grey" /></visual>
@@ -435,5 +428,4 @@
     <dynamics damping="0.0282528" friction="0.08" armature="0.001" />
   </joint>
-  <!-- ========== LEFT ARM ========== -->
   <link name="left_shoulder_pitch_link">
     <inertial>
@@ -508,10 +500,10 @@
     <dynamics damping="0.0282528" friction="0.08" armature="0.01" />
   </joint>
-  <!-- GAP 2 FIX: Inflated wrist mass and inertia for stability -->
   <link name="left_wrist_yaw_link">
     <inertial>
       <origin xyz="0.00382289324376062 1.7394452961339E-08 -0.00320774203668756" rpy="0 0 0" />
-      <mass value="0.15" />
-      <inertia ixx="0.0001" ixy="0" ixz="0" iyy="0.0001" iyz="0" izz="0.0001" />
+      <mass value="0.058058790654763" />
+      <inertia ixx="1.20674298017884E-05" ixy="1.83335345917148E-07" ixz="-2.8402536561247E-06"
+               iyy="8.40130139890341E-06" iyz="2.18479301532613E-07" izz="1.10658034937549E-05" />
     </inertial>
     <visual><geometry><mesh filename="${mesh_dir}/LEFT_WRIST_YAW.STL" /></geometry><material name="Grey" /></visual>
@@ -524,5 +516,5 @@
     <dynamics damping="0.0282528" friction="0.08" armature="0.001" />
   </joint>
-<xacro:include filename="hri_hand.xacro" />
+  <xacro:include filename="hri_hand.xacro" />
   <xacro:hri_hand
       prefix="rh_"

Commit message: feat: complete project (pipeline, training, configs, envs, models)

File: assets/urdf/revexbot1.urdf (robot description, URDF)
Before this commit: robot RevEx_Full_Assembly, 106 links, 105 joints
Links:
- link lh_ee_index_link: mass 0.001 -> 0.01
- link lh_ee_little_link: mass 0.001 -> 0.01
- link lh_ee_middle_link: mass 0.001 -> 0.01
- link lh_ee_ring_link: mass 0.001 -> 0.01
- link lh_ee_thumb_link: mass 0.001 -> 0.01
- link lh_index_DIP: mass 0.0025 -> 0.01
- link lh_little_DIP: mass 0.0025 -> 0.01
- link lh_middle_DIP: mass 0.0025 -> 0.01
- link lh_motor_thumb_DIP: mass 0.0025 -> 0.01
- link lh_ring_DIP: mass 0.0025 -> 0.01
- link lh_thumb_DIP: mass 0.0025 -> 0.01
- link rh_ee_index_link: mass 0.001 -> 0.01
- link rh_ee_little_link: mass 0.001 -> 0.01
- link rh_ee_middle_link: mass 0.001 -> 0.01
- link rh_ee_ring_link: mass 0.001 -> 0.01
- link rh_ee_thumb_link: mass 0.001 -> 0.01
- link rh_index_DIP: mass 0.0025 -> 0.01
- link rh_little_DIP: mass 0.0025 -> 0.01
- link rh_middle_DIP: mass 0.0025 -> 0.01
- link rh_motor_thumb_DIP: mass 0.0025 -> 0.01
- link rh_ring_DIP: mass 0.0025 -> 0.01
- link rh_thumb_DIP: mass 0.0025 -> 0.01

File: assets/xacro/hri_hand.xacro (robot description, xacro)
@@ -8,9 +8,10 @@
     <xacro:property name="pris_y" value="0.005" />
     <xacro:property name="pris_z" value="0.025" />
+    <xacro:property name="safe_min_mass" value="0.01" />
+    <xacro:property name="safe_inertia" value="1.0e-05" />
     <xacro:property name="knucle_mass" value="0.010" />
     <xacro:property name="MCP_mass" value="0.0125" />
     <xacro:property name="PIP_mass" value="0.0125" />
-    <xacro:property name="DIP_mass" value="0.0025" />
-    <xacro:property name="motor_mass" value="0.015" />
+    <xacro:property name="DIP_mass" value="${safe_min_mass}" /> <xacro:property name="motor_mass" value="0.015" />
     <xacro:property name="safe_dummy_mass" value="0.015" />
     <xacro:property name="motor_joint_x" value="0.0" />
@@ -31,5 +32,5 @@
       <inertial>
         <mass value="0.015"/>
-        <inertia ixx="1.0e-05" ixy="0.0" ixz="0.0" iyy="1.0e-05" iyz="0.0" izz="1.0e-05" />
+        <inertia ixx="${safe_inertia}" ixy="0.0" ixz="0.0" iyy="${safe_inertia}" iyz="0.0" izz="${safe_inertia}" />
       </inertial>
     </link>
@@ -68,5 +69,5 @@
         <inertial>
           <mass value="${knucle_mass}"/>
-          <inertia ixx="1.0e-05" ixy="0.0" ixz="0.0" iyy="1.0e-05" iyz="0.0" izz="1.0e-05" />
+          <inertia ixx="${safe_inertia}" ixy="0.0" ixz="0.0" iyy="${safe_inertia}" iyz="0.0" izz="${safe_inertia}" />
         </inertial>
       </link>
@@ -79,5 +80,5 @@
         <visual><geometry><mesh filename="${mesh_dir}/${prefix}f03_al_link_mcp.stl" scale="1.0 1.0 1.0"/></geometry><origin xyz="0.0 ${0.00415 * reflect} -0.00955" rpy="0.0 -1.57 ${3.14 * reflect}"/><material name="white"/></visual>
         <collision><geometry><box size="0.015 0.015 0.035"/></geometry><origin xyz="0.0 0.0 0.015" rpy="0 0 0"/></collision>
-        <inertial><mass value="${MCP_mass}"/><inertia ixx="1.0e-05" ixy="0.0" ixz="0.0" iyy="1.0e-05" iyz="0.0" izz="1.0e-05" /></inertial>
+        <inertial><mass value="${MCP_mass}"/><inertia ixx="${safe_inertia}" ixy="0.0" ixz="0.0" iyy="${safe_inertia}" iyz="0.0" izz="${safe_inertia}" /></inertial>
       </link>
       <joint name="${prefix}${finger_name}_MCP_joint" type="revolute">
@@ -92,5 +93,5 @@
         <visual><geometry><mesh filename="${mesh_dir}/${prefix}f03_al_link_pip.stl" scale="1.0 1.0 1.0"/></geometry><origin xyz="-0.0002 ${0.0093 * reflect} -0.00242" rpy="0.0 -1.57 ${3.14 * reflect}"/><material name="white"/></visual>
         <collision><geometry><box size="0.012 0.012 0.025"/></geometry><origin xyz="0.0 0.0 0.01" rpy="0 0 0"/></collision>
-        <inertial><mass value="${PIP_mass}"/><inertia ixx="1.0e-05" ixy="0.0" ixz="0.0" iyy="1.0e-05" iyz="0.0" izz="1.0e-05" /></inertial>
+        <inertial><mass value="${PIP_mass}"/><inertia ixx="${safe_inertia}" ixy="0.0" ixz="0.0" iyy="${safe_inertia}" iyz="0.0" izz="${safe_inertia}" /></inertial>
       </link>
       <joint name="${prefix}${finger_name}_PIP_joint" type="revolute">
@@ -105,5 +106,5 @@
         <visual><geometry><mesh filename="${mesh_dir}/${prefix}f03_al_link_dip.stl" scale="1.0 1.0 1.0"/></geometry><origin xyz="0.0 ${0.0075 * reflect} -0.0025" rpy="0.0 -1.57 ${3.14 * reflect}"/><material name="lightyellow"><color rgba="1.0 1.0 0.3 1.0"/></material></visual>
         <collision><geometry><box size="0.01 0.01 0.02"/></geometry><origin xyz="0.0 0.0 0.01" rpy="0 0 0"/></collision>
-        <inertial><mass value="${DIP_mass}"/><inertia ixx="1.0e-06" ixy="0.0" ixz="0.0" iyy="1.0e-06" iyz="0.0" izz="1.0e-06" /></inertial>
+        <inertial><mass value="${DIP_mass}"/><inertia ixx="${safe_inertia}" ixy="0.0" ixz="0.0" iyy="${safe_inertia}" iyz="0.0" izz="${safe_inertia}" /></inertial>
       </link>
       <joint name="${prefix}${finger_name}_DIP_joint" type="revolute">
@@ -117,6 +118,6 @@
       <link name="${prefix}ee_${finger_name}_link">
         <inertial>
-          <mass value="0.001"/>
-          <inertia ixx="1.0e-07" ixy="0.0" ixz="0.0" iyy="1.0e-07" iyz="0.0" izz="1.0e-07" />
+          <mass value="${safe_min_mass}"/>
+          <inertia ixx="${safe_inertia}" ixy="0.0" ixz="0.0" iyy="${safe_inertia}" iyz="0.0" izz="${safe_inertia}" />
         </inertial>
       </link>
@@ -127,5 +128,5 @@
       <link name="${prefix}motor_${finger_name}">
         <visual><geometry><box size="${motor_x} ${motor_y} ${motor_z}"/></geometry><origin xyz="0 ${0.02 * reflect} 0"/><material name="black"><color rgba="0.25 0.25 0.25 1"/></material></visual>
-        <inertial><mass value="${motor_mass}"/><inertia ixx="1.0e-05" ixy="0.0" ixz="0.0" iyy="1.0e-05" iyz="0.0" izz="1.0e-05" /></inertial>
+        <inertial><mass value="${motor_mass}"/><inertia ixx="${safe_inertia}" ixy="0.0" ixz="0.0" iyy="${safe_inertia}" iyz="0.0" izz="${safe_inertia}" /></inertial>
       </link>
       <joint name="${prefix}motor_${finger_name}_joint" type="fixed">
@@ -135,5 +136,5 @@
       <link name="${prefix}pris_${finger_name}">
         <visual><geometry><box size="${pris_x} ${pris_y} ${pris_z}"/></geometry><origin xyz="0 0 0"/><material name="black"/></visual>
-        <inertial><mass value="${safe_dummy_mass}"/><inertia ixx="1.0e-05" ixy="0.0" ixz="0.0" iyy="1.0e-05" iyz="0.0" izz="1.0e-05" /></inertial>
+        <inertial><mass value="${safe_dummy_mass}"/><inertia ixx="${safe_inertia}" ixy="0.0" ixz="0.0" iyy="${safe_inertia}" iyz="0.0" izz="${safe_inertia}" /></inertial>
       </link>
       <joint name="${prefix}pris_${finger_name}_joint" type="prismatic">
@@ -153,5 +154,5 @@
         <material name="white"/>
       </visual>
-      <inertial><mass value="${knucle_mass}"/><inertia ixx="1.0e-05" ixy="0.0" ixz="0.0" iyy="1.0e-05" iyz="0.0" izz="1.0e-05" /></inertial>
+      <inertial><mass value="${knucle_mass}"/><inertia ixx="${safe_inertia}" ixy="0.0" ixz="0.0" iyy="${safe_inertia}" iyz="0.0" izz="${safe_inertia}" /></inertial>
     </link>
     <joint name="${prefix}knuckle_thumb_joint" type="fixed">
@@ -162,5 +163,5 @@
       <visual><geometry><mesh filename="${mesh_dir}/${prefix}f03_thumb_joint.stl" scale="1.0 1.0 1.0"/></geometry><origin xyz="0 0 -0.005" rpy="0 0 ${3.14 * reflect}"/><material name="white"/></visual>
       <collision><geometry><box size="0.015 0.015 0.02"/></geometry><origin xyz="0 0 0" rpy="0 0 0"/></collision>
-      <inertial><mass value="${motor_mass}"/><inertia ixx="1.0e-05" ixy="0.0" ixz="0.0" iyy="1.0e-05" iyz="0.0" izz="1.0e-05" /></inertial>
+      <inertial><mass value="${motor_mass}"/><inertia ixx="${safe_inertia}" ixy="0.0" ixz="0.0" iyy="${safe_inertia}" iyz="0.0" izz="${safe_inertia}" /></inertial>
     </link>
     <joint name="${prefix}thumb_jo_joint" type="revolute">
@@ -175,5 +176,5 @@
       <visual><geometry><mesh filename="${mesh_dir}/${prefix}f03_al_link_mcp.stl" scale="1.0 1.0 1.0"/></geometry><origin xyz="0.00955 0.0 0.00415" rpy="${-1.57 * reflect} 0 ${3.14 * reflect}"/><material name="white"/></visual>
       <collision><geometry><box size="0.015 0.015 0.035"/></geometry><origin xyz="0 0 0" rpy="0 0 0"/></collision>
-      <inertial><mass value="${MCP_mass}"/><inertia ixx="1.0e-05" ixy="0.0" ixz="0.0" iyy="1.0e-05" iyz="0.0" izz="1.0e-05" /></inertial>
+      <inertial><mass value="${MCP_mass}"/><inertia ixx="${safe_inertia}" ixy="0.0" ixz="0.0" iyy="${safe_inertia}" iyz="0.0" izz="${safe_inertia}" /></inertial>
     </link>
     <joint name="${prefix}thumb_MCP_joint" type="revolute">
@@ -188,5 +189,5 @@
       <visual><geometry><mesh filename="${mesh_dir}/${prefix}f03_al_link_dip.stl" scale="1.0 1.0 1.0"/></geometry><origin xyz="0.00255 0.0 0.00726" rpy="${-1.57 * reflect} 0 ${3.14 * reflect}"/><material name="lightyellow"><color rgba="1.0 1.0 0.3 1.0"/></material></visual>
       <collision><geometry><box size="0.01 0.01 0.02"/></geometry><origin xyz="0 0 0" rpy="0 0 0"/></collision>
-      <inertial><mass value="${DIP_mass}"/><inertia ixx="1.0e-06" ixy="0.0" ixz="0.0" iyy="1.0e-06" iyz="0.0" izz="1.0e-06" /></inertial>
+      <inertial><mass value="${DIP_mass}"/><inertia ixx="${safe_inertia}" ixy="0.0" ixz="0.0" iyy="${safe_inertia}" iyz="0.0" izz="${safe_inertia}" /></inertial>
     </link>
     <joint name="${prefix}thumb_DIP_joint" type="revolute">
@@ -200,6 +201,6 @@
     <link name="${prefix}ee_thumb_link">
       <inertial>
-        <mass value="0.001"/>
-        <inertia ixx="1.0e-07" ixy="0.0" ixz="0.0" iyy="1.0e-07" iyz="0.0" izz="1.0e-07" />
+        <mass value="${safe_min_mass}"/>
+        <inertia ixx="${safe_inertia}" ixy="0.0" ixz="0.0" iyy="${safe_inertia}" iyz="0.0" izz="${safe_inertia}" />
       </inertial>
     </link>
@@ -210,5 +211,5 @@
     <link name="${prefix}motor_thumb_jo">
       <visual><geometry><box size="${motor_x} ${motor_y} ${motor_z}"/></geometry><origin xyz="0 ${0.02 * reflect} 0"/><material name="black"/></visual>
-      <inertial><mass value="${motor_mass}"/><inertia ixx="1.0e-05" ixy="0.0" ixz="0.0" iyy="1.0e-05" iyz="0.0" izz="1.0e-05" /></inertial>
+      <inertial><mass value="${motor_mass}"/><inertia ixx="${safe_inertia}" ixy="0.0" ixz="0.0" iyy="${safe_inertia}" iyz="0.0" izz="${safe_inertia}" /></inertial>
     </link>
     <joint name="${prefix}motor_thumb_jo_joint" type="fixed">
@@ -218,5 +219,5 @@
     <link name="${prefix}pris_thumb_jo">
       <visual><geometry><box size="${pris_x} ${pris_y} ${pris_z}"/></geometry><origin xyz="0 0 0"/><material name="black"/></visual>
-      <inertial><mass value="${safe_dummy_mass}"/><inertia ixx="1.0e-05" ixy="0.0" ixz="0.0" iyy="1.0e-05" iyz="0.0" izz="1.0e-05" /></inertial>
+      <inertial><mass value="${safe_dummy_mass}"/><inertia ixx="${safe_inertia}" ixy="0.0" ixz="0.0" iyy="${safe_inertia}" iyz="0.0" izz="${safe_inertia}" /></inertial>
     </link>
     <joint name="${prefix}pris_thumb_jo_joint" type="prismatic">
@@ -227,5 +228,5 @@
     <link name="${prefix}motor_thumb_DIP">
       <visual><geometry><box size="${motor_x} ${motor_y} ${motor_z}"/></geometry><origin xyz="0 ${0.02 * reflect} 0"/><material name="black"/></visual>
-      <inertial><mass value="${DIP_mass}"/><inertia ixx="1.0e-06" ixy="0.0" ixz="0.0" iyy="1.0e-06" iyz="0.0" izz="1.0e-06" /></inertial>
+      <inertial><mass value="${safe_min_mass}"/><inertia ixx="${safe_inertia}" ixy="0.0" ixz="0.0" iyy="${safe_inertia}" iyz="0.0" izz="${safe_inertia}" /></inertial>
     </link>
     <joint name="${prefix}motor_thumb_DIP_joint" type="fixed">
@@ -235,5 +236,5 @@
     <link name="${prefix}pris_thumb_DIP">
       <visual><geometry><box size="${pris_x} ${pris_y} ${pris_z}"/></geometry><origin xyz="0 0 0"/><material name="black"/></visual>
-      <inertial><mass value="${safe_dummy_mass}"/><inertia ixx="1.0e-05" ixy="0.0" ixz="0.0" iyy="1.0e-05" iyz="0.0" izz="1.0e-05" /></inertial>
+      <inertial><mass value="${safe_dummy_mass}"/><inertia ixx="${safe_inertia}" ixy="0.0" ixz="0.0" iyy="${safe_inertia}" iyz="0.0" izz="${safe_inertia}" /></inertial>
     </link>
     <joint name="${prefix}pris_thumb_DIP_joint" type="prismatic">
